File: coupon/coupon.kicad_pcb (KiCad board)
At the start: 2 copper layers, 112 x 90 mm, 65 parts, among them J1 5V IN, J2 IN N1 N2 N3, Q1 2N7000, Q10 2N7000, Q11 2N7000, Q12 2N7000, Q13 2N7000, Q14 2N7000, Q15 2N7000, Q16 2N7000, Q17 2N7000, Q18 2N7000, Q19 2N7000, Q2 2N7000, Q20 2N7000, Q21 2N7000, Q22 2N7000, Q23 2N7000, Q24 2N7000, Q25 2N7000, Q26 2N7000, Q3 2N7000, Q4 2N7000, Q5 2N7000, Q6 2N7000, Q7 2N7000, Q8 2N7000, Q9 2N7000

Commit message: Coupon, ALU and hub PCBs routed and DRC clean; fab outputs
pcb.py: power pre-routed as per-column rails from the tile geometry, fixed in
the DSN so the router cannot move them; GND pour before routing; DRC-verified
ground stitching; inset outline while routing; retries until zero unconnected.
Coupon 112x94, ALU 156x214, hub 130x98 mm. docs/bring-up.md and docs/order-1.md.

Co-Authored-By: Claude Fable 5.1 <noreply@anthropic.com>
Claude-Session: https://claude.ai/code/session_019vcbW37ERmrjZaWq55Er3J
Parts:
- moved Q25 4.00 mm to (6.00, 65.2)
- moved D1 4.00 mm to (17.4, 72.8)
- moved Q11 4.00 mm to (6.00, 52.5)
- moved Q12 4.00 mm to (16.2, 52.5)
- moved Q13 4.00 mm to (26.3, 52.5)
- moved Q14 4.00 mm to (36.5, 52.5)
- moved Q15 4.00 mm to (46.6, 52.5)
- moved Q16 4.00 mm to (56.8, 52.5)
- moved Q17 4.00 mm to (67.0, 52.5)
- moved Q18 4.00 mm to (77.1, 52.5)
- moved Q19 4.00 mm to (87.3, 52.5)
- moved Q20 4.00 mm to (87.3, 57.6)
- moved Q21 4.00 mm to (87.3, 62.6)
- moved Q22 4.00 mm to (97.4, 52.5)
- moved Q23 4.00 mm to (97.4, 57.6)
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Routing:
- net GND: track 380.6 -> 567.1 mm, vias 0 -> 12
- net +5V: track 287.8 -> 466.7 mm, vias 0 -> 10
- net N2: track 106.4 -> 141.4 mm, vias 0 -> 2
- net TP_BUS: track 127.3 -> 159.4 mm
- net N1: track 112.8 -> 134.7 mm, vias 1 -> 2
- net TP_NOR: track 58.7 -> 75.6 mm
- net IN: track 142.9 -> 155.3 mm, vias 0 -> 1
- net N3: track 116.3 -> 106.4 mm, vias 0 -> 1
- net TP_RING: track 24.0 -> 28.6 mm, vias 0 -> 1
- net TP_NAND: track 47.2 -> 51.2 mm
- net TP_FO1: track 32.8 -> 36.8 mm
- net TP_FO10: track 146.6 -> 148.9 mm
Other:
- board size 112 x 90 mm -> 112 x 94 mm
