File: boards/06-panel/panel.kicad_sch (KiCad schematic)
At the start: 229 parts, among them J1 BUS, Q1 2N7000, Q10 2N7000, Q11 2N7000, Q12 2N7000, Q13 2N7000, Q14 2N7000, Q15 2N7000, Q16 2N7000, Q17 2N7000, Q18 2N7000, Q19 2N7000, Q2 2N7000, Q20 2N7000, Q21 2N7000, Q22 2N7000, Q23 2N7000, Q24 2N7000, Q25 2N7000, Q26 2N7000, Q27 2N7000, Q28 2N7000, Q29 2N7000, Q3 2N7000, Q30 2N7000, Q31 2N7000, Q32 2N7000, Q33 2N7000, Q34 2N7000, Q35 2N7000, Q36 2N7000, Q37 2N7000, Q38 2N7000, Q39 2N7000, Q4 2N7000, Q40 2N7000, Q41 2N7000, Q42 2N7000, Q43 2N7000, Q44 2N7000, Q45 2N7000, Q46 2N7000, Q47 2N7000, Q48 2N7000, Q49 2N7000, Q5 2N7000, Q50 2N7000, Q6 2N7000, Q7 2N7000, Q8 2N7000, Q9 2N7000, SW1 A3..A0 B3..B0, SW2 SUB EO AI AO BI BA AB OI, SW3 IO II PCE PCL FI HLT - -, SW4 DATA (closed = 1 on the bus), SW5 CLK, SW6 RST

Commit message: Coupon, ALU and hub PCBs routed and DRC clean; fab outputs
pcb.py: power pre-routed as per-column rails from the tile geometry, fixed in
the DSN so the router cannot move them; GND pour before routing; DRC-verified
ground stitching; inset outline while routing; retries until zero unconnected.
Coupon 112x94, ALU 156x214, hub 130x98 mm. docs/bring-up.md and docs/order-1.md.

Co-Authored-By: Claude Fable 5.1 <noreply@anthropic.com>
Claude-Session: https://claude.ai/code/session_019vcbW37ERmrjZaWq55Er3J
Parts:
- H1, H2, H3, H4: footprint MountingHole:MountingHole_3.2mm_M3 -> MountingHole:MountingHole_3.2mm_M3_Pad
- Q1, Q10, Q11, Q12, Q13, Q14, Q15, Q16, Q17, Q18, Q19, Q2, Q20, Q21, Q22, Q23, Q24, Q25, Q26, Q27, Q28, Q29, Q3, Q30, Q31, Q32, Q33, Q34, Q35, Q36, Q37, Q38, Q39, Q4, Q40, Q41, Q42, Q43, Q44, Q45, Q46, Q47, Q48, Q49, Q5, Q50, Q6, Q7, Q8, Q9: footprint Package_TO_SOT_THT:TO-92_Inline -> Package_TO_SOT_THT:TO-92_Inline_Wide
- R113, R114, R115, R116, R117, R118, R119, R120: value 1k -> 47k
- R71, R72, R73, R74, R75, R76, R77, R78: value 47k -> 1k
Connections:
- net A0: now also Q4.2 (G); no longer Q16.2 (G)
- net A1: now also Q3.2 (G); no longer Q15.2 (G)
- net A2: now also Q2.2 (G); no longer Q14.2 (G)
- net A3: now also Q1.2 (G); no longer Q13.2 (G)
- net AB: now also Q35.2 (G); no longer Q43.2 (G)
- net AI: now also Q31.2 (G); no longer Q39.2 (G)
- net AO: now also Q32.2 (G); no longer Q40.2 (G)
- net B0: now also Q8.2 (G); no longer Q20.2 (G)
- net B1: now also Q7.2 (G); no longer Q19.2 (G)
- net B2: now also Q6.2 (G); no longer Q18.2 (G)
- net B3: now also Q5.2 (G); no longer Q17.2 (G)
- net BA: now also Q34.2 (G); no longer Q42.2 (G)
- net BI: now also Q33.2 (G); no longer Q41.2 (G)
- net BUS0#: now also Q43.2 (G); no longer Q1.2 (G)
- net BUS1#: now also Q44.2 (G); no longer Q2.2 (G)
- net BUS2#: now also Q45.2 (G); no longer Q3.2 (G)
- net BUS3#: now also Q46.2 (G); no longer Q4.2 (G)
- net CF: now also Q25.2 (G); no longer Q33.2 (G)
- net CLK: now also Q27.2 (G); no longer Q35.2 (G)
- net CLK_N: now also Q47.2 (G); no longer Q5.2 (G)
- net CLK_S1: now also Q47.3 (D), Q48.2 (G), R117.2; no longer Q5.3 (D), Q6.2 (G), R75.2
- net CLK_S2: now also Q48.3 (D), R118.2; no longer Q6.3 (D), R76.2
- net D0: now also Q43.3 (D), R113.2; no longer Q1.3 (D), R71.2
- net D1: now also Q44.3 (D), R114.2; no longer Q2.3 (D), R72.2
- net D2: now also Q45.3 (D), R115.2; no longer Q3.3 (D), R73.2
- net D3: now also Q46.3 (D), R116.2; no longer Q4.3 (D), R74.2
- net EO: now also Q30.2 (G); no longer Q38.2 (G)
- net FI: now also Q41.2 (G); no longer Q49.2 (G)
- net HLT: now also Q42.2 (G); no longer Q50.2 (G)
- net II: now also Q38.2 (G); no longer Q46.2 (G)
- net IO: now also Q37.2 (G); no longer Q45.2 (G)
- net M0: now also Q24.2 (G); no longer Q32.2 (G)
- net M1: now also Q23.2 (G); no longer Q31.2 (G)
- net M2: now also Q22.2 (G); no longer Q30.2 (G)
- net M3: now also Q21.2 (G); no longer Q29.2 (G)
- net M4: now also Q20.2 (G); no longer Q28.2 (G)
- net M5: now also Q19.2 (G); no longer Q27.2 (G)
- net M6: now also Q18.2 (G); no longer Q26.2 (G)
- net M7: now also Q17.2 (G); no longer Q25.2 (G)
- net OI: now also Q36.2 (G); no longer Q44.2 (G)
- net PC0: now also Q16.2 (G); no longer Q24.2 (G)
- net PC1: now also Q15.2 (G); no longer Q23.2 (G)
- net PC2: now also Q14.2 (G); no longer Q22.2 (G)
- net PC3: now also Q13.2 (G); no longer Q21.2 (G)
- net PCE: now also Q39.2 (G); no longer Q47.2 (G)
- net PCL: now also Q40.2 (G); no longer Q48.2 (G)
- net RST: now also Q28.2 (G); no longer Q36.2 (G)
- net RST_N: now also Q49.2 (G); no longer Q7.2 (G)
- net RST_S1: now also Q49.3 (D), Q50.2 (G), R119.2; no longer Q7.3 (D), Q8.2 (G), R77.2
- net RST_S2: now also Q50.3 (D), R120.2; no longer Q8.3 (D), R78.2
- net SUB: now also Q29.2 (G); no longer Q37.2 (G)
- net ZF: now also Q26.2 (G); no longer Q34.2 (G)
- net at D28.1 (K): now also Q26.3 (D); no longer Q34.3 (D)
- net at D28.2 (A): now also R96.2; no longer R104.2
- net at Q14.3 (D): now also D16.1 (K); no longer D8.1 (K)
- net at Q32.3 (D): now also D34.1 (K); no longer D26.1 (K)
- net at R84.2: now also D16.2 (A); no longer D8.2 (A)
- net at R83.2: now also D15.2 (A); no longer D7.2 (A)
- net at Q37.3 (D): now also D39.1 (K); no longer D31.1 (K)
- net at D10.2 (A): now also R78.2; no longer R86.2
- net at D5.1 (K): now also Q3.3 (D); no longer Q11.3 (D)
- net at D38.1 (K): now also Q36.3 (D); no longer Q44.3 (D)
- net at D38.2 (A): now also R106.2; no longer R114.2
- net at D9.2 (A): now also R77.2; no longer R85.2
- net at D10.1 (K): now also Q8.3 (D); no longer Q16.3 (D)
- net at D39.2 (A): now also R107.2; no longer R115.2
- net at Q12.3 (D): now also D14.1 (K); no longer D6.1 (K)
- net at R82.2: now also D14.2 (A); no longer D6.2 (A)
- net at D9.1 (K): now also Q7.3 (D); no longer Q15.3 (D)
- net at Q23.3 (D): now also D25.1 (K); no longer D17.1 (K)
- net at D13.2 (A): now also R81.2; no longer R89.2
- net at Q39.3 (D): now also D41.1 (K); no longer D33.1 (K)
- net at R109.2: now also D41.2 (A); no longer D33.2 (A)
- net at D34.2 (A): now also R102.2; no longer R110.2
- net at D42.1 (K): now also Q40.3 (D); no longer Q48.3 (D)
- net at Q41.3 (D): now also D43.1 (K); no longer D35.1 (K)
- net at Q22.3 (D): now also D24.1 (K); no longer D16.1 (K)
- net at Q30.3 (D): now also D32.1 (K); no longer D24.1 (K)
- net at R90.2: now also D22.2 (A); no longer D14.2 (A)
- net at D42.2 (A): now also R110.2; no longer R118.2
- net at D44.1 (K): now also Q42.3 (D); no longer Q50.3 (D)
- net at D22.1 (K): now also Q20.3 (D); no longer Q28.3 (D)
- net at R98.2: now also D30.2 (A); no longer D22.2 (A)
- net at R112.2: now also D44.2 (A); no longer D36.2 (A)
- net at R97.2: now also D29.2 (A); no longer D21.2 (A)
- net at Q10.3 (D): now also D12.1 (K); no longer D4.1 (K)
- net at R93.2: now also D25.2 (A); no longer D17.2 (A)
- net at D19.2 (A): now also R87.2; no longer R95.2
- net at D37.2 (A): now also R105.2; no longer R113.2
- net at D27.1 (K): now also Q25.3 (D); no longer Q33.3 (D)
- net at D27.2 (A): now also R95.2; no longer R103.2
- net at D23.2 (A): now also R91.2; no longer R99.2
- net at D40.1 (K): now also Q38.3 (D); no longer Q46.3 (D)
- net at D40.2 (A): now also R108.2; no longer R116.2
- net at Q18.3 (D): now also D20.1 (K); no longer D12.1 (K)
- net at R94.2: now also D26.2 (A); no longer D18.2 (A)
- net at R92.2: now also D24.2 (A); no longer D16.2 (A)
- net at Q27.3 (D): now also D29.1 (K); no longer D21.1 (K)
- net at D5.2 (A): now also R73.2; no longer R81.2
- net at R100.2: now also D32.2 (A); no longer D24.2 (A)
- net at D3.1 (K): now also Q1.3 (D); no longer Q9.3 (D)
- net at R79.2: now also D11.2 (A); no longer D3.2 (A)
- net at D30.1 (K): now also Q28.3 (D); no longer Q36.3 (D)
- net at D20.2 (A): now also R88.2; no longer R96.2
- net at D11.1 (K): now also Q9.3 (D); no longer Q17.3 (D)
- net at D13.1 (K): now also Q11.3 (D); no longer Q19.3 (D)
- net at Q31.3 (D): now also D33.1 (K); no longer D25.1 (K)
- net at R101.2: now also D33.2 (A); no longer D25.2 (A)
- net at D12.2 (A): now also R80.2; no longer R88.2
- net at D4.2 (A): now also R72.2; no longer R80.2
- net at D31.2 (A): now also R99.2; no longer R107.2
- net at D15.1 (K): now also Q13.3 (D); no longer Q21.3 (D)
- net at R111.2: now also D43.2 (A); no longer D35.2 (A)
- net at D19.1 (K): now also Q17.3 (D); no longer Q25.3 (D)
- net at D18.1 (K): now also Q16.3 (D); no longer Q24.3 (D)
- net at Q35.3 (D): now also D37.1 (K); no longer D29.1 (K)
- net at D7.1 (K): now also Q5.3 (D); no longer Q13.3 (D)
- net at Q29.3 (D): now also D31.1 (K); no longer D23.1 (K)
- net at D36.1 (K): now also Q34.3 (D); no longer Q42.3 (D)
- new net: D7.2 (A), R75.2
- new net: D3.2 (A), R71.2
- new net: D26.1 (K), Q24.3 (D)
- new net: D18.2 (A), R86.2
- new net: D4.1 (K), Q2.3 (D)
- new net: D8.1 (K), Q6.3 (D)
- new net: D23.1 (K), Q21.3 (D)
- new net: D17.1 (K), Q15.3 (D)
- new net: D17.2 (A), R85.2
- new net: D6.1 (K), Q4.3 (D)
- new net: D6.2 (A), R74.2
- new net: D35.1 (K), Q33.3 (D)
- new net: D35.2 (A), R103.2
- new net: D21.1 (K), Q19.3 (D)
- new net: D21.2 (A), R89.2
- new net: D8.2 (A), R76.2
- new net: D36.2 (A), R104.2

Commit message: Panel: input port and control switches for the new lines; hub regenerated
INP gates the four data switches onto the bus through open-drain drivers
(IN instruction). The third control switch row carries MI, MO, WRL, WRH,
ONE, F0, F1 and INP with an LED per line. 80 transistors, 56 LEDs.

Co-Authored-By: Claude Fable 5.1 <noreply@anthropic.com>
Claude-Session: https://claude.ai/code/session_019vcbW37ERmrjZaWq55Er3J
Parts:
- removed J1: BUS, Connector_IDC:IDC-Header_2x25_P2.54mm_Vertical, symbol Connector_Generic:Conn_02x25_Odd_Even
- removed SW4: DATA (closed = 1 on the bus), Button_Switch_THT:SW_DIP_SPSTx04_Slide_9.78x12.34mm_W7.62mm_P2.54mm, symbol Switch:SW_DIP_x04
- removed SW5: CLK, Button_Switch_THT:SW_PUSH_6mm, symbol Switch:SW_Push
- added D45, D46, D47, D48, D49, D50, D51, D52, D53, D54, D55, D56, D57, D58: LED, LED_THT:LED_D3.0mm, symbol Device:LED
- added J1: BUS, Connector_IDC:IDC-Header_2x32_P2.54mm_Vertical, symbol Connector_Generic:Conn_02x32_Odd_Even
- added Q51, Q52, Q53, Q54, Q55, Q56, Q57, Q58, Q59, Q60, Q61, Q62, Q63, Q64, Q65, Q66, Q67, Q68, Q69, Q70, Q71, Q72, Q73, Q74, Q75, Q76, Q77, Q78, Q79, Q80: 2N7000, Package_TO_SOT_THT:TO-92_Inline_Wide, symbol Transistor_FET:2N7000
- added R121, R122, R123, R124, R125, R126, R127, R128, R129, R130, R131, R132, R133, R134, R135, R136, R137, R138, R139, R140, R141, R142, R143, R144, R145, R146, R147, R148, R149, R150: 1k, Resistor_THT:R_Axial_DIN0207_L6.3mm_D2.5mm_P5.08mm_Vertical, symbol Device:R
- added R151, R152, R153, R154, R155, R156, R157, R158, R159, R160, R161, R162, R163, R164, R165, R166: 47k, Resistor_THT:R_Axial_DIN0207_L6.3mm_D2.5mm_P5.08mm_Vertical, symbol Device:R
- added SW4: MI MO WRL WRH ONE F0 F1 INP, Button_Switch_THT:SW_DIP_SPSTx08_Slide_9.78x22.5mm_W7.62mm_P2.54mm, symbol Switch:SW_DIP_x08
- added SW5: DATA (input port, read by IN), Button_Switch_THT:SW_DIP_SPSTx04_Slide_9.78x12.34mm_W7.62mm_P2.54mm, symbol Switch:SW_DIP_x04
- added SW7: RST, Button_Switch_THT:SW_PUSH_6mm, symbol Switch:SW_Push
- R113, R114, R115, R116, R117, R118, R119, R120: value 47k -> 1k
- R24, R29: value 220k -> 10k
- R25, R30: value 100k -> 10k
- R26, R31, R33, R34, R35, R36, R37, R41, R42, R46: value 1Meg -> 10k
- R38, R43: value 1Meg -> 220k
- R39, R44: value 1Meg -> 100k
- R71, R72, R73, R74, R75, R76, R77, R78, R79, R80, R81, R82, R83, R84, R85, R86, R87, R88, R89, R90, R91, R92, R93, R94: value 1k -> 1Meg
- SW2: value SUB EO AI AO BI BA AB OI -> SUB EO AI AO BI BO BA AB
- SW3: value IO II PCE PCL FI HLT - - -> OI IO II PCE PCL FI HLT MAI
- SW6: value RST -> CLK
Connections:
- net +5V: now also J1.1 (Pin_1), J1.2 (Pin_2), J1.63 (Pin_63), R121.1, R122.1, R123.1, R124.1, R125.1, R126.1, R127.1, R128.1, R129.1, R130.1, R131.1, R132.1, R133.1, R134.1, R135.1, R136.1, R137.1, R138.1, R139.1, R140.1, R141.1, R142.1, R143.1, R144.1, R145.1, R146.1, R147.1, R148.1, R149.1, R150.1, R151.1, R152.1, R153.1, R154.1, R155.1, R156.1, R157.1, R158.1, R159.1, R160.1, R161.1, R162.1, R163.1, R164.1, R165.1, R166.1, SW4.1, SW4.2, SW4.3, SW4.4, SW4.5, SW4.6, SW4.7, SW4.8, SW5.1, SW5.2, SW5.3, SW5.4, SW7.1; no longer R71.1, R72.1, R73.1, R74.1, R75.1, R76.1, R77.1, R78.1, R79.1, R80.1, R81.1, R82.1, R83.1, R84.1, R85.1, R86.1, R87.1, R88.1, R89.1, R90.1, R91.1, R92.1, R93.1, R94.1
- net A0: now also R47.1, J1.13 (Pin_13); no longer R33.1
- net A1: now also R48.1, J1.14 (Pin_14); no longer R34.1
- net A2: now also R49.1, J1.15 (Pin_15); no longer R35.1
- net A3: now also R50.1, J1.16 (Pin_16); no longer R36.1
- net AB: now also Q40.2 (G), R16.2, R62.1, J1.46 (Pin_46); no longer Q35.2 (G), R15.2, R47.1
- net AI: now also Q35.2 (G), R57.1, J1.41 (Pin_41); no longer Q31.2 (G), R43.1
- net AO: now also Q36.2 (G), R58.1, J1.42 (Pin_42); no longer Q32.2 (G), R44.1
- net B0: now also R51.1, J1.17 (Pin_17); no longer R37.1
- net B1: now also R52.1, J1.18 (Pin_18); no longer R38.1
- net B2: now also R53.1, J1.19 (Pin_19); no longer R39.1
- net B3: now also R54.1, J1.20 (Pin_20); no longer R40.1
- net BA: now also Q39.2 (G), R15.2, R61.1, J1.45 (Pin_45); no longer Q34.2 (G), R14.2, R46.1
- net BI: now also Q37.2 (G), R59.1, J1.43 (Pin_43); no longer Q33.2 (G), R45.1
- net BUS0#: now also J1.9 (Pin_9), Q57.2 (G), Q64.3 (D); no longer Q43.2 (G)
- net BUS1#: now also J1.10 (Pin_10), Q58.2 (G), Q68.3 (D); no longer Q44.2 (G)
- net BUS2#: now also J1.11 (Pin_11), Q59.2 (G), Q72.3 (D); no longer Q45.2 (G)
- net BUS3#: now also J1.12 (Pin_12), Q60.2 (G), Q76.3 (D); no longer Q46.2 (G)
- net CF: now also Q13.2 (G), R91.1, J1.37 (Pin_37); no longer Q25.2 (G), R67.1
- net CLK: now also Q15.2 (G), R93.1, J1.5 (Pin_5); no longer Q27.2 (G), R69.1
- net CLK_N: now also R39.2, R40.2, Q77.2 (G); no longer Q47.2 (G), R25.2, R26.2
- net CLK_S1: now also Q77.3 (D), Q78.2 (G), R163.2; no longer Q47.3 (D), Q48.2 (G), R117.2
- net CLK_S2: now also R40.1, R41.1, Q78.3 (D), R164.2; no longer Q48.3 (D), R118.2, R26.1, R27.1
- net D0: now also Q57.3 (D), R151.2; no longer Q43.3 (D), R113.2
- net D1: now also Q58.3 (D), R152.2; no longer Q44.3 (D), R114.2
- net D2: now also Q59.3 (D), R153.2; no longer Q45.3 (D), R115.2
- net D3: now also Q60.3 (D), R154.2; no longer Q46.3 (D), R116.2
- net EO: now also Q34.2 (G), R56.1, J1.40 (Pin_40); no longer Q30.2 (G), R42.1
- net FI: now also Q46.2 (G), R22.2, R68.1, J1.52 (Pin_52); no longer Q41.2 (G), R21.2, R53.1
- net GND: now also R35.1, R36.1, R71.2, R72.2, R73.2, R74.2, R75.2, R76.2, R77.2, R78.2, R79.2, R80.2, R81.2, R82.2, R83.2, R84.2, R85.2, R86.2, R87.2, R88.2, R89.2, R90.2, R91.2, R92.2, R93.2, R94.2, J1.3 (Pin_3), J1.4 (Pin_4), J1.6 (Pin_6), J1.64 (Pin_64), J1.8 (Pin_8), Q51.1 (S), Q52.1 (S), Q53.1 (S), Q54.1 (S), Q55.1 (S), Q56.1 (S), Q57.1 (S), Q58.1 (S), Q59.1 (S), Q60.1 (S), Q62.1 (S), Q63.1 (S), Q64.1 (S), Q66.1 (S), Q67.1 (S), Q68.1 (S), Q70.1 (S), Q71.1 (S), Q72.1 (S), Q74.1 (S), Q75.1 (S), Q76.1 (S), Q77.1 (S), Q78.1 (S), Q79.1 (S), Q80.1 (S), SW5.5, SW5.6; no longer R24.2, R29.2, R33.2, R34.2, R35.2, R36.2, R37.2, R39.2, R40.2, R41.2, R42.2, R44.2, R45.2, R46.2
- net HLT: now also Q47.2 (G), R23.2, R69.1, J1.53 (Pin_53); no longer Q42.2 (G), R22.2, R54.1
- net II: now also Q43.2 (G), R19.2, R65.1, J1.49 (Pin_49); no longer Q38.2 (G), R18.2, R50.1
- net IO: now also Q42.2 (G), R18.2, R64.1, J1.48 (Pin_48); no longer Q37.2 (G), R17.2, R49.1
- net M0: now also Q32.2 (G), J1.29 (Pin_29); no longer Q24.2 (G), R59.1
- net M1: now also Q31.2 (G), J1.30 (Pin_30); no longer Q23.2 (G), R60.1
- net M2: now also Q30.2 (G), J1.31 (Pin_31); no longer Q22.2 (G), R61.1
- net M3: now also Q29.2 (G), J1.32 (Pin_32); no longer Q21.2 (G), R62.1
- net M4: now also Q28.2 (G), J1.33 (Pin_33); no longer Q20.2 (G), R63.1
- net M5: now also Q27.2 (G), J1.34 (Pin_34); no longer Q19.2 (G), R64.1
- net M6: now also Q26.2 (G), J1.35 (Pin_35); no longer Q18.2 (G), R65.1
- net M7: now also Q25.2 (G), J1.36 (Pin_36); no longer Q17.2 (G), R66.1
- net OI: now also Q41.2 (G), R17.2, R63.1, J1.47 (Pin_47); no longer Q36.2 (G), R16.2, R48.1
- net PC0: now also Q24.2 (G), R83.1, J1.21 (Pin_21); no longer Q16.2 (G), R55.1
- net PC1: now also Q23.2 (G), R84.1, J1.22 (Pin_22); no longer Q15.2 (G), R56.1
- net PC2: now also Q22.2 (G), R85.1, J1.23 (Pin_23); no longer Q14.2 (G), R57.1
- net PC3: now also Q21.2 (G), R86.1, J1.24 (Pin_24); no longer Q13.2 (G), R58.1
- net PCE: now also Q44.2 (G), R20.2, R66.1, J1.50 (Pin_50); no longer Q39.2 (G), R19.2, R51.1
- net PCL: now also Q45.2 (G), R21.2, R67.1, J1.51 (Pin_51); no longer Q40.2 (G), R20.2, R52.1
- net RST: now also Q16.2 (G), R94.1, J1.7 (Pin_7); no longer Q28.2 (G), R70.1
- net RST_N: now also R44.2, R45.2, Q79.2 (G); no longer Q49.2 (G), R30.2, R31.2
- net RST_S1: now also Q79.3 (D), Q80.2 (G), R165.2; no longer Q49.3 (D), Q50.2 (G), R119.2
- net RST_S2: now also R45.1, R46.1, Q80.3 (D), R166.2; no longer Q50.3 (D), R120.2, R31.1, R32.1
- net SUB: now also Q33.2 (G), R55.1, J1.39 (Pin_39); no longer Q29.2 (G), R41.1
- net ZF: now also Q14.2 (G), R92.1, J1.38 (Pin_38); no longer Q26.2 (G), R68.1
- net at D21.2 (A): now also R113.2; no longer R89.2
- net at D36.2 (A): now also R128.2; no longer R104.2
- net at D26.2 (A): now also R118.2; no longer R94.2
- net at D17.2 (A): now also R109.2; no longer R85.2
- net at D35.2 (A): now also R127.2; no longer R103.2
- net at R106.2: now also D14.2 (A); no longer D38.2 (A)
- net at D10.2 (A): now also R102.2; no longer R78.2
- net at D4.2 (A): now also R96.2; no longer R72.2
- net at D37.2 (A): now also R129.2; no longer R105.2
- net at D15.2 (A): now also R107.2; no longer R83.2
- net at R101.2: now also D9.2 (A); no longer D33.2 (A)
- net at D12.2 (A): now also R104.2; no longer R80.2
- net at D13.2 (A): now also R105.2; no longer R81.2
- net at D7.2 (A): now also R99.2; no longer R75.2
- net at D30.2 (A): now also R122.2; no longer R98.2
- net at SW3.10: now also R23.1
- net at SW3.9: now also R24.1
- net at D5.2 (A): now also R97.2; no longer R73.2
- net at R111.2: now also D19.2 (A); no longer D43.2 (A)
- net at D23.2 (A): now also R115.2; no longer R91.2
- net at D11.2 (A): now also R103.2; no longer R79.2
- net at D41.2 (A): now also R133.2; no longer R109.2
- net at D1.2 (A): now also R41.2; no longer R27.2
- net at D2.2 (A): now also R46.2; no longer R32.2
- net at R28.1: now also SW4.13; no longer SW6.2
- net at R110.2: now also D18.2 (A); no longer D42.2 (A)
- net at D31.2 (A): now also R123.2; no longer R99.2
- net at D8.2 (A): now also R100.2; no longer R76.2
- net at D24.2 (A): now also R116.2; no longer R92.2
- net at D25.2 (A): now also R117.2; no longer R93.2
- net at D28.2 (A): now also R120.2; no longer R96.2
- net at D6.2 (A): now also R98.2; no longer R74.2
- net at D32.2 (A): now also R124.2; no longer R100.2
- net at D34.2 (A): now also R126.2; no longer R102.2
- net at D16.2 (A): now also R108.2; no longer R84.2
- net at D3.2 (A): now also R95.2; no longer R71.2
- net at D29.2 (A): now also R121.2; no longer R97.2
- net at R112.2: now also D20.2 (A); no longer D44.2 (A)
- net at D27.2 (A): now also R119.2; no longer R95.2
- net at D40.2 (A): now also R132.2; no longer R108.2
- net at D22.2 (A): now also R114.2; no longer R90.2
- net at D39.2 (A): now also R131.2; no longer R107.2
- new net: D46.1 (K), Q44.3 (D)
- new net: D53.1 (K), Q51.3 (D)
- new net: Q61.1 (S), Q62.3 (D)
- new net: R31.1, SW4.10
- new net: R30.1, SW4.11
- new net: R29.1, SW4.12
- new net: R27.1, SW4.14
- new net: R26.1, SW4.15
- new net: R25.1, SW4.16
- new net: R32.1, SW4.9
- new net: D49.2 (A), R141.2
- new net: D49.1 (K), Q47.3 (D)
- new net: R42.1, SW7.2
- new net: D57.1 (K), Q55.3 (D)
- new net: D46.2 (A), R138.2
- new net: D48.2 (A), R140.2
- new net: D47.2 (A), R139.2
- new net: D53.2 (A), R145.2
- new net: C4.1, R42.2, R43.1, R44.1
- new net: D45.2 (A), R137.2
- new net: C3.1, R37.2, R38.1, R39.1
- new net: D47.1 (K), Q45.3 (D)
- new net: D44.2 (A), R136.2
- new net: D56.2 (A), R148.2
- new net: D33.2 (A), R125.2
- new net: D38.2 (A), R130.2
- new net: R33.1, SW5.8
- new net: D58.2 (A), R150.2
- new net: D51.1 (K), Q49.3 (D)
- new net: R34.1, SW5.7
- new net: D45.1 (K), Q43.3 (D)
- new net: Q65.1 (S), Q66.3 (D)
- new net: D54.1 (K), Q52.3 (D)
- new net: D54.2 (A), R146.2
- new net: D57.2 (A), R149.2
- new net: D50.1 (K), Q48.3 (D)
- new net: D50.2 (A), R142.2
- new net: D55.1 (K), Q53.3 (D)
- new net: D43.2 (A), R135.2
- new net: D51.2 (A), R143.2
- new net: R37.1, SW6.2
- new net: D48.1 (K), Q46.3 (D)
- new net: D55.2 (A), R147.2
- new net: D58.1 (K), Q56.3 (D)
- new net: Q73.1 (S), Q74.3 (D)
- new net: Q69.1 (S), Q70.3 (D)
- new net: D52.1 (K), Q50.3 (D)
- new net: D52.2 (A), R144.2
- new net: D56.1 (K), Q54.3 (D)
- new net: D42.2 (A), R134.2
- new net BO: J1.44 (Pin_44), Q38.2 (G), R14.2, R60.1
- new net F0: J1.60 (Pin_60), Q54.2 (G), R30.2, R76.1
- new net F1: J1.61 (Pin_61), Q55.2 (G), R31.2, R77.1
- new net IN0: Q63.3 (D), Q64.2 (G), R156.2
- new net IN0N: Q61.3 (D), Q63.2 (G), R155.2
- new net IN1: Q67.3 (D), Q68.2 (G), R158.2
- new net IN1N: Q65.3 (D), Q67.2 (G), R157.2
- new net IN2: Q71.3 (D), Q72.2 (G), R160.2
- new net IN2N: Q69.3 (D), Q71.2 (G), R159.2
- new net IN3: Q75.3 (D), Q76.2 (G), R162.2
- new net IN3N: Q73.3 (D), Q75.2 (G), R161.2
- new net INP: J1.62 (Pin_62), Q56.2 (G), Q61.2 (G), Q65.2 (G), Q69.2 (G), Q73.2 (G), R32.2, R78.1
- new net MAI: J1.54 (Pin_54), Q48.2 (G), R24.2, R70.1
- new net MI: J1.55 (Pin_55), Q49.2 (G), R25.2, R71.1
- new net MO: J1.56 (Pin_56), Q50.2 (G), R26.2, R72.1
- new net ONE: J1.59 (Pin_59), Q53.2 (G), R29.2, R75.1
- new net PC4: J1.25 (Pin_25), Q20.2 (G), R87.1
- new net PC5: J1.26 (Pin_26), Q19.2 (G), R88.1
- new net PC6: J1.27 (Pin_27), Q18.2 (G), R89.1
- new net PC7: J1.28 (Pin_28), Q17.2 (G), R90.1
- new net SW0: Q62.2 (G), R33.2, R79.1
- new net SW1: Q66.2 (G), R34.2, R80.1
- new net SW2: Q70.2 (G), R35.2, R81.1
- new net SW3: Q74.2 (G), R36.2, R82.1
- new net WRH: J1.58 (Pin_58), Q52.2 (G), R28.2, R74.1
- new net WRL: J1.57 (Pin_57), Q51.2 (G), R27.2, R73.1
- no-connect marks 2 -> 0
Other:
- note added: "80 transistors, 56 LEDs. Level switches connect a line to +5V through 10k: a switch left on can never fight a board that pulls the line low, it only adds a 1 where nothing else drives. Every switched or observed line has a 1Meg pull-down so it reads 0 when no board drives it. The DATA switches are the input port: a closed switch is a 1, and while INP=1 the four bits are driven onto the bus (open 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"
- note added: "INPUT PORT: when INP=1 each closed DATA switch (SW_i=1) pulls BUS_i# low, i.e. puts a 1 on the bus. NAND(INP, SW_i) -> inverter -> open-drain transistor, the same driver every board uses"
- note added: "LED_BO"
- note added: "LED_F0"
- note added: "LED_F1"
- note added: "LED_INP"
- note added: "LED_MAI"
- note added: "LED_MI"
- note added: "LED_MO"
- note added: "LED_ONE"
- note added: "LED_PC4"
- note added: "LED_PC5"
- note added: "LED_PC6"
- note added: "LED_PC7"
- note added: "LED_WRH"
- note added: "LED_WRL"
- note removed: "50 transistors, 42 LEDs. Level switches connect a line to +5V through 10k: a switch left on can never fight a board that pulls the line low, it only adds a 1 where nothing else drives. Every switched or observed line has a 1Meg pull-down so it reads 0 when no board drives it. DATA switches pull BUS_i# to GND directly (that is what an open-drain driver does), so closed = 1 on the bus. CLK and RST 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"
