File: boards/07-hub/hub.kicad_sch (KiCad schematic)
At the start: 28 parts, among them J1 USB_B, J2 BUS, J3 BUS, J4 BUS, J5 BUS, J6 BUS, J7 BUS, J8 BUS, J9 BUS

Commit message: Coupon, ALU and hub PCBs routed and DRC clean; fab outputs
pcb.py: power pre-routed as per-column rails from the tile geometry, fixed in
the DSN so the router cannot move them; GND pour before routing; DRC-verified
ground stitching; inset outline while routing; retries until zero unconnected.
Coupon 112x94, ALU 156x214, hub 130x98 mm. docs/bring-up.md and docs/order-1.md.

Co-Authored-By: Claude Fable 5.1 <noreply@anthropic.com>
Claude-Session: https://claude.ai/code/session_019vcbW37ERmrjZaWq55Er3J
Parts:
- H1, H2, H3, H4: footprint MountingHole:MountingHole_3.2mm_M3 -> MountingHole:MountingHole_3.2mm_M3_Pad

Commit message: Panel: input port and control switches for the new lines; hub regenerated
INP gates the four data switches onto the bus through open-drain drivers
(IN instruction). The third control switch row carries MI, MO, WRL, WRH,
ONE, F0, F1 and INP with an LED per line. 80 transistors, 56 LEDs.

Co-Authored-By: Claude Fable 5.1 <noreply@anthropic.com>
Claude-Session: https://claude.ai/code/session_019vcbW37ERmrjZaWq55Er3J
Parts:
- removed J2, J3, J4, J5, J6, J7, J8, J9: BUS, Connector_IDC:IDC-Header_2x25_P2.54mm_Vertical, symbol Connector_Generic:Conn_02x25_Odd_Even
- added J2, J3, J4, J5, J6, J7, J8, J9: BUS, Connector_IDC:IDC-Header_2x32_P2.54mm_Vertical, symbol Connector_Generic:Conn_02x32_Odd_Even
- added R10, R11, R12, R13, R6, R7, R8, R9: 1Meg, Resistor_THT:R_Axial_DIN0207_L6.3mm_D2.5mm_P5.08mm_Vertical, symbol Device:R
Connections:
- net +5V: now also J2.1 (Pin_1), J2.2 (Pin_2), J2.63 (Pin_63), J3.1 (Pin_1), J3.2 (Pin_2), J3.63 (Pin_63), J4.1 (Pin_1), J4.2 (Pin_2), J4.63 (Pin_63), J5.1 (Pin_1), J5.2 (Pin_2), J5.63 (Pin_63), J6.1 (Pin_1), J6.2 (Pin_2), J6.63 (Pin_63), J7.1 (Pin_1), J7.2 (Pin_2), J7.63 (Pin_63), J8.1 (Pin_1), J8.2 (Pin_2), J8.63 (Pin_63), J9.1 (Pin_1), J9.2 (Pin_2), J9.63 (Pin_63)
- net A0: now also J2.13 (Pin_13), J3.13 (Pin_13), J4.13 (Pin_13), J5.13 (Pin_13), J6.13 (Pin_13), J7.13 (Pin_13), J8.13 (Pin_13), J9.13 (Pin_13)
- net A1: now also J2.14 (Pin_14), J3.14 (Pin_14), J4.14 (Pin_14), J5.14 (Pin_14), J6.14 (Pin_14), J7.14 (Pin_14), J8.14 (Pin_14), J9.14 (Pin_14)
- net A2: now also J2.15 (Pin_15), J3.15 (Pin_15), J4.15 (Pin_15), J5.15 (Pin_15), J6.15 (Pin_15), J7.15 (Pin_15), J8.15 (Pin_15), J9.15 (Pin_15)
- net A3: now also J2.16 (Pin_16), J3.16 (Pin_16), J4.16 (Pin_16), J5.16 (Pin_16), J6.16 (Pin_16), J7.16 (Pin_16), J8.16 (Pin_16), J9.16 (Pin_16)
- net AB: now also J2.46 (Pin_46), J3.46 (Pin_46), J4.46 (Pin_46), J5.46 (Pin_46), J6.46 (Pin_46), J7.46 (Pin_46), J8.46 (Pin_46), J9.46 (Pin_46)
- net AI: now also J2.41 (Pin_41), J3.41 (Pin_41), J4.41 (Pin_41), J5.41 (Pin_41), J6.41 (Pin_41), J7.41 (Pin_41), J8.41 (Pin_41), J9.41 (Pin_41)
- net AO: now also J2.42 (Pin_42), J3.42 (Pin_42), J4.42 (Pin_42), J5.42 (Pin_42), J6.42 (Pin_42), J7.42 (Pin_42), J8.42 (Pin_42), J9.42 (Pin_42)
- net B0: now also J2.17 (Pin_17), J3.17 (Pin_17), J4.17 (Pin_17), J5.17 (Pin_17), J6.17 (Pin_17), J7.17 (Pin_17), J8.17 (Pin_17), J9.17 (Pin_17)
- net B1: now also J2.18 (Pin_18), J3.18 (Pin_18), J4.18 (Pin_18), J5.18 (Pin_18), J6.18 (Pin_18), J7.18 (Pin_18), J8.18 (Pin_18), J9.18 (Pin_18)
- net B2: now also J2.19 (Pin_19), J3.19 (Pin_19), J4.19 (Pin_19), J5.19 (Pin_19), J6.19 (Pin_19), J7.19 (Pin_19), J8.19 (Pin_19), J9.19 (Pin_19)
- net B3: now also J2.20 (Pin_20), J3.20 (Pin_20), J4.20 (Pin_20), J5.20 (Pin_20), J6.20 (Pin_20), J7.20 (Pin_20), J8.20 (Pin_20), J9.20 (Pin_20)
- net BA: now also J2.45 (Pin_45), J3.45 (Pin_45), J4.45 (Pin_45), J5.45 (Pin_45), J6.45 (Pin_45), J7.45 (Pin_45), J8.45 (Pin_45), J9.45 (Pin_45)
- net BI: now also J2.43 (Pin_43), J3.43 (Pin_43), J4.43 (Pin_43), J5.43 (Pin_43), J6.43 (Pin_43), J7.43 (Pin_43), J8.43 (Pin_43), J9.43 (Pin_43)
- net BUS0#: now also J2.9 (Pin_9), J3.9 (Pin_9), J4.9 (Pin_9), J5.9 (Pin_9), J6.9 (Pin_9), J7.9 (Pin_9), J8.9 (Pin_9), J9.9 (Pin_9)
- net BUS1#: now also J2.10 (Pin_10), J3.10 (Pin_10), J4.10 (Pin_10), J5.10 (Pin_10), J6.10 (Pin_10), J7.10 (Pin_10), J8.10 (Pin_10), J9.10 (Pin_10)
- net BUS2#: now also J2.11 (Pin_11), J3.11 (Pin_11), J4.11 (Pin_11), J5.11 (Pin_11), J6.11 (Pin_11), J7.11 (Pin_11), J8.11 (Pin_11), J9.11 (Pin_11)
- net BUS3#: now also J2.12 (Pin_12), J3.12 (Pin_12), J4.12 (Pin_12), J5.12 (Pin_12), J6.12 (Pin_12), J7.12 (Pin_12), J8.12 (Pin_12), J9.12 (Pin_12)
- net CF: now also J2.37 (Pin_37), J3.37 (Pin_37), J4.37 (Pin_37), J5.37 (Pin_37), J6.37 (Pin_37), J7.37 (Pin_37), J8.37 (Pin_37), J9.37 (Pin_37)
- net CLK: now also J2.5 (Pin_5), J3.5 (Pin_5), J4.5 (Pin_5), J5.5 (Pin_5), J6.5 (Pin_5), J7.5 (Pin_5), J8.5 (Pin_5), J9.5 (Pin_5)
- net EO: now also J2.40 (Pin_40), J3.40 (Pin_40), J4.40 (Pin_40), J5.40 (Pin_40), J6.40 (Pin_40), J7.40 (Pin_40), J8.40 (Pin_40), J9.40 (Pin_40)
- net FI: now also J2.52 (Pin_52), J3.52 (Pin_52), J4.52 (Pin_52), J5.52 (Pin_52), J6.52 (Pin_52), J7.52 (Pin_52), J8.52 (Pin_52), J9.52 (Pin_52)
- net GND: now also J2.3 (Pin_3), J2.4 (Pin_4), J2.6 (Pin_6), J2.64 (Pin_64), J2.8 (Pin_8), J3.3 (Pin_3), J3.4 (Pin_4), J3.6 (Pin_6), J3.64 (Pin_64), J3.8 (Pin_8), J4.3 (Pin_3), J4.4 (Pin_4), J4.6 (Pin_6), J4.64 (Pin_64), J4.8 (Pin_8), J5.3 (Pin_3), J5.4 (Pin_4), J5.6 (Pin_6), J5.64 (Pin_64), J5.8 (Pin_8), J6.3 (Pin_3), J6.4 (Pin_4), J6.6 (Pin_6), J6.64 (Pin_64), J6.8 (Pin_8), J7.3 (Pin_3), J7.4 (Pin_4), J7.6 (Pin_6), J7.64 (Pin_64), J7.8 (Pin_8), J8.3 (Pin_3), J8.4 (Pin_4), J8.6 (Pin_6), J8.64 (Pin_64), J8.8 (Pin_8), J9.3 (Pin_3), J9.4 (Pin_4), J9.6 (Pin_6), J9.64 (Pin_64), J9.8 (Pin_8), R10.2, R11.2, R12.2, R13.2, R6.2, R7.2, R8.2, R9.2
- net HLT: now also J2.53 (Pin_53), J3.53 (Pin_53), J4.53 (Pin_53), J5.53 (Pin_53), J6.53 (Pin_53), J7.53 (Pin_53), J8.53 (Pin_53), J9.53 (Pin_53)
- net II: now also J2.49 (Pin_49), J3.49 (Pin_49), J4.49 (Pin_49), J5.49 (Pin_49), J6.49 (Pin_49), J7.49 (Pin_49), J8.49 (Pin_49), J9.49 (Pin_49)
- net IO: now also J2.48 (Pin_48), J3.48 (Pin_48), J4.48 (Pin_48), J5.48 (Pin_48), J6.48 (Pin_48), J7.48 (Pin_48), J8.48 (Pin_48), J9.48 (Pin_48)
- net M0: now also J2.29 (Pin_29), J3.29 (Pin_29), J4.29 (Pin_29), J5.29 (Pin_29), J6.29 (Pin_29), J7.29 (Pin_29), J8.29 (Pin_29), J9.29 (Pin_29), R6.1
- net M1: now also J2.30 (Pin_30), J3.30 (Pin_30), J4.30 (Pin_30), J5.30 (Pin_30), J6.30 (Pin_30), J7.30 (Pin_30), J8.30 (Pin_30), J9.30 (Pin_30), R7.1
- net M2: now also J2.31 (Pin_31), J3.31 (Pin_31), J4.31 (Pin_31), J5.31 (Pin_31), J6.31 (Pin_31), J7.31 (Pin_31), J8.31 (Pin_31), J9.31 (Pin_31), R8.1
- net M3: now also J2.32 (Pin_32), J3.32 (Pin_32), J4.32 (Pin_32), J5.32 (Pin_32), J6.32 (Pin_32), J7.32 (Pin_32), J8.32 (Pin_32), J9.32 (Pin_32), R9.1
- net M4: now also J2.33 (Pin_33), J3.33 (Pin_33), J4.33 (Pin_33), J5.33 (Pin_33), J6.33 (Pin_33), J7.33 (Pin_33), J8.33 (Pin_33), J9.33 (Pin_33), R10.1
- net M5: now also J2.34 (Pin_34), J3.34 (Pin_34), J4.34 (Pin_34), J5.34 (Pin_34), J6.34 (Pin_34), J7.34 (Pin_34), J8.34 (Pin_34), J9.34 (Pin_34), R11.1
- net M6: now also J2.35 (Pin_35), J3.35 (Pin_35), J4.35 (Pin_35), J5.35 (Pin_35), J6.35 (Pin_35), J7.35 (Pin_35), J8.35 (Pin_35), J9.35 (Pin_35), R12.1
- net M7: now also J2.36 (Pin_36), J3.36 (Pin_36), J4.36 (Pin_36), J5.36 (Pin_36), J6.36 (Pin_36), J7.36 (Pin_36), J8.36 (Pin_36), J9.36 (Pin_36), R13.1
- net OI: now also J2.47 (Pin_47), J3.47 (Pin_47), J4.47 (Pin_47), J5.47 (Pin_47), J6.47 (Pin_47), J7.47 (Pin_47), J8.47 (Pin_47), J9.47 (Pin_47)
- net PC0: now also J2.21 (Pin_21), J3.21 (Pin_21), J4.21 (Pin_21), J5.21 (Pin_21), J6.21 (Pin_21), J7.21 (Pin_21), J8.21 (Pin_21), J9.21 (Pin_21)
- net PC1: now also J2.22 (Pin_22), J3.22 (Pin_22), J4.22 (Pin_22), J5.22 (Pin_22), J6.22 (Pin_22), J7.22 (Pin_22), J8.22 (Pin_22), J9.22 (Pin_22)
- net PC2: now also J2.23 (Pin_23), J3.23 (Pin_23), J4.23 (Pin_23), J5.23 (Pin_23), J6.23 (Pin_23), J7.23 (Pin_23), J8.23 (Pin_23), J9.23 (Pin_23)
- net PC3: now also J2.24 (Pin_24), J3.24 (Pin_24), J4.24 (Pin_24), J5.24 (Pin_24), J6.24 (Pin_24), J7.24 (Pin_24), J8.24 (Pin_24), J9.24 (Pin_24)
- net PCE: now also J2.50 (Pin_50), J3.50 (Pin_50), J4.50 (Pin_50), J5.50 (Pin_50), J6.50 (Pin_50), J7.50 (Pin_50), J8.50 (Pin_50), J9.50 (Pin_50)
- net PCL: now also J2.51 (Pin_51), J3.51 (Pin_51), J4.51 (Pin_51), J5.51 (Pin_51), J6.51 (Pin_51), J7.51 (Pin_51), J8.51 (Pin_51), J9.51 (Pin_51)
- net RST: now also J2.7 (Pin_7), J3.7 (Pin_7), J4.7 (Pin_7), J5.7 (Pin_7), J6.7 (Pin_7), J7.7 (Pin_7), J8.7 (Pin_7), J9.7 (Pin_7)
- net SUB: now also J2.39 (Pin_39), J3.39 (Pin_39), J4.39 (Pin_39), J5.39 (Pin_39), J6.39 (Pin_39), J7.39 (Pin_39), J8.39 (Pin_39), J9.39 (Pin_39)
- net ZF: now also J2.38 (Pin_38), J3.38 (Pin_38), J4.38 (Pin_38), J5.38 (Pin_38), J6.38 (Pin_38), J7.38 (Pin_38), J8.38 (Pin_38), J9.38 (Pin_38)
- new net BO: J2.44 (Pin_44), J3.44 (Pin_44), J4.44 (Pin_44), J5.44 (Pin_44), J6.44 (Pin_44), J7.44 (Pin_44), J8.44 (Pin_44), J9.44 (Pin_44)
- new net MAI: J2.54 (Pin_54), J3.54 (Pin_54), J4.54 (Pin_54), J5.54 (Pin_54), J6.54 (Pin_54), J7.54 (Pin_54), J8.54 (Pin_54), J9.54 (Pin_54)
- new net MI: J2.55 (Pin_55), J3.55 (Pin_55), J4.55 (Pin_55), J5.55 (Pin_55), J6.55 (Pin_55), J7.55 (Pin_55), J8.55 (Pin_55), J9.55 (Pin_55)
- new net MO: J2.56 (Pin_56), J3.56 (Pin_56), J4.56 (Pin_56), J5.56 (Pin_56), J6.56 (Pin_56), J7.56 (Pin_56), J8.56 (Pin_56), J9.56 (Pin_56)
- new net PC4: J2.25 (Pin_25), J3.25 (Pin_25), J4.25 (Pin_25), J5.25 (Pin_25), J6.25 (Pin_25), J7.25 (Pin_25), J8.25 (Pin_25), J9.25 (Pin_25)
- new net PC5: J2.26 (Pin_26), J3.26 (Pin_26), J4.26 (Pin_26), J5.26 (Pin_26), J6.26 (Pin_26), J7.26 (Pin_26), J8.26 (Pin_26), J9.26 (Pin_26)
- new net PC6: J2.27 (Pin_27), J3.27 (Pin_27), J4.27 (Pin_27), J5.27 (Pin_27), J6.27 (Pin_27), J7.27 (Pin_27), J8.27 (Pin_27), J9.27 (Pin_27)
- new net PC7: J2.28 (Pin_28), J3.28 (Pin_28), J4.28 (Pin_28), J5.28 (Pin_28), J6.28 (Pin_28), J7.28 (Pin_28), J8.28 (Pin_28), J9.28 (Pin_28)
- new net PWH: J2.58 (Pin_58), J3.58 (Pin_58), J4.58 (Pin_58), J5.58 (Pin_58), J6.58 (Pin_58), J7.58 (Pin_58), J8.58 (Pin_58), J9.58 (Pin_58)
- new net PWL: J2.57 (Pin_57), J3.57 (Pin_57), J4.57 (Pin_57), J5.57 (Pin_57), J6.57 (Pin_57), J7.57 (Pin_57), J8.57 (Pin_57), J9.57 (Pin_57)
- new net SP0: J2.59 (Pin_59), J3.59 (Pin_59), J4.59 (Pin_59), J5.59 (Pin_59), J6.59 (Pin_59), J7.59 (Pin_59), J8.59 (Pin_59), J9.59 (Pin_59)
- new net SP1: J2.60 (Pin_60), J3.60 (Pin_60), J4.60 (Pin_60), J5.60 (Pin_60), J6.60 (Pin_60), J7.60 (Pin_60), J8.60 (Pin_60), J9.60 (Pin_60)
- new net SP2: J2.61 (Pin_61), J3.61 (Pin_61), J4.61 (Pin_61), J5.61 (Pin_61), J6.61 (Pin_61), J7.61 (Pin_61), J8.61 (Pin_61), J9.61 (Pin_61)
- new net SP3: J2.62 (Pin_62), J3.62 (Pin_62), J4.62 (Pin_62), J5.62 (Pin_62), J6.62 (Pin_62), J7.62 (Pin_62), J8.62 (Pin_62), J9.62 (Pin_62)
Other:
- note added: "M-line pull-downs (the memory boards only pull high)"
- note added: "NIBBLE BOARD 07 - BUS HUB: power entry, the four bus pull-ups, the eight M-line pull-downs, and one 64-pin header per board"
- note added: "No logic on this board. 8 identical headers wired pin-for-pin; every board plugs in with a straight 64-way ribbon cable (docs/bus-header.md). Power: USB-B 5 V through a 750 mA polyfuse (the USB plug is the power switch). The BUS0#..BUS3# pull-ups (10k) live here and nowhere else. The M0..M7 pull-downs (1Meg) also live here: the program memory boards diode-OR onto the M lines, so an unselected pag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"
- note removed: "NIBBLE BOARD 07 - BUS HUB: power entry, the four bus pull-ups, and one 50-pin header per board"
- note removed: "No logic on this board. 8 identical headers wired pin-for-pin; every board plugs in with a straight 50-way ribbon cable. Power: USB-B 5 V through a 750 mA polyfuse (the USB plug is the power switch). The BUS0#..BUS3# pull-ups (10k) live here and nowhere else. Bulk capacitance for the whole machine, a power LED, and test loops on every bus line for a logic analyser."

Commit message: Hub: power bars and ground stubs pre-routed through every header, test loops moved off the parts
Pins 1-2 (+5V) and 3-4 (GND) of all four headers sit on bars; pin 63 and 64
stubs reach a bottom +5V bar and a ground via, so no header power pin is
left for the autorouter. The test loops overlapped R13 and J9 courtyards.

Co-Authored-By: Claude Fable 5.1 <noreply@anthropic.com>
Claude-Session: https://claude.ai/code/session_019vcbW37ERmrjZaWq55Er3J
Connections:
- net PWH renamed WRH
- net PWL renamed WRL
- net SP0 renamed ONE
- net SP1 renamed F0
- net SP2 renamed F1
- net SP3 renamed INP
