File: boards/02-registers/registers-testbench.kicad_sch (KiCad schematic)
At the start: 21 parts

Commit message: Silkscreen out from under the connectors; testbench parts kept off the board
The renders showed the 'BUS (pin 1 left)' label under every top-edge
header shroud and the clock's name half under its header; the registers
board name ran into a mounting hole, and the registers testbench's four
bus-driver diodes were being loaded onto the board and parked off its
edge. Testbench symbols (refs 9000 and up) are now written with on_board
and in_bom off and pcb.py skips them too. pcb.py --silk replaces a routed
board's silk from the plan without re-routing; ALU and clock done that
way, DRC still zero. The program board's caps move beside the second
header so its label fits below it.

Co-Authored-By: Claude Fable 5.1 <noreply@anthropic.com>
Claude-Session: https://claude.ai/code/session_019vcbW37ERmrjZaWq55Er3J
Parts:
- D9001, D9002, D9003, D9004: now left out of the parts list
