File: boards/04-program/program.kicad_sch (KiCad schematic)
At the start: 353 parts, among them J1 BUS, J2 PAGE0, J3 PAGE1, J4 PAGE2, J5 PAGE3, Q1 2N7000, Q10 2N7000, Q100 2N7000, Q101 2N7000, Q102 2N7000, Q103 2N7000, Q104 2N7000, Q105 2N7000, Q106 2N7000, Q107 2N7000, Q108 2N7000, Q109 2N7000, Q11 2N7000, Q110 2N7000, Q111 2N7000, Q112 2N7000, Q12 2N7000, Q13 2N7000, Q14 2N7000, Q15 2N7000, Q16 2N7000, Q17 2N7000, Q18 2N7000, Q19 2N7000, Q2 2N7000, Q20 2N7000, Q21 2N7000, Q22 2N7000, Q23 2N7000, Q24 2N7000, Q25 2N7000, Q26 2N7000, Q27 2N7000, Q28 2N7000, Q29 2N7000, Q3 2N7000, Q30 2N7000, Q31 2N7000, Q32 2N7000, Q33 2N7000, Q34 2N7000, Q35 2N7000, Q36 2N7000, Q37 2N7000, Q38 2N7000, Q39 2N7000, Q4 2N7000, Q40 2N7000, Q41 2N7000, Q42 2N7000, Q43 2N7000, Q44 2N7000, Q45 2N7000, Q46 2N7000, Q47 2N7000, Q48 2N7000, Q49 2N7000, Q5 2N7000, Q50 2N7000, Q51 2N7000, Q52 2N7000, Q53 2N7000, Q54 2N7000, Q55 2N7000, Q56 2N7000, Q57 2N7000, Q58 2N7000, Q59 2N7000, Q6 2N7000, Q60 2N7000, Q61 2N7000, Q62 2N7000, Q63 2N7000, Q64 2N7000, Q65 2N7000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

Commit message: Program board: second bus header in parallel (D039)
Both 64-way headers carry every line, not only PC and M: unused pins get
passive labels instead of no-connects, so pages daisy-chain and the ribbon
between them is a complete bus. The second header sits at the top right,
the caps and page jumpers move below the headers, and the board grows
12 mm to 216 x 250 so two shrouded sockets and the corner hole fit along
the top edge. ERC clean; the SPICE export is unchanged (connectors do not
export). The column preview draws the second header and hops pages 2 and
up from the previous page instead of running each to the hub.

Co-Authored-By: Claude Fable 5.1 <noreply@anthropic.com>
Claude-Session: https://claude.ai/code/session_019vcbW37ERmrjZaWq55Er3J
Parts:
- removed J2: PAGE0, Connector_PinHeader_2.54mm:PinHeader_1x03_P2.54mm_Vertical, symbol Connector_Generic:Conn_01x03
- added J2: BUS, Connector_IDC:IDC-Header_2x32_P2.54mm_Vertical, symbol Connector_Generic:Conn_02x32_Odd_Even
- added J6: PAGE3, Connector_PinHeader_2.54mm:PinHeader_1x03_P2.54mm_Vertical, symbol Connector_Generic:Conn_01x03
- J3: value PAGE1 -> PAGE0
- J4: value PAGE2 -> PAGE1
- J5: value PAGE3 -> PAGE2
Connections:
- net +5V: now also J2.1 (Pin_1), J2.2 (Pin_2), J2.63 (Pin_63)
- net GND: now also J2.3 (Pin_3), J2.4 (Pin_4), J2.6 (Pin_6), J2.64 (Pin_64), J2.8 (Pin_8)
- net JS0: now also J3.2 (Pin_2)
- net JS1: now also J4.2 (Pin_2); no longer J3.2 (Pin_2)
- net JS2: now also J5.2 (Pin_2); no longer J4.2 (Pin_2)
- net JS3: now also J6.2 (Pin_2); no longer J5.2 (Pin_2)
- net M0: now also J2.29 (Pin_29)
- net M1: now also J2.30 (Pin_30)
- net M2: now also J2.31 (Pin_31)
- net M3: now also J2.32 (Pin_32)
- net M4: now also J2.33 (Pin_33)
- net M5: now also J2.34 (Pin_34)
- net M6: now also J2.35 (Pin_35)
- net M7: now also J2.36 (Pin_36)
- net PC0: now also J2.21 (Pin_21)
- net PC1: now also J2.22 (Pin_22)
- net PC2: now also J2.23 (Pin_23)
- net PC3: now also J2.24 (Pin_24)
- net PC4: now also J3.1 (Pin_1), J2.25 (Pin_25)
- net PC5: now also J4.1 (Pin_1), J2.26 (Pin_26); no longer J3.1 (Pin_1)
- net PC6: now also J5.1 (Pin_1), J2.27 (Pin_27); no longer J4.1 (Pin_1)
- net PC7: now also J2.28 (Pin_28), J6.1 (Pin_1); no longer J5.1 (Pin_1)
- net PN0: now also J3.3 (Pin_3)
- net PN1: now also J4.3 (Pin_3); no longer J3.3 (Pin_3)
- net PN2: now also J5.3 (Pin_3); no longer J4.3 (Pin_3)
- net PN3: now also J6.3 (Pin_3); no longer J5.3 (Pin_3)
- net BUS1#: now reaches J1.10 (Pin_10)
- net BUS1#: now also J2.10 (Pin_10)
- net BUS2#: now reaches J1.11 (Pin_11)
- net BUS2#: now also J2.11 (Pin_11)
- net BUS3#: now reaches J1.12 (Pin_12)
- net BUS3#: now also J2.12 (Pin_12)
- net A0: now reaches J1.13 (Pin_13)
- net A0: now also J2.13 (Pin_13)
- net A1: now reaches J1.14 (Pin_14)
- net A1: now also J2.14 (Pin_14)
- net A2: now reaches J1.15 (Pin_15)
- net A2: now also J2.15 (Pin_15)
- net A3: now reaches J1.16 (Pin_16)
- net A3: now also J2.16 (Pin_16)
- net B0: now reaches J1.17 (Pin_17)
- net B0: now also J2.17 (Pin_17)
- net B1: now reaches J1.18 (Pin_18)
- net B1: now also J2.18 (Pin_18)
- net B2: now reaches J1.19 (Pin_19)
- net B2: now also J2.19 (Pin_19)
- net B3: now reaches J1.20 (Pin_20)
- net B3: now also J2.20 (Pin_20)
- net CF: now reaches J1.37 (Pin_37)
- net CF: now also J2.37 (Pin_37)
- net ZF: now reaches J1.38 (Pin_38)
- net ZF: now also J2.38 (Pin_38)
- net SUB: now reaches J1.39 (Pin_39)
- net SUB: now also J2.39 (Pin_39)
- net EO: now reaches J1.40 (Pin_40)
- net EO: now also J2.40 (Pin_40)
- net AI: now reaches J1.41 (Pin_41)
- net AI: now also J2.41 (Pin_41)
- net AO: now reaches J1.42 (Pin_42)
- net AO: now also J2.42 (Pin_42)
- net BI: now reaches J1.43 (Pin_43)
- net BI: now also J2.43 (Pin_43)
- net BO: now reaches J1.44 (Pin_44)
- net BO: now also J2.44 (Pin_44)
- net BA: now reaches J1.45 (Pin_45)
- net BA: now also J2.45 (Pin_45)
- net AB: now reaches J1.46 (Pin_46)
- net AB: now also J2.46 (Pin_46)
- net OI: now reaches J1.47 (Pin_47)
- net OI: now also J2.47 (Pin_47)
- net IO: now reaches J1.48 (Pin_48)
- net IO: now also J2.48 (Pin_48)
- net II: now reaches J1.49 (Pin_49)
- net II: now also J2.49 (Pin_49)
- net CLK: now reaches J1.5 (Pin_5)
- net CLK: now also J2.5 (Pin_5)
- net PCE: now reaches J1.50 (Pin_50)
- net PCE: now also J2.50 (Pin_50)
- net PCL: now reaches J1.51 (Pin_51)
- net PCL: now also J2.51 (Pin_51)
- net FI: now reaches J1.52 (Pin_52)
- net FI: now also J2.52 (Pin_52)
- net HLT: now reaches J1.53 (Pin_53)
- net HLT: now also J2.53 (Pin_53)
- net MAI: now reaches J1.54 (Pin_54)
- net MAI: now also J2.54 (Pin_54)
- net MI: now reaches J1.55 (Pin_55)
- net MI: now also J2.55 (Pin_55)
- net MO: now reaches J1.56 (Pin_56)
- net MO: now also J2.56 (Pin_56)
- net WRL: now reaches J1.57 (Pin_57)
- net WRL: now also J2.57 (Pin_57)
- net WRH: now reaches J1.58 (Pin_58)
- net WRH: now also J2.58 (Pin_58)
- net ONE: now reaches J1.59 (Pin_59)
- net ONE: now also J2.59 (Pin_59)
- net F0: now reaches J1.60 (Pin_60)
- net F0: now also J2.60 (Pin_60)
- net F1: now reaches J1.61 (Pin_61)
- net F1: now also J2.61 (Pin_61)
- net INP: now reaches J1.62 (Pin_62)
- net INP: now also J2.62 (Pin_62)
- net RST: now reaches J1.7 (Pin_7)
- net RST: now also J2.7 (Pin_7)
- net BUS0#: now reaches J1.9 (Pin_9)
- net BUS0#: now also J2.9 (Pin_9)
- no-connect marks 40 -> 0
Other:
- note added: "112 transistors, 69 resistors, 17 LEDs, 16 DIP-8 switches, 128 diodes. From the bus: PC7..PC0. To the bus: M7..M0 through diodes (the hub holds M low; several pages OR together). Two headers in parallel: hub in, next page out. PC3..0 select the word. PC7..4 are compared with the four PAGE jumpers: each jumper picks PC(4+i) (pins 1-2, page bit = 1) or its inverse (pins 2-3, page bit = 0). A row li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"
- note added: "Both headers carry all 64 lines: the hub's ribbon on the left, the next page's on the right (D039)."
- note removed: "112 transistors, 69 resistors, 17 LEDs, 16 DIP-8 switches, 128 diodes. From the bus header: PC7..PC0. To the bus header: M7..M0 through diodes (the hub holds M low; several pages OR together). PC3..0 select the word. PC7..4 are compared with the four PAGE jumpers: each jumper picks PC(4+i) (pins 1-2, page bit = 1) or its inverse (pins 2-3, page bit = 0). A row line goes high while its word is sel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"
