File: boards/08-memory/memory.kicad_sch (KiCad schematic)
At the start: 1108 parts, among them J1 BUS, Q1 2N7000, Q10 2N7000, Q100 2N7000, Q101 2N7000, Q102 2N7000, Q103 2N7000, Q104 2N7000, Q105 2N7000, Q106 2N7000, Q107 2N7000, Q108 2N7000, Q109 2N7000, Q11 2N7000, Q110 2N7000, Q111 2N7000, Q112 2N7000, Q113 2N7000, Q114 2N7000, Q115 2N7000, Q116 2N7000, Q117 2N7000, Q118 2N7000, Q119 2N7000, Q12 2N7000, Q120 2N7000, Q121 2N7000, Q122 2N7000, Q123 2N7000, Q124 2N7000, Q125 2N7000, Q126 2N7000, Q127 2N7000, Q128 2N7000, Q129 2N7000, Q13 2N7000, Q130 2N7000, Q131 2N7000, Q132 2N7000, Q133 2N7000, Q134 2N7000, Q135 2N7000, Q136 2N7000, Q137 2N7000, Q138 2N7000, Q139 2N7000, Q14 2N7000, Q140 2N7000, Q141 2N7000, Q142 2N7000, Q143 2N7000, Q144 2N7000, Q145 2N7000, Q146 2N7000, Q147 2N7000, Q148 2N7000, Q149 2N7000, Q15 2N7000, Q150 2N7000, Q151 2N7000, Q152 2N7000, Q153 2N7000, Q154 2N7000, Q155 2N7000, Q156 2N7000, Q157 2N7000, Q158 2N7000, Q159 2N7000, Q16 2N7000, Q160 2N7000, Q161 2N7000, Q162 2N7000, Q163 2N7000, Q164 2N7000, Q165 2N7000, Q166 2N7000, Q167 2N7000, Q168 2N7000, Q169 2N7000, Q17 2N7000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

Commit message: Data memory: the write ends at the clock edge (D037)
The write lines were WR = slot AND MI. At the tick boundary the bus data
changes while MI is still dropping through a 22k pull-up, so the write
stacks saw the next tick's bus with the write still on and flipped cells:
TYP passed, the mixed-threshold corner failed (list.asm lost bit 1 on every
read at seed 2), and the new testbench failed 47 of 217 steps at every
corner. Now MIN = NAND(MI, PH1) with a 4.7k pull-up: the write runs in the
second half of the tick and drops within microseconds of the edge, like the
address latch. One more transistor (747). The regenerated export passes
217/217 at TYP, LO, HI and three mixed seeds.

Co-Authored-By: Claude Fable 5.1 <noreply@anthropic.com>
Claude-Session: https://claude.ai/code/session_019vcbW37ERmrjZaWq55Er3J
Parts:
- added Q747: 2N7000, Package_TO_SOT_THT:TO-92_Inline_Wide, symbol Transistor_FET:2N7000
- R58: value 22k -> 4.7k
Connections:
- net BUS0#: now also Q173.2 (G), Q174.3 (D), Q205.2 (G), Q206.3 (D), Q237.2 (G), Q238.3 (D), Q269.2 (G), Q270.3 (D), Q301.2 (G), Q302.3 (D), Q333.2 (G), Q334.3 (D)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; no longer Q172.2 (G), Q173.3 (D), Q204.2 (G), Q205.3 (D), Q236.2 (G), Q237.3 (D), Q268.2 (G), Q269.3 (D), Q300.2 (G), Q301.3 (D), Q332.2 (G), Q333.3 (D)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
- net BUS1#: now also Q181.2 (G), Q182.3 (D), Q213.2 (G), Q214.3 (D), Q245.2 (G), Q246.3 (D), Q277.2 (G), Q278.3 (D), Q309.2 (G), Q310.3 (D), Q341.2 (G), Q342.3 (D)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; no longer Q180.2 (G), Q181.3 (D), Q212.2 (G), Q213.3 (D), Q244.2 (G), Q245.3 (D), Q276.2 (G), Q277.3 (D), Q308.2 (G), Q309.3 (D), Q340.2 (G), Q341.3 (D)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
- net BUS2#: now also Q189.2 (G), Q190.3 (D), Q221.2 (G), Q222.3 (D), Q253.2 (G), Q254.3 (D), Q285.2 (G), Q286.3 (D), Q317.2 (G), Q318.3 (D), Q349.2 (G), Q350.3 (D)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; no longer Q188.2 (G), Q189.3 (D), Q220.2 (G), Q221.3 (D), Q252.2 (G), Q253.3 (D), Q284.2 (G), Q285.3 (D), Q316.2 (G), Q317.3 (D), Q348.2 (G), Q349.3 (D)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
- net BUS3#: now also Q197.2 (G), Q198.3 (D), Q229.2 (G), Q230.3 (D), Q261.2 (G), Q262.3 (D), Q293.2 (G), Q294.3 (D), Q325.2 (G), Q326.3 (D), Q357.2 (G), Q358.3 (D)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; no longer Q196.2 (G), Q197.3 (D), Q228.2 (G), Q229.3 (D), Q260.2 (G), Q261.3 (D), Q292.2 (G), Q293.3 (D), Q324.2 (G), Q325.3 (D), Q356.2 (G), Q357.3 (D)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
- net D0: now also Q171.2 (G), Q203.2 (G), Q235.2 (G), Q267.2 (G), Q299.2 (G), Q331.2 (G), Q363.2 (G), Q395.2 (G), Q427.2 (G), Q459.2 (G), Q491.2 (G), Q523.2 (G)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; no longer Q170.2 (G), Q202.2 (G), Q234.2 (G), Q266.2 (G), Q298.2 (G), Q330.2 (G), Q362.2 (G), Q394.2 (G), Q426.2 (G), Q458.2 (G), Q490.2 (G), Q522.2 (G)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
- net D1: now also Q179.2 (G), Q211.2 (G), Q243.2 (G), Q275.2 (G), Q307.2 (G), Q339.2 (G), Q371.2 (G), Q403.2 (G), Q435.2 (G), Q467.2 (G), Q499.2 (G), Q531.2 (G)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; no longer Q178.2 (G), Q210.2 (G), Q242.2 (G), Q274.2 (G), Q306.2 (G), Q338.2 (G), Q370.2 (G), Q402.2 (G), Q434.2 (G), Q466.2 (G), Q498.2 (G), Q530.2 (G)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
- net D2: now also Q187.2 (G), Q219.2 (G), Q251.2 (G), Q283.2 (G), Q315.2 (G), Q347.2 (G), Q379.2 (G), Q411.2 (G), Q443.2 (G), Q475.2 (G), Q507.2 (G), Q539.2 (G)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; no longer Q186.2 (G), Q218.2 (G), Q250.2 (G), Q282.2 (G), Q314.2 (G), Q346.2 (G), Q378.2 (G), Q410.2 (G), Q442.2 (G), Q474.2 (G), Q506.2 (G), Q538.2 (G)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
- net D3: now also Q195.2 (G), Q227.2 (G), Q259.2 (G), Q291.2 (G), Q323.2 (G), Q355.2 (G), Q387.2 (G), Q419.2 (G), Q451.2 (G), Q483.2 (G), Q515.2 (G), Q547.2 (G)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; no longer Q194.2 (G), Q226.2 (G), Q258.2 (G), Q290.2 (G), Q322.2 (G), Q354.2 (G), Q386.2 (G), Q418.2 (G), Q450.2 (G), Q482.2 (G), Q514.2 (G), Q546.2 (G)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
- net GND: now also Q169.1 (S), Q171.1 (S), Q173.1 (S), Q177.1 (S), Q179.1 (S), Q181.1 (S), Q185.1 (S), Q187.1 (S), Q189.1 (S), Q193.1 (S), Q195.1 (S), Q197.1 (S)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; no longer Q101.1 (S), Q170.1 (S), Q172.1 (S), Q174.1 (S), Q178.1 (S), Q180.1 (S), Q182.1 (S), Q186.1 (S), Q188.1 (S), Q190.1 (S), Q194.1 (S), Q196.1 (S)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
- net MAR0: now also Q683.2 (G); no longer Q682.2 (G)
- net MAR1: now also Q682.2 (G); no longer Q681.2 (G)
- net MAR2: now also Q681.2 (G); no longer Q680.2 (G)
- net MAR3: now also Q680.2 (G); no longer Q679.2 (G)
- net MIN: now also Q105.2 (G), Q109.2 (G), Q113.2 (G), Q117.2 (G), Q121.2 (G), Q125.2 (G), Q129.2 (G), Q133.2 (G), Q137.2 (G), Q141.2 (G), Q145.2 (G), Q149.2 (G)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; no longer Q104.2 (G), Q108.2 (G), Q112.2 (G), Q116.2 (G), Q120.2 (G), Q124.2 (G), Q128.2 (G), Q132.2 (G), Q136.2 (G), Q140.2 (G), Q144.2 (G), Q148.2 (G)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
- net MO: now also Q103.2 (G); no longer Q102.2 (G)
- net MON: now also Q103.3 (D), Q107.2 (G), Q111.2 (G), Q115.2 (G), Q119.2 (G), Q123.2 (G), Q127.2 (G), Q131.2 (G), Q135.2 (G), Q139.2 (G), Q143.2 (G), Q147.2 (G)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; no longer Q102.3 (D), Q106.2 (G), Q110.2 (G), Q114.2 (G), Q118.2 (G), Q122.2 (G), Q126.2 (G), Q130.2 (G), Q134.2 (G), Q138.2 (G), Q142.2 (G), Q146.2 (G)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
- net PH1: now also Q102.2 (G)
- net Q0_0: now also Q168.3 (D), Q169.2 (G), Q172.3 (D), Q175.2 (G), Q687.2 (G); no longer Q167.3 (D), Q168.2 (G), Q171.3 (D), Q174.2 (G), Q686.2 (G)
- net Q0_0N: now also Q168.2 (G), Q170.3 (D); no longer Q167.2 (G), Q168.3 (D)
- net Q0_1: now also Q176.3 (D), Q177.2 (G), Q180.3 (D), Q183.2 (G), Q686.2 (G); no longer Q175.3 (D), Q176.2 (G), Q179.3 (D), Q182.2 (G), Q685.2 (G)
- net Q0_1N: now also Q176.2 (G), Q178.3 (D); no longer Q175.2 (G), Q176.3 (D)
- net Q0_2: now also Q184.3 (D), Q185.2 (G), Q188.3 (D), Q191.2 (G), Q685.2 (G); no longer Q183.3 (D), Q184.2 (G), Q187.3 (D), Q190.2 (G), Q684.2 (G)
- net Q0_2N: now also Q184.2 (G), Q186.3 (D); no longer Q183.2 (G), Q184.3 (D)
- net Q0_3: now also Q192.3 (D), Q193.2 (G), Q196.3 (D), Q199.2 (G), Q684.2 (G); no longer Q191.3 (D), Q192.2 (G), Q195.3 (D), Q198.2 (G), Q683.2 (G)
- net Q0_3N: now also Q192.2 (G), Q194.3 (D); no longer Q191.2 (G), Q192.3 (D)
- net Q10_0: now also Q488.3 (D), Q489.2 (G), Q492.3 (D), Q495.2 (G), Q727.2 (G); no longer Q487.3 (D), Q488.2 (G), Q491.3 (D), Q494.2 (G), Q726.2 (G)
- net Q10_0N: now also Q488.2 (G), Q490.3 (D); no longer Q487.2 (G), Q488.3 (D)
- net Q10_1: now also Q496.3 (D), Q497.2 (G), Q500.3 (D), Q503.2 (G), Q726.2 (G); no longer Q495.3 (D), Q496.2 (G), Q499.3 (D), Q502.2 (G), Q725.2 (G)
- net Q10_1N: now also Q496.2 (G), Q498.3 (D); no longer Q495.2 (G), Q496.3 (D)
- net Q10_2: now also Q504.3 (D), Q505.2 (G), Q508.3 (D), Q511.2 (G), Q725.2 (G); no longer Q503.3 (D), Q504.2 (G), Q507.3 (D), Q510.2 (G), Q724.2 (G)
- net Q10_2N: now also Q504.2 (G), Q506.3 (D); no longer Q503.2 (G), Q504.3 (D)
- net Q10_3: now also Q512.3 (D), Q513.2 (G), Q516.3 (D), Q519.2 (G), Q724.2 (G); no longer Q511.3 (D), Q512.2 (G), Q515.3 (D), Q518.2 (G), Q723.2 (G)
- net Q10_3N: now also Q512.2 (G), Q514.3 (D); no longer Q511.2 (G), Q512.3 (D)
- net Q11_0: now also Q520.3 (D), Q521.2 (G), Q524.3 (D), Q527.2 (G), Q731.2 (G); no longer Q519.3 (D), Q520.2 (G), Q523.3 (D), Q526.2 (G), Q730.2 (G)
- net Q11_0N: now also Q520.2 (G), Q522.3 (D); no longer Q519.2 (G), Q520.3 (D)
- net Q11_1: now also Q528.3 (D), Q529.2 (G), Q532.3 (D), Q535.2 (G), Q730.2 (G); no longer Q527.3 (D), Q528.2 (G), Q531.3 (D), Q534.2 (G), Q729.2 (G)
- net Q11_1N: now also Q528.2 (G), Q530.3 (D); no longer Q527.2 (G), Q528.3 (D)
- net Q11_2: now also Q536.3 (D), Q537.2 (G), Q540.3 (D), Q543.2 (G), Q729.2 (G); no longer Q535.3 (D), Q536.2 (G), Q539.3 (D), Q542.2 (G), Q728.2 (G)
- net Q11_2N: now also Q536.2 (G), Q538.3 (D); no longer Q535.2 (G), Q536.3 (D)
- net Q11_3: now also Q544.3 (D), Q545.2 (G), Q548.3 (D), Q551.2 (G), Q728.2 (G); no longer Q543.3 (D), Q544.2 (G), Q547.3 (D), Q550.2 (G), Q727.2 (G)
- net Q11_3N: now also Q544.2 (G), Q546.3 (D); no longer Q543.2 (G), Q544.3 (D)
- net Q12_0: now also Q552.3 (D), Q553.2 (G), Q556.3 (D), Q559.2 (G), Q735.2 (G); no longer Q551.3 (D), Q552.2 (G), Q555.3 (D), Q558.2 (G), Q734.2 (G)
- net Q12_0N: now also Q552.2 (G), Q554.3 (D); no longer Q551.2 (G), Q552.3 (D)
- net Q12_1: now also Q560.3 (D), Q561.2 (G), Q564.3 (D), Q567.2 (G), Q734.2 (G); no longer Q559.3 (D), Q560.2 (G), Q563.3 (D), Q566.2 (G), Q733.2 (G)
- net Q12_1N: now also Q560.2 (G), Q562.3 (D); no longer Q559.2 (G), Q560.3 (D)
- net Q12_2: now also Q568.3 (D), Q569.2 (G), Q572.3 (D), Q575.2 (G), Q733.2 (G); no longer Q567.3 (D), Q568.2 (G), Q571.3 (D), Q574.2 (G), Q732.2 (G)
- net Q12_2N: now also Q568.2 (G), Q570.3 (D); no longer Q567.2 (G), Q568.3 (D)
- net Q12_3: now also Q576.3 (D), Q577.2 (G), Q580.3 (D), Q583.2 (G), Q732.2 (G); no longer Q575.3 (D), Q576.2 (G), Q579.3 (D), Q582.2 (G), Q731.2 (G)
- net Q12_3N: now also Q576.2 (G), Q578.3 (D); no longer Q575.2 (G), Q576.3 (D)
- net Q13_0: now also Q584.3 (D), Q585.2 (G), Q588.3 (D), Q591.2 (G), Q739.2 (G); no longer Q583.3 (D), Q584.2 (G), Q587.3 (D), Q590.2 (G), Q738.2 (G)
- net Q13_0N: now also Q584.2 (G), Q586.3 (D); no longer Q583.2 (G), Q584.3 (D)
- net Q13_1: now also Q592.3 (D), Q593.2 (G), Q596.3 (D), Q599.2 (G), Q738.2 (G); no longer Q591.3 (D), Q592.2 (G), Q595.3 (D), Q598.2 (G), Q737.2 (G)
- net Q13_1N: now also Q592.2 (G), Q594.3 (D); no longer Q591.2 (G), Q592.3 (D)
- net Q13_2: now also Q600.3 (D), Q601.2 (G), Q604.3 (D), Q607.2 (G), Q737.2 (G); no longer Q599.3 (D), Q600.2 (G), Q603.3 (D), Q606.2 (G), Q736.2 (G)
- net Q13_2N: now also Q600.2 (G), Q602.3 (D); no longer Q599.2 (G), Q600.3 (D)
- net Q13_3: now also Q608.3 (D), Q609.2 (G), Q612.3 (D), Q615.2 (G), Q736.2 (G); no longer Q607.3 (D), Q608.2 (G), Q611.3 (D), Q614.2 (G), Q735.2 (G)
- net Q13_3N: now also Q608.2 (G), Q610.3 (D); no longer Q607.2 (G), Q608.3 (D)
- net Q14_0: now also Q616.3 (D), Q617.2 (G), Q620.3 (D), Q623.2 (G), Q743.2 (G); no longer Q615.3 (D), Q616.2 (G), Q619.3 (D), Q622.2 (G), Q742.2 (G)
- net Q14_0N: now also Q616.2 (G), Q618.3 (D); no longer Q615.2 (G), Q616.3 (D)
- net Q14_1: now also Q624.3 (D), Q625.2 (G), Q628.3 (D), Q631.2 (G), Q742.2 (G); no longer Q623.3 (D), Q624.2 (G), Q627.3 (D), Q630.2 (G), Q741.2 (G)
- net Q14_1N: now also Q624.2 (G), Q626.3 (D); no longer Q623.2 (G), Q624.3 (D)
- net Q14_2: now also Q632.3 (D), Q633.2 (G), Q636.3 (D), Q639.2 (G), Q741.2 (G); no longer Q631.3 (D), Q632.2 (G), Q635.3 (D), Q638.2 (G), Q740.2 (G)
- net Q14_2N: now also Q632.2 (G), Q634.3 (D); no longer Q631.2 (G), Q632.3 (D)
- net Q14_3: now also Q640.3 (D), Q641.2 (G), Q644.3 (D), Q647.2 (G), Q740.2 (G); no longer Q639.3 (D), Q640.2 (G), Q643.3 (D), Q646.2 (G), Q739.2 (G)
- net Q14_3N: now also Q640.2 (G), Q642.3 (D); no longer Q639.2 (G), Q640.3 (D)
- net Q15_0: now also Q648.3 (D), Q649.2 (G), Q652.3 (D), Q655.2 (G), Q747.2 (G); no longer Q647.3 (D), Q648.2 (G), Q651.3 (D), Q654.2 (G), Q746.2 (G)
- net Q15_0N: now also Q648.2 (G), Q650.3 (D); no longer Q647.2 (G), Q648.3 (D)
- net Q15_1: now also Q656.3 (D), Q657.2 (G), Q660.3 (D), Q663.2 (G), Q746.2 (G); no longer Q655.3 (D), Q656.2 (G), Q659.3 (D), Q662.2 (G), Q745.2 (G)
- net Q15_1N: now also Q656.2 (G), Q658.3 (D); no longer Q655.2 (G), Q656.3 (D)
- net Q15_2: now also Q664.3 (D), Q665.2 (G), Q668.3 (D), Q671.2 (G), Q745.2 (G); no longer Q663.3 (D), Q664.2 (G), Q667.3 (D), Q670.2 (G), Q744.2 (G)
- net Q15_2N: now also Q664.2 (G), Q666.3 (D); no longer Q663.2 (G), Q664.3 (D)
- net Q15_3: now also Q672.3 (D), Q673.2 (G), Q676.3 (D), Q679.2 (G), Q744.2 (G); no longer Q671.3 (D), Q672.2 (G), Q675.3 (D), Q678.2 (G), Q743.2 (G)
- net Q15_3N: now also Q672.2 (G), Q674.3 (D); no longer Q671.2 (G), Q672.3 (D)
- net Q1_0: now also Q200.3 (D), Q201.2 (G), Q204.3 (D), Q207.2 (G), Q691.2 (G); no longer Q199.3 (D), Q200.2 (G), Q203.3 (D), Q206.2 (G), Q690.2 (G)
- net Q1_0N: now also Q200.2 (G), Q202.3 (D); no longer Q199.2 (G), Q200.3 (D)
- net Q1_1: now also Q208.3 (D), Q209.2 (G), Q212.3 (D), Q215.2 (G), Q690.2 (G); no longer Q207.3 (D), Q208.2 (G), Q211.3 (D), Q214.2 (G), Q689.2 (G)
- net Q1_1N: now also Q208.2 (G), Q210.3 (D); no longer Q207.2 (G), Q208.3 (D)
- net Q1_2: now also Q216.3 (D), Q217.2 (G), Q220.3 (D), Q223.2 (G), Q689.2 (G); no longer Q215.3 (D), Q216.2 (G), Q219.3 (D), Q222.2 (G), Q688.2 (G)
- net Q1_2N: now also Q216.2 (G), Q218.3 (D); no longer Q215.2 (G), Q216.3 (D)
- net Q1_3: now also Q224.3 (D), Q225.2 (G), Q228.3 (D), Q231.2 (G), Q688.2 (G); no longer Q223.3 (D), Q224.2 (G), Q227.3 (D), Q230.2 (G), Q687.2 (G)
- net Q1_3N: now also Q224.2 (G), Q226.3 (D); no longer Q223.2 (G), Q224.3 (D)
- net Q2_0: now also Q232.3 (D), Q233.2 (G), Q236.3 (D), Q239.2 (G), Q695.2 (G); no longer Q231.3 (D), Q232.2 (G), Q235.3 (D), Q238.2 (G), Q694.2 (G)
- net Q2_0N: now also Q232.2 (G), Q234.3 (D); no longer Q231.2 (G), Q232.3 (D)
- net Q2_1: now also Q240.3 (D), Q241.2 (G), Q244.3 (D), Q247.2 (G), Q694.2 (G); no longer Q239.3 (D), Q240.2 (G), Q243.3 (D), Q246.2 (G), Q693.2 (G)
- net Q2_1N: now also Q240.2 (G), Q242.3 (D); no longer Q239.2 (G), Q240.3 (D)
- net Q2_2: now also Q248.3 (D), Q249.2 (G), Q252.3 (D), Q255.2 (G), Q693.2 (G); no longer Q247.3 (D), Q248.2 (G), Q251.3 (D), Q254.2 (G), Q692.2 (G)
- net Q2_2N: now also Q248.2 (G), Q250.3 (D); no longer Q247.2 (G), Q248.3 (D)
- net Q2_3: now also Q256.3 (D), Q257.2 (G), Q260.3 (D), Q263.2 (G), Q692.2 (G); no longer Q255.3 (D), Q256.2 (G), Q259.3 (D), Q262.2 (G), Q691.2 (G)
- net Q2_3N: now also Q256.2 (G), Q258.3 (D); no longer Q255.2 (G), Q256.3 (D)
- net Q3_0: now also Q264.3 (D), Q265.2 (G), Q268.3 (D), Q271.2 (G), Q699.2 (G); no longer Q263.3 (D), Q264.2 (G), Q267.3 (D), Q270.2 (G), Q698.2 (G)
- net Q3_0N: now also Q264.2 (G), Q266.3 (D); no longer Q263.2 (G), Q264.3 (D)
- net Q3_1: now also Q272.3 (D), Q273.2 (G), Q276.3 (D), Q279.2 (G), Q698.2 (G); no longer Q271.3 (D), Q272.2 (G), Q275.3 (D), Q278.2 (G), Q697.2 (G)
- net Q3_1N: now also Q272.2 (G), Q274.3 (D); no longer Q271.2 (G), Q272.3 (D)
- net Q3_2: now also Q280.3 (D), Q281.2 (G), Q284.3 (D), Q287.2 (G), Q697.2 (G); no longer Q279.3 (D), Q280.2 (G), Q283.3 (D), Q286.2 (G), Q696.2 (G)
- net Q3_2N: now also Q280.2 (G), Q282.3 (D); no longer Q279.2 (G), Q280.3 (D)
- net Q3_3: now also Q288.3 (D), Q289.2 (G), Q292.3 (D), Q295.2 (G), Q696.2 (G); no longer Q287.3 (D), Q288.2 (G), Q291.3 (D), Q294.2 (G), Q695.2 (G)
- net Q3_3N: now also Q288.2 (G), Q290.3 (D); no longer Q287.2 (G), Q288.3 (D)
- net Q4_0: now also Q296.3 (D), Q297.2 (G), Q300.3 (D), Q303.2 (G), Q703.2 (G); no longer Q295.3 (D), Q296.2 (G), Q299.3 (D), Q302.2 (G), Q702.2 (G)
- net Q4_0N: now also Q296.2 (G), Q298.3 (D); no longer Q295.2 (G), Q296.3 (D)
- net Q4_1: now also Q304.3 (D), Q305.2 (G), Q308.3 (D), Q311.2 (G), Q702.2 (G); no longer Q303.3 (D), Q304.2 (G), Q307.3 (D), Q310.2 (G), Q701.2 (G)
- net Q4_1N: now also Q304.2 (G), Q306.3 (D); no longer Q303.2 (G), Q304.3 (D)
- net Q4_2: now also Q312.3 (D), Q313.2 (G), Q316.3 (D), Q319.2 (G), Q701.2 (G); no longer Q311.3 (D), Q312.2 (G), Q315.3 (D), Q318.2 (G), Q700.2 (G)
- net Q4_2N: now also Q312.2 (G), Q314.3 (D); no longer Q311.2 (G), Q312.3 (D)
- net Q4_3: now also Q320.3 (D), Q321.2 (G), Q324.3 (D), Q327.2 (G), Q700.2 (G); no longer Q319.3 (D), Q320.2 (G), Q323.3 (D), Q326.2 (G), Q699.2 (G)
- net Q4_3N: now also Q320.2 (G), Q322.3 (D); no longer Q319.2 (G), Q320.3 (D)
- net Q5_0: now also Q328.3 (D), Q329.2 (G), Q332.3 (D), Q335.2 (G), Q707.2 (G); no longer Q327.3 (D), Q328.2 (G), Q331.3 (D), Q334.2 (G), Q706.2 (G)
- net Q5_0N: now also Q328.2 (G), Q330.3 (D); no longer Q327.2 (G), Q328.3 (D)
- net Q5_1: now also Q336.3 (D), Q337.2 (G), Q340.3 (D), Q343.2 (G), Q706.2 (G); no longer Q335.3 (D), Q336.2 (G), Q339.3 (D), Q342.2 (G), Q705.2 (G)
- net Q5_1N: now also Q336.2 (G), Q338.3 (D); no longer Q335.2 (G), Q336.3 (D)
- net Q5_2: now also Q344.3 (D), Q345.2 (G), Q348.3 (D), Q351.2 (G), Q705.2 (G); no longer Q343.3 (D), Q344.2 (G), Q347.3 (D), Q350.2 (G), Q704.2 (G)
- net Q5_2N: now also Q344.2 (G), Q346.3 (D); no longer Q343.2 (G), Q344.3 (D)
- net Q5_3: now also Q352.3 (D), Q353.2 (G), Q356.3 (D), Q359.2 (G), Q704.2 (G); no longer Q351.3 (D), Q352.2 (G), Q355.3 (D), Q358.2 (G), Q703.2 (G)
- net Q5_3N: now also Q352.2 (G), Q354.3 (D); no longer Q351.2 (G), Q352.3 (D)
- net Q6_0: now also Q360.3 (D), Q361.2 (G), Q364.3 (D), Q367.2 (G), Q711.2 (G); no longer Q359.3 (D), Q360.2 (G), Q363.3 (D), Q366.2 (G), Q710.2 (G)
- net Q6_0N: now also Q360.2 (G), Q362.3 (D); no longer Q359.2 (G), Q360.3 (D)
- net Q6_1: now also Q368.3 (D), Q369.2 (G), Q372.3 (D), Q375.2 (G), Q710.2 (G); no longer Q367.3 (D), Q368.2 (G), Q371.3 (D), Q374.2 (G), Q709.2 (G)
- net Q6_1N: now also Q368.2 (G), Q370.3 (D); no longer Q367.2 (G), Q368.3 (D)
- net Q6_2: now also Q376.3 (D), Q377.2 (G), Q380.3 (D), Q383.2 (G), Q709.2 (G); no longer Q375.3 (D), Q376.2 (G), Q379.3 (D), Q382.2 (G), Q708.2 (G)
- net Q6_2N: now also Q376.2 (G), Q378.3 (D); no longer Q375.2 (G), Q376.3 (D)
- net Q6_3: now also Q384.3 (D), Q385.2 (G), Q388.3 (D), Q391.2 (G), Q708.2 (G); no longer Q383.3 (D), Q384.2 (G), Q387.3 (D), Q390.2 (G), Q707.2 (G)
- net Q6_3N: now also Q384.2 (G), Q386.3 (D); no longer Q383.2 (G), Q384.3 (D)
- net Q7_0: now also Q392.3 (D), Q393.2 (G), Q396.3 (D), Q399.2 (G), Q715.2 (G); no longer Q391.3 (D), Q392.2 (G), Q395.3 (D), Q398.2 (G), Q714.2 (G)
- net Q7_0N: now also Q392.2 (G), Q394.3 (D); no longer Q391.2 (G), Q392.3 (D)
- net Q7_1: now also Q400.3 (D), Q401.2 (G), Q404.3 (D), Q407.2 (G), Q714.2 (G); no longer Q399.3 (D), Q400.2 (G), Q403.3 (D), Q406.2 (G), Q713.2 (G)
- net Q7_1N: now also Q400.2 (G), Q402.3 (D); no longer Q399.2 (G), Q400.3 (D)
- net Q7_2: now also Q408.3 (D), Q409.2 (G), Q412.3 (D), Q415.2 (G), Q713.2 (G); no longer Q407.3 (D), Q408.2 (G), Q411.3 (D), Q414.2 (G), Q712.2 (G)
- net Q7_2N: now also Q408.2 (G), Q410.3 (D); no longer Q407.2 (G), Q408.3 (D)
- net Q7_3: now also Q416.3 (D), Q417.2 (G), Q420.3 (D), Q423.2 (G), Q712.2 (G); no longer Q415.3 (D), Q416.2 (G), Q419.3 (D), Q422.2 (G), Q711.2 (G)
- net Q7_3N: now also Q416.2 (G), Q418.3 (D); no longer Q415.2 (G), Q416.3 (D)
- net Q8_0: now also Q424.3 (D), Q425.2 (G), Q428.3 (D), Q431.2 (G), Q719.2 (G); no longer Q423.3 (D), Q424.2 (G), Q427.3 (D), Q430.2 (G), Q718.2 (G)
- net Q8_0N: now also Q424.2 (G), Q426.3 (D); no longer Q423.2 (G), Q424.3 (D)
- net Q8_1: now also Q432.3 (D), Q433.2 (G), Q436.3 (D), Q439.2 (G), Q718.2 (G); no longer Q431.3 (D), Q432.2 (G), Q435.3 (D), Q438.2 (G), Q717.2 (G)
- net Q8_1N: now also Q432.2 (G), Q434.3 (D); no longer Q431.2 (G), Q432.3 (D)
- net Q8_2: now also Q440.3 (D), Q441.2 (G), Q444.3 (D), Q447.2 (G), Q717.2 (G); no longer Q439.3 (D), Q440.2 (G), Q443.3 (D), Q446.2 (G), Q716.2 (G)
- net Q8_2N: now also Q440.2 (G), Q442.3 (D); no longer Q439.2 (G), Q440.3 (D)
- net Q8_3: now also Q448.3 (D), Q449.2 (G), Q452.3 (D), Q455.2 (G), Q716.2 (G); no longer Q447.3 (D), Q448.2 (G), Q451.3 (D), Q454.2 (G), Q715.2 (G)
- net Q8_3N: now also Q448.2 (G), Q450.3 (D); no longer Q447.2 (G), Q448.3 (D)
- net Q9_0: now also Q456.3 (D), Q457.2 (G), Q460.3 (D), Q463.2 (G), Q723.2 (G); no longer Q455.3 (D), Q456.2 (G), Q459.3 (D), Q462.2 (G), Q722.2 (G)
- net Q9_0N: now also Q456.2 (G), Q458.3 (D); no longer Q455.2 (G), Q456.3 (D)
- net Q9_1: now also Q464.3 (D), Q465.2 (G), Q468.3 (D), Q471.2 (G), Q722.2 (G); no longer Q463.3 (D), Q464.2 (G), Q467.3 (D), Q470.2 (G), Q721.2 (G)
- net Q9_1N: now also Q464.2 (G), Q466.3 (D); no longer Q463.2 (G), Q464.3 (D)
- net Q9_2: now also Q472.3 (D), Q473.2 (G), Q476.3 (D), Q479.2 (G), Q721.2 (G); no longer Q471.3 (D), Q472.2 (G), Q475.3 (D), Q478.2 (G), Q720.2 (G)
- net Q9_2N: now also Q472.2 (G), Q474.3 (D); no longer Q471.2 (G), Q472.3 (D)
- net Q9_3: now also Q480.3 (D), Q481.2 (G), Q484.3 (D), Q487.2 (G), Q720.2 (G); no longer Q479.3 (D), Q480.2 (G), Q483.3 (D), Q486.2 (G), Q719.2 (G)
- net Q9_3N: now also Q480.2 (G), Q482.3 (D); no longer Q479.2 (G), Q480.3 (D)
- net RD0: now also Q107.3 (D), Q174.2 (G), Q182.2 (G), Q190.2 (G), Q198.2 (G); no longer Q105.3 (D), Q173.2 (G), Q181.2 (G), Q189.2 (G), Q197.2 (G)
- net RD1: now also Q111.3 (D), Q206.2 (G), Q214.2 (G), Q222.2 (G), Q230.2 (G); no longer Q109.3 (D), Q205.2 (G), Q213.2 (G), Q221.2 (G), Q229.2 (G)
- net RD10: now also Q147.3 (D), Q494.2 (G), Q502.2 (G), Q510.2 (G), Q518.2 (G); no longer Q145.3 (D), Q493.2 (G), Q501.2 (G), Q509.2 (G), Q517.2 (G)
- net RD11: now also Q151.3 (D), Q526.2 (G), Q534.2 (G), Q542.2 (G), Q550.2 (G); no longer Q149.3 (D), Q525.2 (G), Q533.2 (G), Q541.2 (G), Q549.2 (G)
- net RD12: now also Q155.3 (D), Q558.2 (G), Q566.2 (G), Q574.2 (G), Q582.2 (G); no longer Q153.3 (D), Q557.2 (G), Q565.2 (G), Q573.2 (G), Q581.2 (G)
- net RD13: now also Q159.3 (D), Q590.2 (G), Q598.2 (G), Q606.2 (G), Q614.2 (G); no longer Q157.3 (D), Q589.2 (G), Q597.2 (G), Q605.2 (G), Q613.2 (G)
- net RD14: now also Q163.3 (D), Q622.2 (G), Q630.2 (G), Q638.2 (G), Q646.2 (G); no longer Q161.3 (D), Q621.2 (G), Q629.2 (G), Q637.2 (G), Q645.2 (G)
- net RD15: now also Q167.3 (D), Q654.2 (G), Q662.2 (G), Q670.2 (G), Q678.2 (G); no longer Q165.3 (D), Q653.2 (G), Q661.2 (G), Q669.2 (G), Q677.2 (G)
- net RD2: now also Q115.3 (D), Q238.2 (G), Q246.2 (G), Q254.2 (G), Q262.2 (G); no longer Q113.3 (D), Q237.2 (G), Q245.2 (G), Q253.2 (G), Q261.2 (G)
- net RD3: now also Q119.3 (D), Q270.2 (G), Q278.2 (G), Q286.2 (G), Q294.2 (G); no longer Q117.3 (D), Q269.2 (G), Q277.2 (G), Q285.2 (G), Q293.2 (G)
- net RD4: now also Q123.3 (D), Q302.2 (G), Q310.2 (G), Q318.2 (G), Q326.2 (G); no longer Q121.3 (D), Q301.2 (G), Q309.2 (G), Q317.2 (G), Q325.2 (G)
- net RD5: now also Q127.3 (D), Q334.2 (G), Q342.2 (G), Q350.2 (G), Q358.2 (G); no longer Q125.3 (D), Q333.2 (G), Q341.2 (G), Q349.2 (G), Q357.2 (G)
- net RD6: now also Q131.3 (D), Q366.2 (G), Q374.2 (G), Q382.2 (G), Q390.2 (G); no longer Q129.3 (D), Q365.2 (G), Q373.2 (G), Q381.2 (G), Q389.2 (G)
- net RD7: now also Q135.3 (D), Q398.2 (G), Q406.2 (G), Q414.2 (G), Q422.2 (G); no longer Q133.3 (D), Q397.2 (G), Q405.2 (G), Q413.2 (G), Q421.2 (G)
- net RD8: now also Q139.3 (D), Q430.2 (G), Q438.2 (G), Q446.2 (G), Q454.2 (G); no longer Q137.3 (D), Q429.2 (G), Q437.2 (G), Q445.2 (G), Q453.2 (G)
- net RD9: now also Q143.3 (D), Q462.2 (G), Q470.2 (G), Q478.2 (G), Q486.2 (G); no longer Q141.3 (D), Q461.2 (G), Q469.2 (G), Q477.2 (G), Q485.2 (G)
- net W0#: now also Q104.2 (G), Q106.2 (G); no longer Q103.2 (G), Q105.2 (G)
- net W1#: now also Q108.2 (G), Q110.2 (G); no longer Q107.2 (G), Q109.2 (G)
- net W10#: now also Q144.2 (G), Q146.2 (G); no longer Q143.2 (G), Q145.2 (G)
- net W11#: now also Q148.2 (G), Q150.2 (G); no longer Q147.2 (G), Q149.2 (G)
- net W12#: now also Q152.2 (G), Q154.2 (G); no longer Q151.2 (G), Q153.2 (G)
- net W13#: now also Q156.2 (G), Q158.2 (G); no longer Q155.2 (G), Q157.2 (G)
- net W14#: now also Q160.2 (G), Q162.2 (G); no longer Q159.2 (G), Q161.2 (G)
- net W15#: now also Q164.2 (G), Q166.2 (G); no longer Q163.2 (G), Q165.2 (G)
- net W2#: now also Q112.2 (G), Q114.2 (G); no longer Q111.2 (G), Q113.2 (G)
- net W3#: now also Q116.2 (G), Q118.2 (G); no longer Q115.2 (G), Q117.2 (G)
- net W4#: now also Q120.2 (G), Q122.2 (G); no longer Q119.2 (G), Q121.2 (G)
- net W5#: now also Q124.2 (G), Q126.2 (G); no longer Q123.2 (G), Q125.2 (G)
- net W6#: now also Q128.2 (G), Q130.2 (G); no longer Q127.2 (G), Q129.2 (G)
- net W7#: now also Q132.2 (G), Q134.2 (G); no longer Q131.2 (G), Q133.2 (G)
- net W8#: now also Q136.2 (G), Q138.2 (G); no longer Q135.2 (G), Q137.2 (G)
- net W9#: now also Q140.2 (G), Q142.2 (G); no longer Q139.2 (G), Q141.2 (G)
- net WR0: now also Q105.3 (D), Q170.2 (G), Q172.2 (G), Q178.2 (G), Q180.2 (G), Q186.2 (G), Q188.2 (G), Q194.2 (G), Q196.2 (G); no longer Q103.3 (D), Q169.2 (G), Q171.2 (G), Q177.2 (G), Q179.2 (G), Q185.2 (G), Q187.2 (G), Q193.2 (G), Q195.2 (G)
- net WR1: now also Q109.3 (D), Q202.2 (G), Q204.2 (G), Q210.2 (G), Q212.2 (G), Q218.2 (G), Q220.2 (G), Q226.2 (G), Q228.2 (G); no longer Q107.3 (D), Q201.2 (G), Q203.2 (G), Q209.2 (G), Q211.2 (G), Q217.2 (G), Q219.2 (G), Q225.2 (G), Q227.2 (G)
- net WR10: now also Q145.3 (D), Q490.2 (G), Q492.2 (G), Q498.2 (G), Q500.2 (G), Q506.2 (G), Q508.2 (G), Q514.2 (G), Q516.2 (G); no longer Q143.3 (D), Q489.2 (G), Q491.2 (G), Q497.2 (G), Q499.2 (G), Q505.2 (G), Q507.2 (G), Q513.2 (G), Q515.2 (G)
- net WR11: now also Q149.3 (D), Q522.2 (G), Q524.2 (G), Q530.2 (G), Q532.2 (G), Q538.2 (G), Q540.2 (G), Q546.2 (G), Q548.2 (G); no longer Q147.3 (D), Q521.2 (G), Q523.2 (G), Q529.2 (G), Q531.2 (G), Q537.2 (G), Q539.2 (G), Q545.2 (G), Q547.2 (G)
- net WR12: now also Q153.3 (D), Q554.2 (G), Q556.2 (G), Q562.2 (G), Q564.2 (G), Q570.2 (G), Q572.2 (G), Q578.2 (G), Q580.2 (G); no longer Q151.3 (D), Q553.2 (G), Q555.2 (G), Q561.2 (G), Q563.2 (G), Q569.2 (G), Q571.2 (G), Q577.2 (G), Q579.2 (G)
- net WR13: now also Q157.3 (D), Q586.2 (G), Q588.2 (G), Q594.2 (G), Q596.2 (G), Q602.2 (G), Q604.2 (G), Q610.2 (G), Q612.2 (G); no longer Q155.3 (D), Q585.2 (G), Q587.2 (G), Q593.2 (G), Q595.2 (G), Q601.2 (G), Q603.2 (G), Q609.2 (G), Q611.2 (G)
- net WR14: now also Q161.3 (D), Q618.2 (G), Q620.2 (G), Q626.2 (G), Q628.2 (G), Q634.2 (G), Q636.2 (G), Q642.2 (G), Q644.2 (G); no longer Q159.3 (D), Q617.2 (G), Q619.2 (G), Q625.2 (G), Q627.2 (G), Q633.2 (G), Q635.2 (G), Q641.2 (G), Q643.2 (G)
- net WR15: now also Q165.3 (D), Q650.2 (G), Q652.2 (G), Q658.2 (G), Q660.2 (G), Q666.2 (G), Q668.2 (G), Q674.2 (G), Q676.2 (G); no longer Q163.3 (D), Q649.2 (G), Q651.2 (G), Q657.2 (G), Q659.2 (G), Q665.2 (G), Q667.2 (G), Q673.2 (G), Q675.2 (G)
- net WR2: now also Q113.3 (D), Q234.2 (G), Q236.2 (G), Q242.2 (G), Q244.2 (G), Q250.2 (G), Q252.2 (G), Q258.2 (G), Q260.2 (G); no longer Q111.3 (D), Q233.2 (G), Q235.2 (G), Q241.2 (G), Q243.2 (G), Q249.2 (G), Q251.2 (G), Q257.2 (G), Q259.2 (G)
- net WR3: now also Q117.3 (D), Q266.2 (G), Q268.2 (G), Q274.2 (G), Q276.2 (G), Q282.2 (G), Q284.2 (G), Q290.2 (G), Q292.2 (G); no longer Q115.3 (D), Q265.2 (G), Q267.2 (G), Q273.2 (G), Q275.2 (G), Q281.2 (G), Q283.2 (G), Q289.2 (G), Q291.2 (G)
- net WR4: now also Q121.3 (D), Q298.2 (G), Q300.2 (G), Q306.2 (G), Q308.2 (G), Q314.2 (G), Q316.2 (G), Q322.2 (G), Q324.2 (G); no longer Q119.3 (D), Q297.2 (G), Q299.2 (G), Q305.2 (G), Q307.2 (G), Q313.2 (G), Q315.2 (G), Q321.2 (G), Q323.2 (G)
- net WR5: now also Q125.3 (D), Q330.2 (G), Q332.2 (G), Q338.2 (G), Q340.2 (G), Q346.2 (G), Q348.2 (G), Q354.2 (G), Q356.2 (G); no longer Q123.3 (D), Q329.2 (G), Q331.2 (G), Q337.2 (G), Q339.2 (G), Q345.2 (G), Q347.2 (G), Q353.2 (G), Q355.2 (G)
- net WR6: now also Q129.3 (D), Q362.2 (G), Q364.2 (G), Q370.2 (G), Q372.2 (G), Q378.2 (G), Q380.2 (G), Q386.2 (G), Q388.2 (G); no longer Q127.3 (D), Q361.2 (G), Q363.2 (G), Q369.2 (G), Q371.2 (G), Q377.2 (G), Q379.2 (G), Q385.2 (G), Q387.2 (G)
- net WR7: now also Q133.3 (D), Q394.2 (G), Q396.2 (G), Q402.2 (G), Q404.2 (G), Q410.2 (G), Q412.2 (G), Q418.2 (G), Q420.2 (G); no longer Q131.3 (D), Q393.2 (G), Q395.2 (G), Q401.2 (G), Q403.2 (G), Q409.2 (G), Q411.2 (G), Q417.2 (G), Q419.2 (G)
- net WR8: now also Q137.3 (D), Q426.2 (G), Q428.2 (G), Q434.2 (G), Q436.2 (G), Q442.2 (G), Q444.2 (G), Q450.2 (G), Q452.2 (G); no longer Q135.3 (D), Q425.2 (G), Q427.2 (G), Q433.2 (G), Q435.2 (G), Q441.2 (G), Q443.2 (G), Q449.2 (G), Q451.2 (G)
- net WR9: now also Q141.3 (D), Q458.2 (G), Q460.2 (G), Q466.2 (G), Q468.2 (G), Q474.2 (G), Q476.2 (G), Q482.2 (G), Q484.2 (G); no longer Q139.3 (D), Q457.2 (G), Q459.2 (G), Q465.2 (G), Q467.2 (G), Q473.2 (G), Q475.2 (G), Q481.2 (G), Q483.2 (G)
- net at Q745.3 (D): now also D66.1 (K); no longer D67.1 (K)
- net at D64.1 (K): now also Q743.3 (D); no longer Q742.3 (D)
- net at D24.1 (K): now also Q703.3 (D); no longer Q702.3 (D)
- net at D60.1 (K): now also Q739.3 (D); no longer Q738.3 (D)
- net at D25.1 (K): now also Q704.3 (D); no longer Q703.3 (D)
- net at Q684.3 (D): now also D5.1 (K); no longer D6.1 (K)
- net at D38.1 (K): now also Q717.3 (D); no longer Q716.3 (D)
- net at D42.1 (K): now also Q721.3 (D); no longer Q720.3 (D)
- net at D39.1 (K): now also Q718.3 (D); no longer Q717.3 (D)
- net at D26.1 (K): now also Q705.3 (D); no longer Q704.3 (D)
- net at D58.1 (K): now also Q737.3 (D); no longer Q736.3 (D)
- net at D36.1 (K): now also Q715.3 (D); no longer Q714.3 (D)
- net at Q686.3 (D): now also D7.1 (K); no longer D8.1 (K)
- net at D18.1 (K): now also Q697.3 (D); no longer Q696.3 (D)
- net at D29.1 (K): now also Q708.3 (D); no longer Q707.3 (D)
- net at Q734.3 (D): now also D55.1 (K); no longer D56.1 (K)
- net at D11.1 (K): now also Q690.3 (D); no longer Q689.3 (D)
- net at Q732.3 (D): now also D53.1 (K); no longer D54.1 (K)
- net at D32.1 (K): now also Q711.3 (D); no longer Q710.3 (D)
- net at Q698.3 (D): now also D19.1 (K); no longer D20.1 (K)
- net at D15.1 (K): now also Q694.3 (D); no longer Q693.3 (D)
- net at D33.1 (K): now also Q712.3 (D); no longer Q711.3 (D)
- net at D21.1 (K): now also Q700.3 (D); no longer Q699.3 (D)
- net at D34.1 (K): now also Q713.3 (D); no longer Q712.3 (D)
- net at Q729.3 (D): now also D50.1 (K); no longer D51.1 (K)
- net at D41.1 (K): now also Q720.3 (D); no longer Q719.3 (D)
- net at Q683.3 (D): now also D4.1 (K); no longer D5.1 (K)
- net at D49.1 (K): now also Q728.3 (D); no longer Q727.3 (D)
- net at D61.1 (K): now also Q740.3 (D); no longer Q739.3 (D)
- net at Q735.3 (D): now also D56.1 (K); no longer D57.1 (K)
- net at Q687.3 (D): now also D8.1 (K); no longer D9.1 (K)
- net at D45.1 (K): now also Q724.3 (D); no longer Q723.3 (D)
- net at D12.1 (K): now also Q691.3 (D); no longer Q690.3 (D)
- net at Q688.3 (D): now also D9.1 (K); no longer D10.1 (K)
- net at D46.1 (K): now also Q725.3 (D); no longer Q724.3 (D)
- net at D37.1 (K): now also Q716.3 (D); no longer Q715.3 (D)
- net at D16.1 (K): now also Q695.3 (D); no longer Q694.3 (D)
- net at D23.1 (K): now also Q702.3 (D); no longer Q701.3 (D)
- net at Q679.3 (D): now also Q678.1 (S); no longer D1.1 (K)
- net at D17.1 (K): now also Q696.3 (D); no longer Q695.3 (D)
- net at D35.1 (K): now also Q714.3 (D); no longer Q713.3 (D)
- net at D14.1 (K): now also Q693.3 (D); no longer Q692.3 (D)
- net at D47.1 (K): now also Q726.3 (D); no longer Q725.3 (D)
- net at D48.1 (K): now also Q727.3 (D); no longer Q726.3 (D)
- net at Q685.3 (D): now also D6.1 (K); no longer D7.1 (K)
- net at D65.1 (K): now also Q744.3 (D); no longer Q743.3 (D)
- net at D63.1 (K): now also Q742.3 (D); no longer Q741.3 (D)
- net at D40.1 (K): now also Q719.3 (D); no longer Q718.3 (D)
- net at D43.1 (K): now also Q722.3 (D); no longer Q721.3 (D)
- net at D44.1 (K): now also Q723.3 (D); no longer Q722.3 (D)
- net at Q680.3 (D): now also D1.1 (K); no longer D2.1 (K)
- net at Q706.3 (D): now also D27.1 (K); no longer D28.1 (K)
- net at D13.1 (K): now also Q692.3 (D); no longer Q691.3 (D)
- net at D3.1 (K): now also Q682.3 (D); no longer Q681.3 (D)
- net at D30.1 (K): now also Q709.3 (D); no longer Q708.3 (D)
- net at Q731.3 (D): now also D52.1 (K); no longer D53.1 (K)
- net at D59.1 (K): now also Q738.3 (D); no longer Q737.3 (D)
- net at Q730.3 (D): now also D51.1 (K); no longer D52.1 (K)
- net at D62.1 (K): now also Q741.3 (D); no longer Q740.3 (D)
- net at Q746.3 (D): now also D67.1 (K); no longer D68.1 (K)
- net at D22.1 (K): now also Q701.3 (D); no longer Q700.3 (D)
- net at Q733.3 (D): now also D54.1 (K); no longer D55.1 (K)
- net at D31.1 (K): now also Q710.3 (D); no longer Q709.3 (D)
- new net: Q220.1 (S), Q221.3 (D)
- new net: Q430.1 (S), Q431.3 (D)
- new net: Q580.1 (S), Q581.3 (D)
- new net: Q246.1 (S), Q247.3 (D)
- new net: Q364.1 (S), Q365.3 (D)
- new net: Q510.1 (S), Q511.3 (D)
- new net: Q398.1 (S), Q399.3 (D)
- new net: Q674.1 (S), Q675.3 (D)
- new net: Q390.1 (S), Q391.3 (D)
- new net: Q334.1 (S), Q335.3 (D)
- new net: Q276.1 (S), Q277.3 (D)
- new net: Q212.1 (S), Q213.3 (D)
- new net: Q550.1 (S), Q551.3 (D)
- new net: Q654.1 (S), Q655.3 (D)
- new net: Q500.1 (S), Q501.3 (D)
- new net: Q388.1 (S), Q389.3 (D)
- new net: Q582.1 (S), Q583.3 (D)
- new net: Q170.1 (S), Q171.3 (D)
- new net: Q262.1 (S), Q263.3 (D)
- new net: Q326.1 (S), Q327.3 (D)
- new net: Q668.1 (S), Q669.3 (D)
- new net: Q354.1 (S), Q355.3 (D)
- new net: Q222.1 (S), Q223.3 (D)
- new net: Q204.1 (S), Q205.3 (D)
- new net: Q234.1 (S), Q235.3 (D)
- new net: Q478.1 (S), Q479.3 (D)
- new net: Q402.1 (S), Q403.3 (D)
- new net: Q574.1 (S), Q575.3 (D)
- new net: Q362.1 (S), Q363.3 (D)
- new net: Q462.1 (S), Q463.3 (D)
- new net: Q414.1 (S), Q415.3 (D)
- new net: Q228.1 (S), Q229.3 (D)
- new net: Q302.1 (S), Q303.3 (D)
- new net: Q502.1 (S), Q503.3 (D)
- new net: Q338.1 (S), Q339.3 (D)
- new net: Q412.1 (S), Q413.3 (D)
- new net: Q460.1 (S), Q461.3 (D)
- new net: Q436.1 (S), Q437.3 (D)
- new net: Q452.1 (S), Q453.3 (D)
- new net: Q612.1 (S), Q613.3 (D)
- new net: Q286.1 (S), Q287.3 (D)
- new net: Q534.1 (S), Q535.3 (D)
- new net: Q386.1 (S), Q387.3 (D)
- new net: Q646.1 (S), Q647.3 (D)
- new net: Q484.1 (S), Q485.3 (D)
- new net: Q282.1 (S), Q283.3 (D)
- new net: Q174.1 (S), Q175.3 (D)
- new net: Q314.1 (S), Q315.3 (D)
- new net: Q556.1 (S), Q557.3 (D)
- new net: Q260.1 (S), Q261.3 (D)
- new net: Q350.1 (S), Q351.3 (D)
- new net: Q404.1 (S), Q405.3 (D)
- new net: Q310.1 (S), Q311.3 (D)
- new net: Q606.1 (S), Q607.3 (D)
- new net: Q522.1 (S), Q523.3 (D)
- new net: Q572.1 (S), Q573.3 (D)
- new net: Q396.1 (S), Q397.3 (D)
- new net: Q298.1 (S), Q299.3 (D)
- new net: Q254.1 (S), Q255.3 (D)
- new net: Q470.1 (S), Q471.3 (D)
- new net: Q476.1 (S), Q477.3 (D)
- new net: Q442.1 (S), Q443.3 (D)
- new net: Q306.1 (S), Q307.3 (D)
- new net: Q610.1 (S), Q611.3 (D)
- new net: Q374.1 (S), Q375.3 (D)
- new net: Q638.1 (S), Q639.3 (D)
- new net: Q358.1 (S), Q359.3 (D)
- new net: Q182.1 (S), Q183.3 (D)
- new net: Q242.1 (S), Q243.3 (D)
- new net: Q324.1 (S), Q325.3 (D)
- new net: Q330.1 (S), Q331.3 (D)
- new net: Q244.1 (S), Q245.3 (D)
- new net: Q322.1 (S), Q323.3 (D)
- new net: Q518.1 (S), Q519.3 (D)
- new net: Q238.1 (S), Q239.3 (D)
- new net: Q202.1 (S), Q203.3 (D)
- new net: Q422.1 (S), Q423.3 (D)
- new net: Q524.1 (S), Q525.3 (D)
- new net: Q444.1 (S), Q445.3 (D)
- new net: Q332.1 (S), Q333.3 (D)
- new net: Q340.1 (S), Q341.3 (D)
- new net: Q598.1 (S), Q599.3 (D)
- new net: Q508.1 (S), Q509.3 (D)
- new net: Q492.1 (S), Q493.3 (D)
- new net: Q190.1 (S), Q191.3 (D)
- new net: Q426.1 (S), Q427.3 (D)
- new net: Q446.1 (S), Q447.3 (D)
- new net: Q614.1 (S), Q615.3 (D)
- new net: Q266.1 (S), Q267.3 (D)
- new net: Q602.1 (S), Q603.3 (D)
- new net: Q514.1 (S), Q515.3 (D)
- new net: Q554.1 (S), Q555.3 (D)
- new net: Q290.1 (S), Q291.3 (D)
- new net: Q532.1 (S), Q533.3 (D)
- new net: Q172.1 (S), Q173.3 (D)
- new net: Q506.1 (S), Q507.3 (D)
- new net: Q538.1 (S), Q539.3 (D)
- new net: Q564.1 (S), Q565.3 (D)
- new net: Q498.1 (S), Q499.3 (D)
- new net: Q660.1 (S), Q661.3 (D)
- new net: Q540.1 (S), Q541.3 (D)
- new net: Q420.1 (S), Q421.3 (D)
- new net: Q292.1 (S), Q293.3 (D)
- new net: Q230.1 (S), Q231.3 (D)
- new net: Q188.1 (S), Q189.3 (D)
- new net: Q586.1 (S), Q587.3 (D)
- new net: Q356.1 (S), Q357.3 (D)
- new net: Q410.1 (S), Q411.3 (D)
- new net: Q294.1 (S), Q295.3 (D)
- new net: Q676.1 (S), Q677.3 (D)
- new net: Q370.1 (S), Q371.3 (D)
- new net: Q380.1 (S), Q381.3 (D)
- new net: Q636.1 (S), Q637.3 (D)
- new net: Q428.1 (S), Q429.3 (D)
- new net: Q604.1 (S), Q605.3 (D)
- new net: Q438.1 (S), Q439.3 (D)
- new net: Q180.1 (S), Q181.3 (D)
- new net: Q318.1 (S), Q319.3 (D)
- new net: Q590.1 (S), Q591.3 (D)
- new net: Q278.1 (S), Q279.3 (D)
- new net: Q372.1 (S), Q373.3 (D)
- new net: Q236.1 (S), Q237.3 (D)
- new net: Q594.1 (S), Q595.3 (D)
- new net: Q206.1 (S), Q207.3 (D)
- new net: Q316.1 (S), Q317.3 (D)
- new net: Q482.1 (S), Q483.3 (D)
- new net: Q198.1 (S), Q199.3 (D)
- new net: Q346.1 (S), Q347.3 (D)
- new net: Q458.1 (S), Q459.3 (D)
- new net: Q284.1 (S), Q285.3 (D)
- new net: Q348.1 (S), Q349.3 (D)
- new net: Q308.1 (S), Q309.3 (D)
- new net: Q274.1 (S), Q275.3 (D)
- new net: Q666.1 (S), Q667.3 (D)
- new net: Q622.1 (S), Q623.3 (D)
- new net: Q178.1 (S), Q179.3 (D)
- new net: D68.1 (K), Q747.3 (D)
- new net: D28.1 (K), Q707.3 (D)
- new net: Q670.1 (S), Q671.3 (D)
- new net: Q566.1 (S), Q567.3 (D)
- new net: Q662.1 (S), Q663.3 (D)
- new net: Q588.1 (S), Q589.3 (D)
- new net: Q474.1 (S), Q475.3 (D)
- new net: Q650.1 (S), Q651.3 (D)
- new net: Q406.1 (S), Q407.3 (D)
- new net: Q494.1 (S), Q495.3 (D)
- new net: Q562.1 (S), Q563.3 (D)
- new net: Q652.1 (S), Q653.3 (D)
- new net: Q486.1 (S), Q487.3 (D)
- new net: Q101.1 (S), Q102.3 (D)
- new net: Q252.1 (S), Q253.3 (D)
- new net: Q450.1 (S), Q451.3 (D)
- new net: Q546.1 (S), Q547.3 (D)
- new net: Q490.1 (S), Q491.3 (D)
- new net: Q596.1 (S), Q597.3 (D)
- new net: Q186.1 (S), Q187.3 (D)
- new net: D2.1 (K), Q681.3 (D)
- new net: Q214.1 (S), Q215.3 (D)
- new net: Q434.1 (S), Q435.3 (D)
- new net: Q548.1 (S), Q549.3 (D)
- new net: Q250.1 (S), Q251.3 (D)
- new net: Q526.1 (S), Q527.3 (D)
- new net: Q378.1 (S), Q379.3 (D)
- new net: Q642.1 (S), Q643.3 (D)
- new net: Q300.1 (S), Q301.3 (D)
- new net: Q418.1 (S), Q419.3 (D)
- new net: Q210.1 (S), Q211.3 (D)
- new net: Q634.1 (S), Q635.3 (D)
- new net: Q454.1 (S), Q455.3 (D)
- new net: Q194.1 (S), Q195.3 (D)
- new net: Q394.1 (S), Q395.3 (D)
- new net: Q516.1 (S), Q517.3 (D)
- new net: Q268.1 (S), Q269.3 (D)
- new net: Q558.1 (S), Q559.3 (D)
- new net: Q542.1 (S), Q543.3 (D)
- new net: Q530.1 (S), Q531.3 (D)
- new net: Q468.1 (S), Q469.3 (D)
- new net: Q226.1 (S), Q227.3 (D)
- new net: Q570.1 (S), Q571.3 (D)
- new net: D10.1 (K), Q689.3 (D)
- new net: Q644.1 (S), Q645.3 (D)
- new net: Q628.1 (S), Q629.3 (D)
- new net: Q626.1 (S), Q627.3 (D)
- new net: Q658.1 (S), Q659.3 (D)
- new net: D57.1 (K), Q736.3 (D)
- new net: Q630.1 (S), Q631.3 (D)
- new net: Q342.1 (S), Q343.3 (D)
- new net: Q620.1 (S), Q621.3 (D)
- new net: Q270.1 (S), Q271.3 (D)
- new net: Q578.1 (S), Q579.3 (D)
- new net: Q258.1 (S), Q259.3 (D)
- new net: Q366.1 (S), Q367.3 (D)
- new net: Q382.1 (S), Q383.3 (D)
- new net: Q618.1 (S), Q619.3 (D)
- new net: Q196.1 (S), Q197.3 (D)
- new net: Q466.1 (S), Q467.3 (D)
- new net: D20.1 (K), Q699.3 (D)
- new net: Q218.1 (S), Q219.3 (D)
Other:
- note added: "Cell: 2N7000 + 47k pull-up (NMOS, see docs/gate-cell.md). 747 transistors, 287 resistors, 68 LEDs. From the bus header: BUS3#..BUS0# (an address while MAI, data while MI), MAI, MI, MO, CLK. To the bus: BUS3#..BUS0# driven (open drain) with the addressed slot while MO. The address register is four transparent latches open while MAI and PH1 (S3 of a memory instruction, when B or the operand is on t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"
- note added: "TWO-PHASE CLOCK: only PH1 is used here, to close the address latches and end the write before the rising edge"
- note added: "WORD LINES: WRn = slot n AND MI AND PH1 (write, ends at the clock edge), RDn = slot n AND MO (read)"
- note removed: "Cell: 2N7000 + 47k pull-up (NMOS, see docs/gate-cell.md). 746 transistors, 287 resistors, 68 LEDs. From the bus header: BUS3#..BUS0# (an address while MAI, data while MI), MAI, MI, MO, CLK. To the bus: BUS3#..BUS0# driven (open drain) with the addressed slot while MO. The address register is four transparent latches open while MAI and PH1 (S3 of a memory instruction, when B or the operand is on t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"
- note removed: "TWO-PHASE CLOCK: only PH1 is used here, to close the address latches before the rising edge"
- note removed: "WORD LINES: WRn = slot n AND MI (write), RDn = slot n AND MO (read)"
