File: boards/03-sequencer/sequencer.kicad_sch (KiCad schematic)
At the start: 932 parts, among them J1 BUS, J2 LINK, Q1 2N7000, Q10 2N7000, Q100 2N7000, Q101 2N7000, Q102 2N7000, Q103 2N7000, Q104 2N7000, Q105 2N7000, Q106 2N7000, Q107 2N7000, Q108 2N7000, Q109 2N7000, Q11 2N7000, Q110 2N7000, Q111 2N7000, Q112 2N7000, Q113 2N7000, Q114 2N7000, Q115 2N7000, Q116 2N7000, Q117 2N7000, Q118 2N7000, Q119 2N7000, Q12 2N7000, Q120 2N7000, Q121 2N7000, Q122 2N7000, Q123 2N7000, Q124 2N7000, Q125 2N7000, Q126 2N7000, Q127 2N7000, Q128 2N7000, Q129 2N7000, Q13 2N7000, Q130 2N7000, Q131 2N7000, Q132 2N7000, Q133 2N7000, Q134 2N7000, Q135 2N7000, Q136 2N7000, Q137 2N7000, Q138 2N7000, Q139 2N7000, Q14 2N7000, Q140 2N7000, Q141 2N7000, Q142 2N7000, Q143 2N7000, Q144 2N7000, Q145 2N7000, Q146 2N7000, Q147 2N7000, Q148 2N7000, Q149 2N7000, Q15 2N7000, Q150 2N7000, Q151 2N7000, Q152 2N7000, Q153 2N7000, Q154 2N7000, Q155 2N7000, Q156 2N7000, Q157 2N7000, Q158 2N7000, Q159 2N7000, Q16 2N7000, Q160 2N7000, Q161 2N7000, Q162 2N7000, Q163 2N7000, Q164 2N7000, Q165 2N7000, Q166 2N7000, Q167 2N7000, Q168 2N7000, Q169 2N7000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

Commit message: Sequencer: buffered matrix columns (D041); S4 rows and pads at every crossing (D040)
list.asm at MIX seeds 2 and 3 failed on the whole machine: a control line
falls only through its 1 Meg column pull-down into every board's gates
and the ribbons, 350 to 440 us to 1 V bare and 800 us with cables, most
of a tick, so a register mux sat half open across a clock edge. Each
column's diode node now feeds one inverter and a second inverter (22k)
drives the line. 46 transistors.

The matrix draws a diode at every crossing, DNP where the design has
none, so the pads are on the board; the eight free opcodes get S4 rows;
row pitch 2.54 mm; the pull-downs' GND rail moved beside them (it ran
through their signal pads, DRC caught the short). BOM and position file
exclude DNP. ERC clean; the export has 83 diodes and 586 transistors.
Machine gate on the new sequencer not yet run (list MIX3 in progress).

Co-Authored-By: Claude Fable 5.1 <noreply@anthropic.com>
Claude-Session: https://claude.ai/code/session_019vcbW37ERmrjZaWq55Er3J
Parts:
- added D1000, D1001, D1002, D1003, D1004, D1005, D1006, D1007, D1008, D1009, D1010, D1011, D1012, D1013, D1014, D1015, D1016, D1017, D1018, D1019, D1020, D1021, D1022, D1023, D1024, D1025, D1026, D1027, D1028, D1029, D103, D1030, D1031, D1032, D1033, D1034, D1035, D1036, D1037, D1038, D1039, D104, D1040, D1041, D1042, D1043, D1044, D1045, D1046, D1047, D1048, D1049, D105, D1050, D1051, D1052, D1053, D1054, D106, D107, D108, D109, D110, D111, D112, D113, D114, D115, D116, D117, D118, D119, D120, D121, D122, D123, D124, D125, D126, D127, D128, D129, D130, D131, D132, D133, D134, D135, D136, D137, D138, D139, D140, D141, D142, D143, D144, D145, D146, D147, D148, D149, D150, D151, D152, D153, D154, D155, D156, D157, D158, D159, D160, D161, D162, D163, D164, D165, D166, D167, D168, D169, D170, D171, D172, D173, D174, D175, D176, D177, D178, D179, D180, D181, D182, D183, D184, D185, D186, D187, D188, D189, D190, D191, D192, D193, D194, D195, D196, D197, D198, D199, D200, D201, D202, D203, D204, D205, D206, D207, D208, D209, D210, D211, D212, D213, D214, D215, D216, D217, D218, D219, D220, D221, D222, D223, D224, D225, D226, D227, D228, D229, D230, D231, D232, D233, D234, D235, D236, D237, D238, D239, D240, D241, D242, D243, D244, D245, D246, D247, D248, D249, D250, D251, D252, D253, D254, D255, D256, D257, D258, D259, D260, D261, D262, D263, D264, D265, D266, D267, D268, D269, D270, D271, D272, D273, D274, D275, D276, D277, D278, D279, D280, D281, D282, D283, D284, D285, D286, D287, D288, D289, D290, D291, D292, D293, D294, D295, D296, D297, D298, D299, D300, D301, D302, D303, D304, D305, D306, D307, D308, D309, D310, D311, D312, D313, D314, D315, D316, D317, D318, D319, D320, D321, D322, D323, D324, D325, D326, D327, D328, D329, D330, D331, D332, D333, D334, D335, D336, D337, D338, D339, D340, D341, D342, D343, D344, D345, D346, D347, D348, D349, D350, D351, D352, D353, D354, D355, D356, D357, D358, D359, D360, D361, D362, D363, D364, D365, D366, D367, D368, D369, D370, D371, D372, D373, D374, D375, D376, D377, D378, D379, D380, D381, D382, D383, D384, D385, D386, D387, D388, D389, D390, D391, D392, D393, D394, D395, D396, D397, D398, D399, D400, D401, D402, D403, D404, D405, D406, D407, D408, D409, D410, D411, D412, D413, D414, D415, D416, D417, D418, D419, D420, D421, D422, D423, D424, D425, D426, D427, D428, D429, D430, D431, D432, D433, D434, D435, D436, D437, D438, D439, D440, D441, D442, D443, D444, D445, D446, D447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: 1N4148, Diode_THT:D_DO-35_SOD27_P7.62mm_Horizontal, symbol Device:D
- added Q525, Q526, Q527, Q528, Q529, Q530, Q531, Q532, Q533, Q534, Q535, Q536, Q537, Q538, Q539, Q540, Q541, Q542, Q543, Q544, Q545, Q546, Q547, Q548, Q549, Q550, Q551, Q552, Q553, Q554, Q555, Q556, Q557, Q558, Q559, Q560, Q561, Q562, Q563, Q564, Q565, Q566, Q567, Q568, Q569, Q570, Q571, Q572, Q573, Q574, Q575, Q576, Q577, Q578, Q579, Q580, Q581, Q582, Q583, Q584, Q585, Q586: 2N7000, Package_TO_SOT_THT:TO-92_Inline_Wide, symbol Transistor_FET:2N7000
- added R299, R300, R301, R302, R303, R304, R305, R306, R307, R308, R309, R310: 47k, Resistor_THT:R_Axial_DIN0207_L6.3mm_D2.5mm_P5.08mm_Vertical, symbol Device:R
- added R311, R312, R313, R314, R315, R316, R317, R318, R319, R320, R321, R322, R323, R324, R325, R326, R327, R328, R329: 1k, Resistor_THT:R_Axial_DIN0207_L6.3mm_D2.5mm_P5.08mm_Vertical, symbol Device:R
- added R330, R331, R332, R333, R334, R335, R336, R337, R338, R339, R340, R341, R342, R343, R344, R345, R346, R347, R348, R349, R350, R351, R352: 1Meg, Resistor_THT:R_Axial_DIN0207_L6.3mm_D2.5mm_P5.08mm_Vertical, symbol Device:R
- D100, D101, D102, D20, D21, D22, D23, D24, D25, D26, D27, D28, D29, D30, D31, D32, D33, D34, D35, D36, D37, D38, D39, D40, D41, D43, D44, D45, D46, D47, D48, D50, D51, D52, D53, D54, D55, D56, D57, D58, D59, D60, D61, D62, D63, D64, D66, D67, D68, D69, D70, D71, D74, D75, D76, D77, D78, D79, D80, D81, D82, D83, D84, D85, D86, D87, D89, D92, D93, D94, D95, D96, D97, D98: now not fitted; now left out of the parts list
- R245, R246, R247, R248, R249, R250, R251, R252, R67: value 47k -> 10k
- R254, R256: value 47k -> 22k
- R257, R259, R261, R263, R265, R267, R269, R271, R273, R275: value 1k -> 47k
- R258, R260, R262, R264, R266, R268, R270, R272, R274: value 1k -> 22k
- R276, R278, R280, R282, R284, R286, R288, R290, R292, R294, R296, R298: value 1Meg -> 22k
- R277, R279, R281, R283, R285, R287, R289, R291, R293, R295, R297: value 1Meg -> 47k
Connections:
- net +5V: now also R276.1, R277.1, R278.1, R279.1, R280.1, R281.1, R282.1, R283.1, R284.1, R285.1, R286.1, R287.1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
- net AB: now also Q516.3 (D), R268.2; no longer D24.1 (K), R283.1
- net AI: now also Q506.3 (D), R258.2; no longer D27.1 (K), D32.1 (K), D41.1 (K), D46.1 (K), D52.1 (K), D60.1 (K), D66.1 (K), D71.1 (K), D76.1 (K), D81.1 (K), D90.1 (K), R278.1
- net AO: now also Q508.3 (D), R260.2; no longer D35.1 (K), D57.1 (K), D95.1 (K), R279.1
- net BA: now also Q514.3 (D), R266.2; no longer D21.1 (K), D23.1 (K), R282.1
- net BI: now also Q510.3 (D), R262.2; no longer R280.1
- net BO: now also Q512.3 (D), R264.2; no longer D50.1 (K), D55.1 (K), R281.1
- net BUS0#: now also Q555.3 (D); no longer Q493.3 (D)
- net BUS1#: now also Q559.3 (D); no longer Q497.3 (D)
- net BUS2#: now also Q563.3 (D); no longer Q501.3 (D)
- net BUS3#: now also Q567.3 (D); no longer Q505.3 (D)
- net CFQ: now also Q585.2 (G); no longer Q523.2 (G)
- net CFQ_qn: now also Q497.2 (G); no longer Q481.2 (G)
- net DONE: now also R298.2, Q546.3 (D); no longer D100.1 (K), D20.1 (K), D22.1 (K), D25.1 (K), D29.1 (K), D34.1 (K), D37.1 (K), D44.1 (K), D49.1 (K), D54.1 (K), D59.1 (K), D62.1 (K)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
- net EO: now also Q504.3 (D), R256.2; no longer D26.1 (K), D31.1 (K), D40.1 (K), D45.1 (K), D65.1 (K), D70.1 (K), D75.1 (K), R277.1
- net F0: now also R286.2, Q534.3 (D); no longer D68.1 (K), D78.1 (K), R292.1
- net F1: now also R288.2, Q536.3 (D); no longer D73.1 (K), D79.1 (K), R293.1
- net FI: now also Q522.3 (D), R274.2; no longer D28.1 (K), D33.1 (K), D42.1 (K), D47.1 (K), D67.1 (K), D72.1 (K), D77.1 (K), R286.1
- net GND: now also Q490.1 (S), Q494.1 (S), Q498.1 (S), Q502.1 (S), Q525.1 (S), Q526.1 (S), Q527.1 (S), Q528.1 (S), Q529.1 (S), Q530.1 (S), Q531.1 (S), Q532.1 (S)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; no longer R276.2, R277.2, R278.2, R279.2, R280.2, R281.2, R282.2, R283.2, R284.2, R285.2, R286.2, R287.2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
- net HLT: now also Q524.3 (D), R276.2; no longer D38.1 (K), R287.1
- net II: now also Q548.3 (D), R300.2; no longer Q486.3 (D), R246.2
- net IIN: now also Q547.3 (D), Q548.2 (G), R299.2; no longer Q485.3 (D), Q486.2 (G), R245.2
- net INP: now also R290.2, Q538.3 (D); no longer D61.1 (K), R294.1
- net IO: now also Q520.3 (D), R272.2, Q552.2 (G), Q556.2 (G), Q560.2 (G), Q564.2 (G); no longer D82.1 (K), D88.1 (K), D93.1 (K), Q490.2 (G), Q494.2 (G), Q498.2 (G), Q502.2 (G), R285.1
- net IOD0: now also Q554.3 (D), Q555.2 (G), R304.2; no longer Q492.3 (D), Q493.2 (G), R250.2
- net IOD0N: now also Q552.3 (D), Q554.2 (G), R303.2; no longer Q490.3 (D), Q492.2 (G), R249.2
- net IOD1: now also Q558.3 (D), Q559.2 (G), R306.2; no longer Q496.3 (D), Q497.2 (G), R252.2
- net IOD1N: now also Q556.3 (D), Q558.2 (G), R305.2; no longer Q494.3 (D), Q496.2 (G), R251.2
- net IOD2: now also Q562.3 (D), Q563.2 (G), R308.2; no longer Q500.3 (D), Q501.2 (G), R254.2
- net IOD2N: now also Q560.3 (D), Q562.2 (G), R307.2; no longer Q498.3 (D), Q500.2 (G), R253.2
- net IOD3: now also Q566.3 (D), Q567.2 (G), R310.2; no longer Q504.3 (D), Q505.2 (G), R256.2
- net IOD3N: now also Q564.3 (D), Q566.2 (G), R309.2; no longer Q502.3 (D), Q504.2 (G), R255.2
- net IR0: now also Q576.2 (G); no longer Q514.2 (G)
- net IR1: now also Q575.2 (G); no longer Q513.2 (G)
- net IR2: now also Q574.2 (G); no longer Q512.2 (G)
- net IR3: now also Q573.2 (G); no longer Q511.2 (G)
- net MAI: now also R278.2, Q526.3 (D); no longer D51.1 (K), D56.1 (K), D89.1 (K), D94.1 (K), R288.1
- net MI: now also R280.2, Q528.3 (D); no longer D58.1 (K), D96.1 (K), R289.1
- net MO: now also R282.2, Q530.3 (D); no longer D53.1 (K), D91.1 (K), R290.1
- net OI: now also Q518.3 (D), R270.2; no longer D36.1 (K), R284.1
- net ONE: now also R284.2, Q532.3 (D); no longer D43.1 (K), D48.1 (K), R291.1
- net OP10#: now also Q471.2 (G), Q473.2 (G); no longer Q467.2 (G)
- net OP11#: now also Q475.2 (G), Q477.2 (G); no longer Q469.2 (G)
- net OP12#: now also Q479.2 (G), Q481.2 (G); no longer Q471.2 (G)
- net OP13#: now also Q483.2 (G), Q485.2 (G); no longer Q473.2 (G)
- net OP14#: now also Q487.2 (G), Q489.2 (G); no longer Q475.2 (G)
- net OP15#: now also Q491.2 (G), Q493.2 (G); no longer Q477.2 (G)
- net OP3#: now also Q495.2 (G); no longer Q479.2 (G)
- net OP4#: now also Q498.2 (G); no longer Q482.2 (G)
- net OP8#: now also Q465.2 (G)
- net OP9#: now also Q467.2 (G), Q469.2 (G); no longer Q465.2 (G)
- net OPR0: now also Q553.2 (G), Q584.2 (G); no longer Q491.2 (G), Q522.2 (G)
- net OPR1: now also Q557.2 (G), Q583.2 (G); no longer Q495.2 (G), Q521.2 (G)
- net OPR2: now also Q561.2 (G), Q582.2 (G); no longer Q499.2 (G), Q520.2 (G)
- net OPR3: now also Q565.2 (G), Q581.2 (G); no longer Q503.2 (G), Q519.2 (G)
- net OPR4: now also Q580.2 (G); no longer Q518.2 (G)
- net OPR5: now also Q579.2 (G); no longer Q517.2 (G)
- net OPR6: now also Q578.2 (G); no longer Q516.2 (G)
- net OPR7: now also Q577.2 (G); no longer Q515.2 (G)
- net PCE: now also Q551.3 (D), R302.2; no longer Q489.3 (D), R248.2
- net PCEN: now also Q549.3 (D), Q550.3 (D), Q551.2 (G), R301.2; no longer Q487.3 (D), Q488.3 (D), Q489.2 (G), R247.2
- net PCL: now also R292.2, Q540.3 (D); no longer D101.1 (K), D102.1 (K), D84.1 (K), D98.1 (K), R295.1
- net PCR: now also R294.2, Q542.3 (D); no longer D63.1 (K), R296.1
- net RAI: now also R296.2, Q544.3 (D); no longer D99.1 (K), R297.1
- net R_F0_3: now also D21.2 (A), D22.2 (A), D23.2 (A), D24.2 (A), D25.2 (A), D26.2 (A), D27.2 (A), D28.2 (A), D29.2 (A), D30.2 (A), D31.2 (A), D32.2 (A)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
- net R_F10_3: now also D273.2 (A), D274.2 (A), D275.2 (A), D276.2 (A), D277.2 (A), D278.2 (A), D279.2 (A), D280.2 (A), D281.2 (A), D282.2 (A), D283.2 (A), D284.2 (A)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; no longer D55.2 (A), D56.2 (A)
- net R_F10_4: now also D296.2 (A), D297.2 (A), D298.2 (A), D299.2 (A), D300.2 (A), D301.2 (A), D302.2 (A), D303.2 (A), D304.2 (A), D305.2 (A), D306.2 (A), D307.2 (A)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; no longer D57.2 (A), D58.2 (A), D59.2 (A)
- net R_F11_3: now also D319.2 (A), D320.2 (A), D321.2 (A), D322.2 (A), D323.2 (A), D324.2 (A), D325.2 (A), D326.2 (A), D327.2 (A), D328.2 (A), D329.2 (A), D330.2 (A)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; no longer D60.2 (A), D61.2 (A), D62.2 (A)
- net R_F12_3: now also D342.2 (A), D343.2 (A), D344.2 (A), D345.2 (A), D346.2 (A), D347.2 (A), D348.2 (A), D349.2 (A), D350.2 (A), D351.2 (A), D352.2 (A), D353.2 (A)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; no longer D63.2 (A), D64.2 (A)
- net R_F13_3: now also D365.2 (A), D366.2 (A), D367.2 (A), D368.2 (A), D369.2 (A), D370.2 (A), D371.2 (A), D372.2 (A), D373.2 (A), D374.2 (A), D375.2 (A), D376.2 (A)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; no longer D65.2 (A), D66.2 (A), D67.2 (A), D68.2 (A), D69.2 (A)
- net R_F14_3: now also D388.2 (A), D389.2 (A), D390.2 (A), D391.2 (A), D392.2 (A), D393.2 (A), D394.2 (A), D395.2 (A), D396.2 (A), D397.2 (A), D398.2 (A), D399.2 (A)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; no longer D70.2 (A), D71.2 (A), D72.2 (A), D73.2 (A), D74.2 (A)
- net R_F15_3: now also D411.2 (A), D412.2 (A), D413.2 (A), D414.2 (A), D415.2 (A), D416.2 (A), D417.2 (A), D418.2 (A), D419.2 (A), D420.2 (A), D421.2 (A), D422.2 (A)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; no longer D75.2 (A), D76.2 (A), D77.2 (A), D78.2 (A), D79.2 (A), D80.2 (A)
- net R_F1_3: now also D43.2 (A), D44.2 (A), D45.2 (A), D46.2 (A), D47.2 (A), D48.2 (A), D49.2 (A), D50.2 (A), D51.2 (A), D52.2 (A), D53.2 (A), D54.2 (A)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; no longer D21.2 (A), D22.2 (A)
- net R_F2_3: now also D66.2 (A), D67.2 (A), D68.2 (A), D69.2 (A), D70.2 (A), D71.2 (A), D72.2 (A), D73.2 (A), D74.2 (A), D75.2 (A), D76.2 (A), D77.2 (A)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; no longer D23.2 (A), D24.2 (A), D25.2 (A)
- net R_F3_3: now also D100.2 (A), D101.2 (A), D102.2 (A), D89.2 (A), D90.2 (A), D91.2 (A), D92.2 (A), D93.2 (A), D94.2 (A), D95.2 (A), D96.2 (A), D97.2 (A)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; no longer D26.2 (A), D27.2 (A), D28.2 (A), D29.2 (A)
- net R_F4_3: now also D112.2 (A), D113.2 (A), D114.2 (A), D115.2 (A), D116.2 (A), D117.2 (A), D118.2 (A), D119.2 (A), D120.2 (A), D121.2 (A), D122.2 (A), D123.2 (A)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; no longer D30.2 (A), D31.2 (A), D32.2 (A), D33.2 (A), D34.2 (A)
- net R_F5_3: now also D135.2 (A), D136.2 (A), D137.2 (A), D138.2 (A), D139.2 (A), D140.2 (A), D141.2 (A), D142.2 (A), D143.2 (A), D144.2 (A), D145.2 (A), D146.2 (A)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; no longer D35.2 (A), D36.2 (A), D37.2 (A)
- net R_F6_3: now also D158.2 (A), D159.2 (A), D160.2 (A), D161.2 (A), D162.2 (A), D163.2 (A), D164.2 (A), D165.2 (A), D166.2 (A), D167.2 (A), D168.2 (A), D169.2 (A)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; no longer D38.2 (A)
- net R_F7_3: now also D181.2 (A), D182.2 (A), D183.2 (A), D184.2 (A), D185.2 (A), D186.2 (A), D187.2 (A), D188.2 (A), D189.2 (A), D190.2 (A), D191.2 (A), D192.2 (A)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; no longer D39.2 (A), D40.2 (A), D41.2 (A), D42.2 (A), D43.2 (A), D44.2 (A)
- net R_F8_3: now also D204.2 (A), D205.2 (A), D206.2 (A), D207.2 (A), D208.2 (A), D209.2 (A), D210.2 (A), D211.2 (A), D212.2 (A), D213.2 (A), D214.2 (A), D215.2 (A)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; no longer D45.2 (A), D46.2 (A), D47.2 (A), D48.2 (A), D49.2 (A)
- net R_F9_3: now also D227.2 (A), D228.2 (A), D229.2 (A), D230.2 (A), D231.2 (A), D232.2 (A), D233.2 (A), D234.2 (A), D235.2 (A), D236.2 (A), D237.2 (A), D238.2 (A)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; no longer D50.2 (A), D51.2 (A)
- net R_F9_4: now also D250.2 (A), D251.2 (A), D252.2 (A), D253.2 (A), D254.2 (A), D255.2 (A), D256.2 (A), D257.2 (A), D258.2 (A), D259.2 (A), D260.2 (A), D261.2 (A)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; no longer D52.2 (A), D53.2 (A), D54.2 (A)
- net R_JCC: now also Q495.3 (D), Q496.3 (D), Q497.3 (D), R251.2, D1009.2 (A), D1010.2 (A), D1011.2 (A), D1012.2 (A), D1013.2 (A), D1014.2 (A), D1015.2 (A), D1016.2 (A)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; no longer D101.2 (A), Q479.3 (D), Q480.3 (D), Q481.3 (D), R243.2
- net R_JZZ: now also Q498.3 (D), Q499.3 (D), Q500.3 (D), R252.2, D1032.2 (A), D1033.2 (A), D1034.2 (A), D1035.2 (A), D1036.2 (A), D1037.2 (A), D1038.2 (A), D1039.2 (A)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; no longer D102.2 (A), Q482.3 (D), Q483.3 (D), Q484.3 (D), R244.2
- net R_OP10_3: now also Q471.3 (D), Q472.3 (D), R239.2, D733.2 (A), D734.2 (A), D735.2 (A), D736.2 (A), D737.2 (A), D738.2 (A), D739.2 (A), D740.2 (A), D741.2 (A)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; no longer Q467.3 (D), Q468.3 (D), R237.2
- net R_OP11_3: now also Q475.3 (D), Q476.3 (D), R241.2, D779.2 (A), D780.2 (A), D781.2 (A), D782.2 (A), D783.2 (A), D784.2 (A), D785.2 (A), D786.2 (A), D787.2 (A)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; no longer Q469.3 (D), Q470.3 (D), R238.2
- net R_OP12_3: now also Q479.3 (D), Q480.3 (D), R243.2, D825.2 (A), D826.2 (A), D827.2 (A), D828.2 (A), D829.2 (A), D830.2 (A), D831.2 (A), D832.2 (A), D833.2 (A)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; no longer Q471.3 (D), Q472.3 (D), R239.2
- net R_OP13_3: now also Q483.3 (D), Q484.3 (D), R245.2, D871.2 (A), D872.2 (A), D873.2 (A), D874.2 (A), D875.2 (A), D876.2 (A), D877.2 (A), D878.2 (A), D879.2 (A)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; no longer Q473.3 (D), Q474.3 (D), R240.2
- net R_OP14_3: now also Q487.3 (D), Q488.3 (D), R247.2, D917.2 (A), D918.2 (A), D919.2 (A), D920.2 (A), D921.2 (A), D922.2 (A), D923.2 (A), D924.2 (A), D925.2 (A)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; no longer Q475.3 (D), Q476.3 (D), R241.2
- net R_OP15_3: now also Q491.3 (D), Q492.3 (D), R249.2, D963.2 (A), D964.2 (A), D965.2 (A), D966.2 (A), D967.2 (A), D968.2 (A), D969.2 (A), D970.2 (A), D971.2 (A)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; no longer Q477.3 (D), Q478.3 (D), R242.2
- net R_OP1_3: now also D434.2 (A), D435.2 (A), D436.2 (A), D437.2 (A), D438.2 (A), D439.2 (A), D440.2 (A), D441.2 (A), D442.2 (A), D443.2 (A), D444.2 (A), D445.2 (A)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; no longer D81.2 (A), D82.2 (A), D83.2 (A)
- net R_OP2_3: now also D457.2 (A), D458.2 (A), D459.2 (A), D460.2 (A), D461.2 (A), D462.2 (A), D463.2 (A), D464.2 (A), D465.2 (A), D466.2 (A), D467.2 (A), D468.2 (A)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; no longer D84.2 (A), D85.2 (A)
- net R_OP3_3: now also D480.2 (A), D481.2 (A), D482.2 (A), D483.2 (A), D484.2 (A), D485.2 (A), D486.2 (A), D487.2 (A), D488.2 (A), D489.2 (A), D490.2 (A), D491.2 (A)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; no longer D86.2 (A)
- net R_OP4_3: now also D503.2 (A), D504.2 (A), D505.2 (A), D506.2 (A), D507.2 (A), D508.2 (A), D509.2 (A), D510.2 (A), D511.2 (A), D512.2 (A), D513.2 (A), D514.2 (A)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; no longer D87.2 (A)
- net R_OP5_3: now also D526.2 (A), D527.2 (A), D528.2 (A), D529.2 (A), D530.2 (A), D531.2 (A), D532.2 (A), D533.2 (A), D534.2 (A), D535.2 (A), D536.2 (A), D537.2 (A)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; no longer D88.2 (A), D89.2 (A)
- net R_OP5_4: now also D549.2 (A), D550.2 (A), D551.2 (A), D552.2 (A), D553.2 (A), D554.2 (A), D555.2 (A), D556.2 (A), D557.2 (A), D558.2 (A), D559.2 (A), D560.2 (A)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; no longer D90.2 (A), D91.2 (A), D92.2 (A)
- net R_OP6_3: now also D572.2 (A), D573.2 (A), D574.2 (A), D575.2 (A), D576.2 (A), D577.2 (A), D578.2 (A), D579.2 (A), D580.2 (A), D581.2 (A), D582.2 (A), D583.2 (A)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; no longer D93.2 (A), D94.2 (A)
- net R_OP6_4: now also D595.2 (A), D596.2 (A), D597.2 (A), D598.2 (A), D599.2 (A), D600.2 (A), D601.2 (A), D602.2 (A), D603.2 (A), D604.2 (A), D605.2 (A), D606.2 (A)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; no longer D95.2 (A), D96.2 (A), D97.2 (A)
- net R_OP7_3: now also D618.2 (A), D619.2 (A), D620.2 (A), D621.2 (A), D622.2 (A), D623.2 (A), D624.2 (A), D625.2 (A), D626.2 (A), D627.2 (A), D628.2 (A), D629.2 (A)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; no longer D100.2 (A), D98.2 (A), D99.2 (A)
- net R_OP8_3: now also D641.2 (A), D642.2 (A), D643.2 (A), D644.2 (A), D645.2 (A), D646.2 (A), D647.2 (A), D648.2 (A), D649.2 (A), D650.2 (A), D651.2 (A), D652.2 (A)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
- net R_OP9_3: now also Q467.3 (D), Q468.3 (D), R237.2, D687.2 (A), D688.2 (A), D689.2 (A), D690.2 (A), D691.2 (A), D692.2 (A), D693.2 (A), D694.2 (A), D695.2 (A)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; no longer Q465.3 (D), Q466.3 (D), R236.2
- net SUB: now also Q502.3 (D), R254.2; no longer D30.1 (K), D39.1 (K), R276.1
- net T0: now also Q547.2 (G), Q568.2 (G); no longer Q485.2 (G), Q506.2 (G)
- net T1: now also Q549.2 (G), Q569.2 (G); no longer Q487.2 (G), Q507.2 (G)
- net T2: now also Q550.2 (G), Q570.2 (G); no longer Q488.2 (G), Q508.2 (G)
- net T3: now also Q571.2 (G); no longer Q509.2 (G)
- net T3N: now also Q496.2 (G), Q499.2 (G); no longer Q480.2 (G), Q483.2 (G)
- net T3NB: now also Q480.2 (G), Q484.2 (G), Q488.2 (G), Q492.2 (G); no longer Q466.2 (G), Q470.2 (G), Q474.2 (G), Q478.2 (G)
- net T4: now also Q572.2 (G); no longer Q510.2 (G)
- net T4N: now also Q466.2 (G), Q470.2 (G), Q474.2 (G), Q478.2 (G), Q482.2 (G), Q486.2 (G), Q490.2 (G), Q494.2 (G)
- net ZFQ: now also Q586.2 (G); no longer Q524.2 (G)
- net ZFQ_qn: now also Q500.2 (G); no longer Q484.2 (G)
- net at D12.1 (K): now also Q579.3 (D); no longer Q517.3 (D)
- net at D12.2 (A): now also R322.2; no longer R268.2
- net at D15.1 (K): now also Q582.3 (D); no longer Q520.3 (D)
- net at D17.1 (K): now also Q584.3 (D); no longer Q522.3 (D)
- net at D17.2 (A): now also R327.2; no longer R273.2
- net at D8.1 (K): now also Q575.3 (D); no longer Q513.3 (D)
- net at D4.1 (K): now also Q571.3 (D); no longer Q509.3 (D)
- net at D4.2 (A): now also R314.2; no longer R260.2
- net at D14.1 (K): now also Q581.3 (D); no longer Q519.3 (D)
- net at D2.1 (K): now also Q569.3 (D); no longer Q507.3 (D)
- net at D2.2 (A): now also R312.2; no longer R258.2
- net at D14.2 (A): now also R324.2; no longer R270.2
- net EO_mn: now reaches Q503.3 (D)
- net EO_mn: now also Q504.2 (G), R255.2; no longer Q502.1 (S)
- net at D3.2 (A): now also R313.2; no longer R259.2
- net at D1.2 (A): now also R311.2; no longer R257.2
- net at D7.1 (K): now also Q574.3 (D); no longer Q512.3 (D)
- net at D7.2 (A): now also R317.2; no longer R263.2
- net at D3.1 (K): now also Q570.3 (D); no longer Q508.3 (D)
- net at D6.1 (K): now also Q573.3 (D); no longer Q511.3 (D)
- net at D18.2 (A): now also R328.2; no longer R274.2
- net at D16.1 (K): now also Q583.3 (D); no longer Q521.3 (D)
- net at D16.2 (A): now also R326.2; no longer R272.2
- net at D9.2 (A): now also R319.2; no longer R265.2
- net at D11.2 (A): now also R321.2; no longer R267.2
- net at D1.1 (K): now also Q568.3 (D); no longer Q506.3 (D)
- net at D5.1 (K): now also Q572.3 (D); no longer Q510.3 (D)
- net at D5.2 (A): now also R315.2; no longer R261.2
- net at D15.2 (A): now also R325.2; no longer R271.2
- net at D19.2 (A): now also R329.2; no longer R275.2
- net at D10.1 (K): now also Q577.3 (D); no longer Q515.3 (D)
- net at D10.2 (A): now also R320.2; no longer R266.2
- net at D6.2 (A): now also R316.2; no longer R262.2
- net at D13.2 (A): now also R323.2; no longer R269.2
- net at D18.1 (K): now also Q585.3 (D); no longer Q523.3 (D)
- net at D8.2 (A): now also R318.2; no longer R264.2
- net at D13.1 (K): now also Q580.3 (D); no longer Q518.3 (D)
- net at D9.1 (K): now also Q576.3 (D); no longer Q514.3 (D)
- net at D19.1 (K): now also Q586.3 (D); no longer Q524.3 (D)
- net at D11.1 (K): now also Q578.3 (D); no longer Q516.3 (D)
- new net: Q564.1 (S), Q565.3 (D)
- new net: Q560.1 (S), Q561.3 (D)
- new net: Q556.1 (S), Q557.3 (D)
- new net: Q552.1 (S), Q553.3 (D)
- new net AB_m: D1016.1 (K), D1039.1 (K), D119.1 (K), D142.1 (K), D165.1 (K), D188.1 (K), D211.1 (K), D234.1 (K), D257.1 (K), D27.1 (K), D280.1 (K), D303.1 (K)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
- new net AB_mn: Q515.3 (D), Q516.2 (G), R267.2
- new net AI_m: D1011.1 (K), D1034.1 (K), D114.1 (K), D137.1 (K), D160.1 (K), D183.1 (K), D206.1 (K), D22.1 (K), D229.1 (K), D252.1 (K), D275.1 (K), D298.1 (K)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
- new net AI_mn: Q505.3 (D), Q506.2 (G), R257.2
- new net AO_m: D1012.1 (K), D1035.1 (K), D115.1 (K), D138.1 (K), D161.1 (K), D184.1 (K), D207.1 (K), D23.1 (K), D230.1 (K), D253.1 (K), D276.1 (K), D299.1 (K)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
- new net AO_mn: Q507.3 (D), Q508.2 (G), R259.2
- new net BA_m: D1015.1 (K), D1038.1 (K), D118.1 (K), D141.1 (K), D164.1 (K), D187.1 (K), D210.1 (K), D233.1 (K), D256.1 (K), D26.1 (K), D279.1 (K), D302.1 (K)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
- new net BA_mn: Q513.3 (D), Q514.2 (G), R265.2
- new net BI_m: D1013.1 (K), D1036.1 (K), D116.1 (K), D139.1 (K), D162.1 (K), D185.1 (K), D208.1 (K), D231.1 (K), D24.1 (K), D254.1 (K), D277.1 (K), D300.1 (K)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
- new net BI_mn: Q509.3 (D), Q510.2 (G), R261.2
- new net BO_m: D1014.1 (K), D1037.1 (K), D117.1 (K), D140.1 (K), D163.1 (K), D186.1 (K), D209.1 (K), D232.1 (K), D25.1 (K), D255.1 (K), D278.1 (K), D301.1 (K)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
- new net BO_mn: Q511.3 (D), Q512.2 (G), R263.2
- new net DONE_m: D1008.1 (K), D1031.1 (K), D1054.1 (K), D111.1 (K), D134.1 (K), D157.1 (K), D180.1 (K), D203.1 (K), D226.1 (K), D249.1 (K), D272.1 (K), D295.1 (K)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
- new net DONE_mn: Q545.3 (D), Q546.2 (G), R297.2
- new net EO_m: D1010.1 (K), D1033.1 (K), D113.1 (K), D136.1 (K), D159.1 (K), D182.1 (K), D205.1 (K), D21.1 (K), D228.1 (K), D251.1 (K), D274.1 (K), D297.1 (K)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
- new net F0_m: D1002.1 (K), D1025.1 (K), D1048.1 (K), D105.1 (K), D128.1 (K), D151.1 (K), D174.1 (K), D197.1 (K), D220.1 (K), D243.1 (K), D266.1 (K), D289.1 (K)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
- new net F0_mn: Q533.3 (D), Q534.2 (G), R285.2
- new net F1_m: D1003.1 (K), D1026.1 (K), D1049.1 (K), D106.1 (K), D129.1 (K), D152.1 (K), D175.1 (K), D198.1 (K), D221.1 (K), D244.1 (K), D267.1 (K), D290.1 (K)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
- new net F1_mn: Q535.3 (D), Q536.2 (G), R287.2
- new net FI_m: D1019.1 (K), D1042.1 (K), D122.1 (K), D145.1 (K), D168.1 (K), D191.1 (K), D214.1 (K), D237.1 (K), D260.1 (K), D283.1 (K), D30.1 (K), D306.1 (K)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
- new net FI_mn: Q521.3 (D), Q522.2 (G), R273.2
- new net HLT_m: D100.1 (K), D1020.1 (K), D1043.1 (K), D123.1 (K), D146.1 (K), D169.1 (K), D192.1 (K), D215.1 (K), D238.1 (K), D261.1 (K), D284.1 (K), D307.1 (K)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
- new net HLT_mn: Q523.3 (D), Q524.2 (G), R275.2
- new net INP_m: D1004.1 (K), D1027.1 (K), D1050.1 (K), D107.1 (K), D130.1 (K), D153.1 (K), D176.1 (K), D199.1 (K), D222.1 (K), D245.1 (K), D268.1 (K), D291.1 (K)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
- new net INP_mn: Q537.3 (D), Q538.2 (G), R289.2
- new net IO_m: D1018.1 (K), D1041.1 (K), D121.1 (K), D144.1 (K), D167.1 (K), D190.1 (K), D213.1 (K), D236.1 (K), D259.1 (K), D282.1 (K), D29.1 (K), D305.1 (K)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
- new net IO_mn: Q519.3 (D), Q520.2 (G), R271.2
- new net MAI_m: D101.1 (K), D1021.1 (K), D1044.1 (K), D124.1 (K), D147.1 (K), D170.1 (K), D193.1 (K), D216.1 (K), D239.1 (K), D262.1 (K), D285.1 (K), D308.1 (K)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
- new net MAI_mn: Q525.3 (D), Q526.2 (G), R277.2
- new net MI_m: D102.1 (K), D1022.1 (K), D1045.1 (K), D125.1 (K), D148.1 (K), D171.1 (K), D194.1 (K), D217.1 (K), D240.1 (K), D263.1 (K), D286.1 (K), D309.1 (K)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
- new net MI_mn: Q527.3 (D), Q528.2 (G), R279.2
- new net MO_m: D1000.1 (K), D1023.1 (K), D103.1 (K), D1046.1 (K), D126.1 (K), D149.1 (K), D172.1 (K), D195.1 (K), D218.1 (K), D241.1 (K), D264.1 (K), D287.1 (K)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
- new net MO_mn: Q529.3 (D), Q530.2 (G), R281.2
- new net OI_m: D1017.1 (K), D1040.1 (K), D120.1 (K), D143.1 (K), D166.1 (K), D189.1 (K), D212.1 (K), D235.1 (K), D258.1 (K), D28.1 (K), D281.1 (K), D304.1 (K)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
- new net OI_mn: Q517.3 (D), Q518.2 (G), R269.2
- new net ONE_m: D1001.1 (K), D1024.1 (K), D104.1 (K), D1047.1 (K), D127.1 (K), D150.1 (K), D173.1 (K), D196.1 (K), D219.1 (K), D242.1 (K), D265.1 (K), D288.1 (K)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
- new net ONE_mn: Q531.3 (D), Q532.2 (G), R283.2
- new net PCL_m: D1005.1 (K), D1028.1 (K), D1051.1 (K), D108.1 (K), D131.1 (K), D154.1 (K), D177.1 (K), D200.1 (K), D223.1 (K), D246.1 (K), D269.1 (K), D292.1 (K)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
- new net PCL_mn: Q539.3 (D), Q540.2 (G), R291.2
- new net PCR_m: D1006.1 (K), D1029.1 (K), D1052.1 (K), D109.1 (K), D132.1 (K), D155.1 (K), D178.1 (K), D201.1 (K), D224.1 (K), D247.1 (K), D270.1 (K), D293.1 (K)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
- new net PCR_mn: Q541.3 (D), Q542.2 (G), R293.2
- new net RAI_m: D1007.1 (K), D1030.1 (K), D1053.1 (K), D110.1 (K), D133.1 (K), D156.1 (K), D179.1 (K), D202.1 (K), D225.1 (K), D248.1 (K), D271.1 (K), D294.1 (K)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
- new net RAI_mn: Q543.3 (D), Q544.2 (G), R295.2
- new net R_OP10_4: D756.2 (A), D757.2 (A), D758.2 (A), D759.2 (A), D760.2 (A), D761.2 (A), D762.2 (A), D763.2 (A), D764.2 (A), D765.2 (A), D766.2 (A), D767.2 (A)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
- new net R_OP11_4: D802.2 (A), D803.2 (A), D804.2 (A), D805.2 (A), D806.2 (A), D807.2 (A), D808.2 (A), D809.2 (A), D810.2 (A), D811.2 (A), D812.2 (A), D813.2 (A)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
- new net R_OP12_4: D848.2 (A), D849.2 (A), D850.2 (A), D851.2 (A), D852.2 (A), D853.2 (A), D854.2 (A), D855.2 (A), D856.2 (A), D857.2 (A), D858.2 (A), D859.2 (A)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
- new net R_OP13_4: D894.2 (A), D895.2 (A), D896.2 (A), D897.2 (A), D898.2 (A), D899.2 (A), D900.2 (A), D901.2 (A), D902.2 (A), D903.2 (A), D904.2 (A), D905.2 (A)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
- new net R_OP14_4: D940.2 (A), D941.2 (A), D942.2 (A), D943.2 (A), D944.2 (A), D945.2 (A), D946.2 (A), D947.2 (A), D948.2 (A), D949.2 (A), D950.2 (A), D951.2 (A)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
- new net R_OP15_4: D1000.2 (A), D1001.2 (A), D1002.2 (A), D1003.2 (A), D1004.2 (A), D1005.2 (A), D1006.2 (A), D1007.2 (A), D1008.2 (A), D986.2 (A), D987.2 (A), D988.2 (A)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
- new net R_OP8_4: D664.2 (A), D665.2 (A), D666.2 (A), D667.2 (A), D668.2 (A), D669.2 (A), D670.2 (A), D671.2 (A), D672.2 (A), D673.2 (A), D674.2 (A), D675.2 (A)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
- new net R_OP9_4: D710.2 (A), D711.2 (A), D712.2 (A), D713.2 (A), D714.2 (A), D715.2 (A), D716.2 (A), D717.2 (A), D718.2 (A), D719.2 (A), D720.2 (A), D721.2 (A)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
- new net SUB_m: D1009.1 (K), D1032.1 (K), D112.1 (K), D135.1 (K), D158.1 (K), D181.1 (K), D20.1 (K), D204.1 (K), D227.1 (K), D250.1 (K), D273.1 (K), D296.1 (K)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
- new net SUB_mn: Q501.3 (D), Q502.2 (G), R253.2
Other:
- note added: "COLUMN BUFFERS (D041): the diode node of each column has a 1 Meg pull-down and feeds one inverter; a second inverter (22k) drives the control line, so the line falls through a transistor in microseconds instead of decaying through 1 Meg into every board and the ribbons."
- note added: "Cell: 2N7000 + 47k pull-up (NMOS, see docs/gate-cell.md). 586 transistors, 352 resistors, 83 matrix diodes, 19 LEDs. From the bus header: M7..M0 (the program memory word), CF and ZF (from the ALU), CLK, RST. To the bus header: II, PCE and the matrix columns SUB EO AI AO BI BO BA AB OI IO PCL FI HLT MAI MI MO ONE F0 F1 INP; BUS3#..BUS0# driven (open drain) with OPR3..0 while IO. To board 09 (count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"
- note added: "MATRIX ROWS: one per instruction for S3, and for S4 where the instruction uses it (the four memory accesses) and for every free opcode. Row = NOR(OPn#, T3N) or NOR(OPn#, T4N); family rows also include F#. JC/JZ have a conditional row for PCL: NOR(OP#, T3N, flag-not). 10k pull-ups: a row drives up to ten diodes into 1 Meg column pull-downs."
- note added: "OP10 (free) S4"
- note added: "OP11 (free) S4"
- note added: "OP12 (free) S4"
- note added: "OP13 (free) S4"
- note added: "OP14 (free) S4"
- note added: "OP15 (free) S4"
- note added: "OP8 (free) S4"
- note added: "OP9 (free) S4"
- note added: "Rows are driven by the NOR gates on the left (10k pull-ups); a diode pulls its column high while the row is high; columns have 1 Meg pull-downs and a buffer to the bus header. Every crossing has a pad pair on the board; a crossed-out diode is not fitted. Add an instruction: solder diodes on a free row."
- note removed: "Cell: 2N7000 + 47k pull-up (NMOS, see docs/gate-cell.md). 524 transistors, 298 resistors, 83 matrix diodes, 19 LEDs. From the bus header: M7..M0 (the program memory word), CF and ZF (from the ALU), CLK, RST. To the bus header: II, PCE and the matrix columns SUB EO AI AO BI BO BA AB OI IO PCL FI HLT MAI MI MO ONE F0 F1 INP; BUS3#..BUS0# driven (open drain) with OPR3..0 while IO. To board 09 (count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"
- note removed: "MATRIX ROWS: one per instruction for S3, and for S4 where the instruction uses it (the four memory accesses). Row = NOR(OPn#, T3N) or NOR(OPn#, T4N); family rows also include F#. JC/JZ have a conditional row for PCL: NOR(OP#, T3N, flag-not). 10k pull-ups: a row drives up to ten diodes into 1 Meg column pull-downs."
- note removed: "Rows are driven by the NOR gates on the left (10k pull-ups); a diode pulls its column high while the row is high; columns have 1 Meg pull-downs and go to the bus header. Add an instruction: add diodes."
