File: cards/coupon/coupon-testbench.kicad_sch (KiCad schematic)
At the start: 5 parts

Commit message: Coupon respun with every cell on it (D056): the bench's expected readings from its own netlist
The coupon is what proves the simulations right before the second order, and
the old one measured only the inverter. It now carries, each with a test
loop: the 5-inverter ring (a buffered loop and a raw one on the ring node),
fan-out 1 and 10, NAND3 and NOR3, the bus driver against 10k, the clock
card's oscillator (its Schmitt pair and 100k + 47 nF, the same parts drawn
on the sheet), a master-slave flip-flop wired as a toggle with the
asynchronous reset the counters and the sequencer use, the D053 line
driver (1k inverter, 100 ohm, diode, 10k pull-down; 3.3 nF clipped on at
the bench), a diode-connected transistor on 4.7k that reads its own
threshold, and a program row (3.3k, 1N4148, 220k). Inputs IN N1 N2 N3 RST
on a 6-pin header with 1 Meg pull-downs, power on a 2-pin header for the
bench supply, fifteen loops. 57 transistors on six tile columns of one
100 x 100 card; ERC 0, one freerouting pass, DRC 0 errors (one dangling
trunk end), 0 open under JLCPCB's minimum rules too.

sim/tb_coupon.py simulates the routed card's kicad export (or the gate list
plus the sheet parts, which agree at every uniform corner) at TYP, LO, HI
and MIX seeds 1..3, a x10 probe on every loop, and writes the bands the
bench must land in: sim/results/coupon_expected.md. Ring 5.9 to 23.6 us
(14.6 typical), fan-out-1 rise 10 to 12 us, fan-out-10 rise 67 to 77 us,
stacks under 2 mV, Schmitt hysteresis 0.4 V about the threshold,
oscillator 1.64 to 2.55 ms, Q at half that with one edge per clock edge,
DRV 4.0 V high, 6.6 us up and 49 us down into 3.3 nF, VTO 0.88 to 3.02 V,
ROM 4.52 V, 5 to 8 mA with IN low and 11 to 14 mA with IN high.

Two things the testbench found before the copper did: with low-threshold
transistors the ring swings only to 1.6 to 3 V and a high-threshold buffer
never switches (the buffered loop was blind at two MIX seeds; hence the
raw RING0 loop), and while RST holds the flip-f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
Parts:
- added V9006: VPWL, symbol Simulation_SPICE:VPWL
Connections:
- net GND: now also V9006.2
- new net RST: V9006.1
Other:
- note added: ".ic v(RING0)=0 v(X)=0"
- note added: ".tran 0.5u 12m"
- note added: "TESTBENCH: IN toggles at 1 kHz, N1..N3 are stepped through 000,100,110,111, RST is high for the first millisecond. Excluded from the board; sim/tb_coupon.py is the measured bench."
- note removed: ".ic v(RING0)=0"
- note removed: ".tran 0.2u 4m"
- note removed: "TESTBENCH: IN toggles at 1 kHz, N1..N3 are stepped through 000,100,110,111. Excluded from the board."
