File: cards/alu3/alu3.kicad_pcb (KiCad board)
At the start: 2 copper layers, 100 x 100 mm, 126 parts, among them J1 BUS, J2 IN, Q1 2N7000, Q10 2N7000, Q11 2N7000, Q12 2N7000, Q13 2N7000, Q14 2N7000, Q15 2N7000, Q16 2N7000, Q17 2N7000, Q18 2N7000, Q19 2N7000, Q2 2N7000, Q20 2N7000, Q21 2N7000, Q22 2N7000, Q23 2N7000, Q24 2N7000, Q25 2N7000, Q26 2N7000, Q27 2N7000, Q28 2N7000, Q29 2N7000, Q3 2N7000, Q30 2N7000, Q31 2N7000, Q32 2N7000, Q33 2N7000, Q34 2N7000, Q35 2N7000, Q36 2N7000, Q37 2N7000, Q38 2N7000, Q39 2N7000, Q4 2N7000, Q40 2N7000, Q41 2N7000, Q42 2N7000, Q43 2N7000, Q44 2N7000, Q45 2N7000, Q46 2N7000, Q47 2N7000, Q48 2N7000, Q49 2N7000, Q5 2N7000, Q50 2N7000, Q51 2N7000, Q52 2N7000, Q53 2N7000, Q54 2N7000, Q55 2N7000, Q56 2N7000, Q57 2N7000, Q58 2N7000, Q59 2N7000, Q6 2N7000, Q60 2N7000, Q61 2N7000, Q62 2N7000, Q63 2N7000, Q64 2N7000, Q65 2N7000, Q66 2N7000, Q67 2N7000, Q68 2N7000, Q69 2N7000, Q7 2N7000, Q70 2N7000, Q71 2N7000, Q72 2N7000, Q73 2N7000, Q8 2N7000, Q9 2N7000

Commit message: The bus headers go on the back of all 26 boards, no track moved; the silkscreen refitted (D059, D062)
An IDC socket lies across its ribbon, so the ribbon could never run along a
row of cards as drawn. It runs behind them, and the 64-pin headers are
soldered on the back. This commit is that move, made in place on the routed
boards: no board was routed again.

How the header sits (D062): in the holes it had, turned over top to bottom,
notch toward the top edge. A pin of the odd row is then in the hole its even
neighbour had, so the two signals of every pair of pins change places: CLK
is pin 6, RST pin 8, +5V pins 1, 2 and 64. bus.py keeps both tables: PINS,
what the header's pins carry, and HOLES, what the copper was routed to.

The proof, on all 26 boards against 992a90f (sim/board_diff.py):
  netlist the same, element for element; every track, every via and every
  hole the same; each copper and mask layer differs by two pad shapes per
  header (pin 1's square went to the hole beside it, both on +5V) and the
  ground pour's outline round those two pads, nowhere else by more than a
  tenth of a micrometre.
sim/rebuild_check.py runs every builder into a scratch directory: each
writes the plan and the netlist that are committed, so a rebuild gives
this board. order_check.py --machine holds every pad of the 27 headers to
bus.py and requires them on the back.

What the move costs: on the ribbon RST had a ground conductor on both
sides; now one neighbour is BUS1#. tb_rst_neighbour.py puts the two lines
on the bench with every gate the routed boards hang on them: RST rises
0.28 to 0.43 V when BUS1# is released, against a lowest threshold of 0.8 V
(sim/results/rst_neighbour.md). The machine deck's crosstalk option now
couples the pins that are neighbours on the ribbon; the crosstalk stage of
the machine gate has to be run again on that order.

Silkscreen (pcb.fit_silk): every label to 1.0 mm where it has room, off
pads, vias, outlines and other labels, out from under the pa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
Parts:
- J1: moved to B.Cu
- moved J1 2.54 mm to (10.6, 4.96), turned to -90 degrees
Connections:
- J1 pad 11: unconnected-(J1-Pin_11-Pad11) -> BUS3#
- J1 pad 12: BUS3# -> unconnected-(J1-Pin_12-Pad12)
- J1 pad 15: unconnected-(J1-Pin_15-Pad15) -> A3
- J1 pad 16: A3 -> unconnected-(J1-Pin_16-Pad16)
- J1 pad 19: unconnected-(J1-Pin_19-Pad19) -> B3
- J1 pad 20: B3 -> unconnected-(J1-Pin_20-Pad20)
- J1 pad 37: CF -> ZF
- J1 pad 38: ZF -> CF
- J1 pad 39: SUB -> EO
- J1 pad 40: EO -> SUB
- J1 pad 5: unconnected-(J1-Pin_5-Pad5) -> GND
- J1 pad 59: ONE -> F0
- J1 pad 6: GND -> unconnected-(J1-Pin_6-Pad6)
- J1 pad 60: F0 -> ONE
- J1 pad 61: F1 -> unconnected-(J1-Pin_61-Pad61)
- J1 pad 62: unconnected-(J1-Pin_62-Pad62) -> F1
- J1 pad 63: +5V -> GND
- J1 pad 64: GND -> +5V
- J1 pad 7: unconnected-(J1-Pin_7-Pad7) -> GND
- J1 pad 8: GND -> unconnected-(J1-Pin_8-Pad8)
Other:
- board text added: "2"
- board text added: "63"
- board text added: "64"
- board text added: "HEADER HERE"
- board text added: "HEADER ON THE BACK"
- board text added: "NOTCH TO TOP"

Commit message: Silk: the front no longer says HEADER ON THE BACK; the back says HEADER HERE, which is enough
A "not here" note under the holes on every board, the kind of text that
narrates instead of naming. The back carries the header's outline with
HEADER HERE and NOTCH TO TOP; the front keeps the pin numbers 1, 2, 63,
64. All 26 boards re-silked in place from their plans (no re-route, the
schematics untouched); the order gate's silk rule now wants HEADER HERE
on the back and no HEADER ON THE BACK anywhere. Gate all pass, every
builder writes what is committed, parts tables unchanged.

Co-Authored-By: Claude Fable 5.1 <noreply@anthropic.com>
Claude-Session: https://claude.ai/code/session_01RktbhdQjDu7SpFpvkevyUU
Other:
- board text removed: "HEADER ON THE BACK"
Changed lines of the file:
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@@
-		)
-	)
-	(gr_text "HEADER ON THE BACK"
-		(at 26.63 11.4 0)
-		(layer "F.SilkS")
-		(effects
-			(font
-				(size 1 1)
-				(thickness 0.15)
-			)
-			(justify left)
 		)
 	)

Commit message: The Nibble logo on the front silkscreen of every board
lib/logo/nibble.png traced by sim/logo.py (potracer) into two silkscreen
footprints, lib/nibble.pretty/Logo_Nibble (icon and word, 27 x 8 mm) and
Logo_Nibble_Icon (8 x 8): filled polygons, holes slit in. At 8 mm the
ribbon's lines print 0.39 mm wide and 0.24 mm apart; the fab's minimum
is 0.15. No pads, no copper, out of the parts list and the position file.

pcb.py places it on every board before the labels are fitted
(place_logo): icon and word where a patch 27 x 8 mm is free of pads,
vias, outlines, courtyards, the labels and 1 mm of edge, the icon alone
otherwise, the nearest such patch to the board's name; the fitter then
keeps the labels off it. 25 boards took the full logo, the coupon the
icon. All 26 re-silked in place (no re-route, the schematics untouched).
The order gate wants exactly one logo on a board; bom.py counts it as no
part. Two pcbnew quirks met on the way: a footprint removed in the
fitter's process makes the next loaded board untyped (every hidden
reference became an obstacle and BUS0 on the hub fell back to 0.8 mm),
and after a text is removed the footprints are untyped too, so resilk
takes the old logo off before the texts.

Gate all pass on all 26, every builder writes what is committed, parts
tables unchanged. The pilot's three zips are new again (order-1.md).

Co-Authored-By: Claude Fable 5.1 <noreply@anthropic.com>
Claude-Session: https://claude.ai/code/session_01RktbhdQjDu7SpFpvkevyUU
Parts:
- added LOGO: Logo_Nibble, Logo_Nibble, F.Cu at (40.1, 90.9)

Commit message: The logo on the sequencer alone: one maker's mark, not a product line
With the logo on all 26 the machine looked factory-made. It stays on the
sequencer, the big board in the middle that people look at; the cards
carry their name. A board gets the logo when its plan says extra.logo
(the sequencer's builder does), none otherwise, and the order gate holds
each board to its plan. The 25 cards re-silked in place (no re-route).
Gate all pass, builders write what is committed, parts tables unchanged.
The pilot's three zips are new again (order-1.md).

Co-Authored-By: Claude Fable 5.1 <noreply@anthropic.com>
Claude-Session: https://claude.ai/code/session_01RktbhdQjDu7SpFpvkevyUU
Parts:
- removed LOGO: Logo_Nibble, Logo_Nibble
