File: cards/memctl/memctl.kicad_pcb (KiCad board)
At the start: 2 copper layers, 100 x 100 mm, 108 parts, among them J1 BUS, J2 LINK, Q1 2N7000, Q10 2N7000, Q11 2N7000, Q12 2N7000, Q13 2N7000, Q14 2N7000, Q15 2N7000, Q16 2N7000, Q17 2N7000, Q18 2N7000, Q19 2N7000, Q2 2N7000, Q20 2N7000, Q21 2N7000, Q22 2N7000, Q23 2N7000, Q24 2N7000, Q25 2N7000, Q26 2N7000, Q27 2N7000, Q28 2N7000, Q29 2N7000, Q3 2N7000, Q30 2N7000, Q31 2N7000, Q32 2N7000, Q33 2N7000, Q34 2N7000, Q35 2N7000, Q36 2N7000, Q37 2N7000, Q38 2N7000, Q39 2N7000, Q4 2N7000, Q40 2N7000, Q41 2N7000, Q42 2N7000, Q43 2N7000, Q44 2N7000, Q45 2N7000, Q46 2N7000, Q47 2N7000, Q48 2N7000, Q49 2N7000, Q5 2N7000, Q50 2N7000, Q51 2N7000, Q52 2N7000, Q53 2N7000, Q54 2N7000, Q55 2N7000, Q56 2N7000, Q57 2N7000, Q58 2N7000, Q59 2N7000, Q6 2N7000, Q7 2N7000, Q8 2N7000, Q9 2N7000

Commit message: Memory control: the address latch and the write take a mid-tick pulse (D054)
gcd, list and logic at mixed-threshold seed 2, with the clock card in the
deck, each wrote its first STORE to the wrong slot (12, 9 and 15 instead
of 0) and computed faithfully from there. A probed rerun of gcd to 134 ms
(memctl PH1, ENM, MAR, slot 0's SEL, WRE and cells): at the rising edge
ending the MAI tick the sequencer stepped when CLK passed 2 V and AO put
the STORE data on the bus 10 us later; the memory control card's PH1 NOR
saw the edge only at 3 V, and its address-latch enable (MAI AND PH1)
closed 12 us after the bus had changed, so MAR took the data as the
address. The write window (MI AND PH1) had the same exposure. D037's rule,
"PH1 closes before the rising edge on which everything else changes",
holds only if every card sees the edge at the same instant; with a 35 us
edge and 0.8 to 3.0 V thresholds they did not (D053 sharpens the edge;
this commit takes the memory out of the race altogether).

memory.py, build_ctl (and the reference board in build): CLKD is CLK
through 100k into 2.2 nF, drawn on the sheet; MPH = NOR(CLK, NOT CLKD) is
high from the falling edge of CLK until CLKD decays past a threshold,
60 to 350 us. ENM = MAI AND MPH, MIN = NAND(MI, MPH). The latch closes and
the write ends hundreds of microseconds before the next rising edge, when
the bus and the control lines have been stable for 700 us. PH1/PH2 leave
the card (57 transistors, was 59). cards/memctl regenerated and re-routed:
DRC 0, 0 unconnected, renders read; the slot card is unchanged.

tb_memory: --race is the edge as the memory card saw it in the machine:
CLK rises over 35 us, the bus switches 10 us into the rise, the control
lines 100 us after it (they lag every edge by 60 to 170 us in the machine;
a first version switched them with the bus and MAI closed the latch
itself, no failure). The bench's clock now runs a cycle before the first
case so the first tick has its falling edge too. The gate-list n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
Parts:
- removed Q58, Q59: 2N7000, TO-92_Inline_Wide
- added C3: 2.2n, C_Disc_D5.0mm_W2.5mm_P2.50mm, F.Cu at (86.0, 64.0)
- R12, R17, R22, R27, R29: value 47k -> 22k
- R13, R18, R23, R28: value 22k -> 47k
- R3: value 10k -> 47k
- R33: value 22k -> 4.7k
- R34: value 4.7k -> 22k
- R35: value 22k -> 1k
- R39: value 1k -> 100k
- moved R34 60.2 mm to (47.4, 75.7)
- moved Q53 59.1 mm to (52.5, 79.5), turned to 180 degrees
- moved R39 51.0 mm to (80.0, 64.0), turned to -90 degrees
- moved D4 46.4 mm to (57.6, 68.1)
- moved D3 21.6 mm to (57.6, 52.8)
- moved D1 21.6 mm to (57.6, 22.4)
- moved D2 21.6 mm to (57.6, 37.6)
- moved R35 13.3 mm to (55.1, 16.0)
- moved Q56 8.89 mm to (55.1, 57.3)
- moved Q57 8.89 mm to (55.1, 72.5)
- moved Q55 8.25 mm to (55.1, 42.0)
- moved R36 6.35 mm to (55.1, 31.2)
- moved R37 6.35 mm to (55.1, 46.5)
- moved R38 6.35 mm to (55.1, 61.7)
- moved R10 5.08 mm to (16.7, 32.5)
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Connections:
- Q1 pad 2: CLK -> CLKD
- Q1 pad 3: CLKN -> CLKDN
- Q10 pad 1: Net-(Q10-S) -> GND
- Q10 pad 2: MAI -> ENMN
- Q10 pad 3: ENMN -> ENM
- Q11 pad 2: PH1 -> D0
- Q11 pad 3: Net-(Q10-S) -> MAR0_dn
- Q12 pad 1: GND -> Net-(Q12-S)
- Q12 pad 2: ENMN -> D0
- Q12 pad 3: ENM -> MAR0_m1
- Q13 pad 2: D0 -> ENM
- Q13 pad 3: MAR0_dn -> Net-(Q12-S)
- Q14 pad 2: D0 -> ENM
- Q14 pad 3: MAR0_m1 -> MAR0_m2
- Q15 pad 2: ENM -> MAR0_dn
- Q16 pad 2: ENM -> MAR0_m1
- Q16 pad 3: MAR0_m2 -> MAR0
- Q17 pad 2: MAR0_dn -> MAR0_qn
- Q18 pad 2: MAR0_m1 -> MAR0
- Q18 pad 3: MAR0 -> MAR0_qn
- Q19 pad 2: MAR0_qn -> MAR0_m2
- Q2 pad 3: PH1 -> MPH
- Q20 pad 1: Net-(Q20-S) -> GND
- Q20 pad 2: MAR0 -> D1
- Q20 pad 3: MAR0_qn -> MAR1_dn
- Q21 pad 1: GND -> Net-(Q21-S)
- Q21 pad 2: MAR0_m2 -> D1
- Q21 pad 3: Net-(Q20-S) -> MAR1_m1
- Q22 pad 2: D1 -> ENM
- Q22 pad 3: MAR1_dn -> Net-(Q21-S)
- Q23 pad 2: D1 -> ENM
- Q23 pad 3: MAR1_m1 -> MAR1_m2
- Q24 pad 2: ENM -> MAR1_dn
- Q25 pad 2: ENM -> MAR1_m1
- Q25 pad 3: MAR1_m2 -> MAR1
- Q26 pad 2: MAR1_dn -> MAR1_qn
- Q27 pad 2: MAR1_m1 -> MAR1
- Q27 pad 3: MAR1 -> MAR1_qn
- Q28 pad 2: MAR1_qn -> MAR1_m2
- Q29 pad 1: Net-(Q29-S) -> GND
- Q29 pad 2: MAR1 -> D2
- Q29 pad 3: MAR1_qn -> MAR2_dn
- Q3 pad 2: PH2 -> CLKDN
- Q3 pad 3: PH1 -> MPH
- Q30 pad 1: GND -> Net-(Q30-S)
- Q30 pad 2: MAR1_m2 -> D2
- Q30 pad 3: Net-(Q29-S) -> MAR2_m1
- Q31 pad 2: D2 -> ENM
- Q31 pad 3: MAR2_dn -> Net-(Q30-S)
- Q32 pad 2: D2 -> ENM
- Q32 pad 3: MAR2_m1 -> MAR2_m2
- Q33 pad 2: ENM -> MAR2_dn
- Q34 pad 2: ENM -> MAR2_m1
- Q34 pad 3: MAR2_m2 -> MAR2
- Q35 pad 2: MAR2_dn -> MAR2_qn
- Q36 pad 2: MAR2_m1 -> MAR2
- Q36 pad 3: MAR2 -> MAR2_qn
- Q37 pad 2: MAR2_qn -> MAR2_m2
- Q38 pad 1: Net-(Q38-S) -> GND
- Q38 pad 2: MAR2 -> D3
- Q38 pad 3: MAR2_qn -> MAR3_dn
- Q39 pad 1: GND -> Net-(Q39-S)
- Q39 pad 2: MAR2_m2 -> D3
- Q39 pad 3: Net-(Q38-S) -> MAR3_m1
- Q4 pad 2: CLKN -> BUS0#
- Q4 pad 3: PH2 -> D0
- Q40 pad 2: D3 -> ENM
- Q40 pad 3: MAR3_dn -> Net-(Q39-S)
- Q41 pad 2: D3 -> ENM
- Q41 pad 3: MAR3_m1 -> MAR3_m2
- Q42 pad 2: ENM -> MAR3_dn
- Q43 pad 2: ENM -> MAR3_m1
- Q43 pad 3: MAR3_m2 -> MAR3
- Q44 pad 2: MAR3_dn -> MAR3_qn
- Q45 pad 2: MAR3_m1 -> MAR3
- Q45 pad 3: MAR3 -> MAR3_qn
- Q46 pad 2: MAR3_qn -> MAR3_m2
- Q47 pad 1: Net-(Q47-S) -> GND
- Q47 pad 2: MAR3 -> MAR0
- Q47 pad 3: MAR3_qn -> MAR0N
- Q48 pad 2: MAR3_m2 -> MAR1
- Q48 pad 3: Net-(Q47-S) -> MAR1N
- Q49 pad 2: MAR0 -> MAR2
- Q49 pad 3: MAR0N -> MAR2N
- Q5 pad 2: PH1 -> BUS1#
- Q5 pad 3: PH2 -> D1
- Q50 pad 2: MAR1 -> MAR3
- Q50 pad 3: MAR1N -> MAR3N
- Q51 pad 1: GND -> Net-(Q51-S)
- Q51 pad 2: MAR2 -> MI
- Q51 pad 3: MAR2N -> MIN
- Q52 pad 2: MAR3 -> MPH
- Q52 pad 3: MAR3N -> Net-(Q51-S)
- Q53 pad 1: Net-(Q53-S) -> GND
- Q53 pad 2: MI -> MO
- Q53 pad 3: MIN -> MON
- Q54 pad 2: PH1 -> MAR3
- Q54 pad 3: Net-(Q53-S) -> Net-(D1-K)
- Q55 pad 2: MO -> MAR2
- Q55 pad 3: MON -> Net-(D2-K)
- Q56 pad 2: MAR3 -> MAR1
- Q56 pad 3: Net-(D1-K) -> Net-(D3-K)
- Q57 pad 2: MAR2 -> MAR0
- Q57 pad 3: Net-(D2-K) -> Net-(D4-K)
- Q6 pad 2: BUS0# -> BUS2#
- Q6 pad 3: D0 -> D2
- Q7 pad 2: BUS1# -> BUS3#
- Q7 pad 3: D1 -> D3
- Q8 pad 1: GND -> Net-(Q8-S)
- Q8 pad 2: BUS2# -> MAI
- Q8 pad 3: D2 -> ENMN
- Q9 pad 2: BUS3# -> MPH
- Q9 pad 3: D3 -> Net-(Q8-S)
- R1 pad 1: CLKN -> CLKDN
- R10 pad 2: MAR0_dn -> MAR0_m1
- R11 pad 2: MAR0_m1 -> MAR0_m2
- R12 pad 2: MAR0_m2 -> MAR0
- R13 pad 1: MAR0 -> MAR0_qn
- R14 pad 1: MAR0_qn -> MAR1_dn
- R15 pad 1: MAR1_dn -> MAR1_m1
- R16 pad 1: MAR1_m1 -> MAR1_m2
- R17 pad 1: MAR1_m2 -> MAR1
- R18 pad 2: MAR1 -> MAR1_qn
- R19 pad 2: MAR1_qn -> MAR2_dn
- R2 pad 1: PH1 -> MPH
- R20 pad 2: MAR2_dn -> MAR2_m1
- R21 pad 2: MAR2_m1 -> MAR2_m2
- R22 pad 2: MAR2_m2 -> MAR2
- R23 pad 1: MAR2 -> MAR2_qn
- R24 pad 1: MAR2_qn -> MAR3_dn
- R25 pad 1: MAR3_dn -> MAR3_m1
- R26 pad 1: MAR3_m1 -> MAR3_m2
- R27 pad 1: MAR3_m2 -> MAR3
- R28 pad 2: MAR3 -> MAR3_qn
- R29 pad 2: MAR3_qn -> MAR0N
- R3 pad 1: PH2 -> D0
- R30 pad 2: MAR0N -> MAR1N
- R31 pad 2: MAR1N -> MAR2N
- R32 pad 2: MAR2N -> MAR3N
- R33 pad 2: MAR3N -> MIN
- R34 pad 1: MIN -> +5V
- R34 pad 2: +5V -> MON
- R35 pad 1: MON -> Net-(D1-A)
- R36 pad 1: Net-(D1-A) -> Net-(D2-A)
- R37 pad 1: Net-(D2-A) -> Net-(D3-A)
- R38 pad 1: Net-(D3-A) -> Net-(D4-A)
- R39 pad 1: +5V -> CLK
- R39 pad 2: Net-(D4-A) -> CLKD
- R4 pad 1: D0 -> D1
- R5 pad 1: D1 -> D2
- R6 pad 1: D2 -> D3
- R7 pad 1: D3 -> ENMN
- R8 pad 2: ENMN -> ENM
- R9 pad 2: ENM -> MAR0_dn
Routing:
- net CLK: track 22.9 -> 140.0 mm, vias 0 -> 1
- net CLKD: track 0.00 -> 116.3 mm
- net MPH: track 0.00 -> 101.5 mm
- net PH1: track 84.8 -> 0.00 mm
- net MAR0_qn: track 11.5 -> 69.8 mm
- net MAR2_qn: track 11.5 -> 69.5 mm
- net MAR3_qn: track 11.8 -> 67.1 mm, vias 0 -> 1
- net MAR1_qn: track 11.6 -> 65.7 mm, vias 0 -> 2
- net MO: track 38.7 -> 90.2 mm, vias 1 -> 0
- net MON: track 69.7 -> 20.8 mm
- net MIN: track 96.7 -> 48.8 mm
- net MI: track 29.0 -> 72.6 mm, vias 0 -> 1
- net ENMN: track 23.5 -> 64.8 mm
- net MAI: track 83.4 -> 120.3 mm, vias 0 -> 1
- net CLKN: track 34.2 -> 0.00 mm
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
Commit message: The bus headers go on the back of all 26 boards, no track moved; the silkscreen refitted (D059, D062)
An IDC socket lies across its ribbon, so the ribbon could never run along a
row of cards as drawn. It runs behind them, and the 64-pin headers are
soldered on the back. This commit is that move, made in place on the routed
boards: no board was routed again.

How the header sits (D062): in the holes it had, turned over top to bottom,
notch toward the top edge. A pin of the odd row is then in the hole its even
neighbour had, so the two signals of every pair of pins change places: CLK
is pin 6, RST pin 8, +5V pins 1, 2 and 64. bus.py keeps both tables: PINS,
what the header's pins carry, and HOLES, what the copper was routed to.

The proof, on all 26 boards against 992a90f (sim/board_diff.py):
  netlist the same, element for element; every track, every via and every
  hole the same; each copper and mask layer differs by two pad shapes per
  header (pin 1's square went to the hole beside it, both on +5V) and the
  ground pour's outline round those two pads, nowhere else by more than a
  tenth of a micrometre.
sim/rebuild_check.py runs every builder into a scratch directory: each
writes the plan and the netlist that are committed, so a rebuild gives
this board. order_check.py --machine holds every pad of the 27 headers to
bus.py and requires them on the back.

What the move costs: on the ribbon RST had a ground conductor on both
sides; now one neighbour is BUS1#. tb_rst_neighbour.py puts the two lines
on the bench with every gate the routed boards hang on them: RST rises
0.28 to 0.43 V when BUS1# is released, against a lowest threshold of 0.8 V
(sim/results/rst_neighbour.md). The machine deck's crosstalk option now
couples the pins that are neighbours on the ribbon; the crosstalk stage of
the machine gate has to be run again on that order.

Silkscreen (pcb.fit_silk): every label to 1.0 mm where it has room, off
pads, vias, outlines and other labels, out from under the pa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
Parts:
- J1: moved to B.Cu
- moved J1 2.54 mm to (10.6, 4.96), turned to -90 degrees
Connections:
- J1 pad 10: BUS1# -> BUS0#
- J1 pad 11: BUS2# -> BUS3#
- J1 pad 12: BUS3# -> BUS2#
- J1 pad 5: CLK -> GND
- J1 pad 53: unconnected-(J1-Pin_53-Pad53) -> MAI
- J1 pad 54: MAI -> unconnected-(J1-Pin_54-Pad54)
- J1 pad 55: MI -> MO
- J1 pad 56: MO -> MI
- J1 pad 6: GND -> CLK
- J1 pad 63: +5V -> GND
- J1 pad 64: GND -> +5V
- J1 pad 7: unconnected-(J1-Pin_7-Pad7) -> GND
- J1 pad 8: GND -> unconnected-(J1-Pin_8-Pad8)
- J1 pad 9: BUS0# -> BUS1#
Other:
- board text added: "2"
- board text added: "63"
- board text added: "64"
- board text added: "HEADER HERE"
- board text added: "HEADER ON THE BACK"
- board text added: "NOTCH TO TOP"

Commit message: Silk: the front no longer says HEADER ON THE BACK; the back says HEADER HERE, which is enough
A "not here" note under the holes on every board, the kind of text that
narrates instead of naming. The back carries the header's outline with
HEADER HERE and NOTCH TO TOP; the front keeps the pin numbers 1, 2, 63,
64. All 26 boards re-silked in place from their plans (no re-route, the
schematics untouched); the order gate's silk rule now wants HEADER HERE
on the back and no HEADER ON THE BACK anywhere. Gate all pass, every
builder writes what is committed, parts tables unchanged.

Co-Authored-By: Claude Fable 5.1 <noreply@anthropic.com>
Claude-Session: https://claude.ai/code/session_01RktbhdQjDu7SpFpvkevyUU
Other:
- board text removed: "HEADER ON THE BACK"
Changed lines of the file:
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@@
-		)
-	)
-	(gr_text "HEADER ON THE BACK"
-		(at 26.63 11.4 0)
-		(layer "F.SilkS")
-		(effects
-			(font
-				(size 1 1)
-				(thickness 0.15)
-			)
-			(justify left)
 		)
 	)

Commit message: The Nibble logo on the front silkscreen of every board
lib/logo/nibble.png traced by sim/logo.py (potracer) into two silkscreen
footprints, lib/nibble.pretty/Logo_Nibble (icon and word, 27 x 8 mm) and
Logo_Nibble_Icon (8 x 8): filled polygons, holes slit in. At 8 mm the
ribbon's lines print 0.39 mm wide and 0.24 mm apart; the fab's minimum
is 0.15. No pads, no copper, out of the parts list and the position file.

pcb.py places it on every board before the labels are fitted
(place_logo): icon and word where a patch 27 x 8 mm is free of pads,
vias, outlines, courtyards, the labels and 1 mm of edge, the icon alone
otherwise, the nearest such patch to the board's name; the fitter then
keeps the labels off it. 25 boards took the full logo, the coupon the
icon. All 26 re-silked in place (no re-route, the schematics untouched).
The order gate wants exactly one logo on a board; bom.py counts it as no
part. Two pcbnew quirks met on the way: a footprint removed in the
fitter's process makes the next loaded board untyped (every hidden
reference became an obstacle and BUS0 on the hub fell back to 0.8 mm),
and after a text is removed the footprints are untyped too, so resilk
takes the old logo off before the texts.

Gate all pass on all 26, every builder writes what is committed, parts
tables unchanged. The pilot's three zips are new again (order-1.md).

Co-Authored-By: Claude Fable 5.1 <noreply@anthropic.com>
Claude-Session: https://claude.ai/code/session_01RktbhdQjDu7SpFpvkevyUU
Parts:
- added LOGO: Logo_Nibble, Logo_Nibble, F.Cu at (68.1, 80.4)

Commit message: The logo on the sequencer alone: one maker's mark, not a product line
With the logo on all 26 the machine looked factory-made. It stays on the
sequencer, the big board in the middle that people look at; the cards
carry their name. A board gets the logo when its plan says extra.logo
(the sequencer's builder does), none otherwise, and the order gate holds
each board to its plan. The 25 cards re-silked in place (no re-route).
Gate all pass, builders write what is committed, parts tables unchanged.
The pilot's three zips are new again (order-1.md).

Co-Authored-By: Claude Fable 5.1 <noreply@anthropic.com>
Claude-Session: https://claude.ai/code/session_01RktbhdQjDu7SpFpvkevyUU
Parts:
- removed LOGO: Logo_Nibble, Logo_Nibble
