File: cards/clock/clock.kicad_pcb (KiCad board)
At the start: 2 copper layers, 100 x 100 mm, 56 parts, among them J1 BUS, J2 SLOW, Q1 2N7000, Q10 2N7000, Q11 2N7000, Q12 2N7000, Q13 2N7000, Q14 2N7000, Q15 2N7000, Q16 2N7000, Q17 2N7000, Q2 2N7000, Q3 2N7000, Q4 2N7000, Q5 2N7000, Q6 2N7000, Q7 2N7000, Q8 2N7000, Q9 2N7000, SW1 RUN

Commit message: Clock card: the hold-off is on the card (D064); the machine's deck is the one the 74 runs proved
sim/build_clock_card.py adds the two parts of D064: Q18, a 2N7000 with its
gate on the RST line, its drain through R24, 100 ohm, to the oscillator's
timing node X, its source on the tiles' ground trunk, which is extended
down to it (routed once without that, the pour left the source pad on an
island of its own). The card's export is the one before plus
  MQ18 Net-_Q18-D_ RST GND 2N7000
  R24 X Net-_Q18-D_ 100
and nothing else. Routed in one attempt, DRC clean, every label at 1.0 mm.
The print, the two renders and the assembly drawing looked at.

The machine deck built from this card is the deck the queue ran with
HOLD=1, element for element: the clock's subcircuit the same with the two
parts' names changed, the rest of the deck the same (checked against the
saved deck of the MIX2 start at POR_V0 3.133881 V). So the 62 starts
(sim/results/starts_hold.md) and the 12 crosstalk runs
(sim/results/gate26_cross.md) are this card's.

The order: one more 2N7000 (3516) and one more 100 ohm (6); the buy
column does not move. docs: cards.md, cards/README.md, DECISIONS.md D064
(on the card), audit.md (the crosstalk stage paid, the part counts).

Co-Authored-By: Claude Fable 5.1 <noreply@anthropic.com>
Claude-Session: https://claude.ai/code/session_01RktbhdQjDu7SpFpvkevyUU
Parts:
- added Q18: 2N7000, TO-92_Inline_Wide, F.Cu at (23.1, 66.0)
- added R24: 100, R_Axial_DIN0207_L6.3mm_D2.5mm_P5.08mm_Vertical, F.Cu at (33.0, 64.0)
Routing:
- net SA: track 67.3 -> 104.9 mm
- net X: track 51.1 -> 65.9 mm
- net RST: track 80.6 -> 90.0 mm
- net GND: track 138.0 -> 147.3 mm
- net +5V: track 268.3 -> 274.7 mm
- net RD: track 87.0 -> 80.8 mm
- net Net-(Q18-D): track 0.00 -> 6.11 mm
- net PB: track 102.7 -> 107.0 mm
- net PN: track 95.6 -> 91.4 mm
- net RUNSW: track 108.4 -> 112.0 mm
- net VD2: track 59.3 -> 56.1 mm
- net CLK: track 98.9 -> 101.8 mm
- net HLTN: track 39.9 -> 37.2 mm
- net RT: track 28.6 -> 29.6 mm
- net SB: track 63.3 -> 63.1 mm, vias 0 -> 1

Commit message: Silk: the front no longer says HEADER ON THE BACK; the back says HEADER HERE, which is enough
A "not here" note under the holes on every board, the kind of text that
narrates instead of naming. The back carries the header's outline with
HEADER HERE and NOTCH TO TOP; the front keeps the pin numbers 1, 2, 63,
64. All 26 boards re-silked in place from their plans (no re-route, the
schematics untouched); the order gate's silk rule now wants HEADER HERE
on the back and no HEADER ON THE BACK anywhere. Gate all pass, every
builder writes what is committed, parts tables unchanged.

Co-Authored-By: Claude Fable 5.1 <noreply@anthropic.com>
Claude-Session: https://claude.ai/code/session_01RktbhdQjDu7SpFpvkevyUU
Other:
- board text removed: "HEADER ON THE BACK"
Changed lines of the file:
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@@
-		)
-	)
-	(gr_text "HEADER ON THE BACK"
-		(at 26.63 12.2 0)
-		(layer "F.SilkS")
-		(effects
-			(font
-				(size 1 1)
-				(thickness 0.15)
-			)
-			(justify left)
 		)
 	)

Commit message: The Nibble logo on the front silkscreen of every board
lib/logo/nibble.png traced by sim/logo.py (potracer) into two silkscreen
footprints, lib/nibble.pretty/Logo_Nibble (icon and word, 27 x 8 mm) and
Logo_Nibble_Icon (8 x 8): filled polygons, holes slit in. At 8 mm the
ribbon's lines print 0.39 mm wide and 0.24 mm apart; the fab's minimum
is 0.15. No pads, no copper, out of the parts list and the position file.

pcb.py places it on every board before the labels are fitted
(place_logo): icon and word where a patch 27 x 8 mm is free of pads,
vias, outlines, courtyards, the labels and 1 mm of edge, the icon alone
otherwise, the nearest such patch to the board's name; the fitter then
keeps the labels off it. 25 boards took the full logo, the coupon the
icon. All 26 re-silked in place (no re-route, the schematics untouched).
The order gate wants exactly one logo on a board; bom.py counts it as no
part. Two pcbnew quirks met on the way: a footprint removed in the
fitter's process makes the next loaded board untyped (every hidden
reference became an obstacle and BUS0 on the hub fell back to 0.8 mm),
and after a text is removed the footprints are untyped too, so resilk
takes the old logo off before the texts.

Gate all pass on all 26, every builder writes what is committed, parts
tables unchanged. The pilot's three zips are new again (order-1.md).

Co-Authored-By: Claude Fable 5.1 <noreply@anthropic.com>
Claude-Session: https://claude.ai/code/session_01RktbhdQjDu7SpFpvkevyUU
Parts:
- added LOGO: Logo_Nibble, Logo_Nibble, F.Cu at (61.6, 41.9)

Commit message: The logo on the sequencer alone: one maker's mark, not a product line
With the logo on all 26 the machine looked factory-made. It stays on the
sequencer, the big board in the middle that people look at; the cards
carry their name. A board gets the logo when its plan says extra.logo
(the sequencer's builder does), none otherwise, and the order gate holds
each board to its plan. The 25 cards re-silked in place (no re-route).
Gate all pass, builders write what is committed, parts tables unchanged.
The pilot's three zips are new again (order-1.md).

Co-Authored-By: Claude Fable 5.1 <noreply@anthropic.com>
Claude-Session: https://claude.ai/code/session_01RktbhdQjDu7SpFpvkevyUU
Parts:
- removed LOGO: Logo_Nibble, Logo_Nibble

Commit message: Clock card: the pot's leg holes for the Bourns PTV09A-4; pcb.py --refit
The Alpha RD901F-40 the card was drawn for is not at DigiKey or LCSC; the
Bourns PTV09A-4020F-B105 (1 M linear, 9 mm, shaft up) is, with the same
three pins 2.5 mm apart and its two mounting legs 8.8 mm apart, 7.0 mm
behind the pins, in 2.2 mm holes (the Alpha's are slots 9.6 mm apart,
7.5 mm back). lib/nibble.pretty gets the footprint, drawn from the
maker's recommended layout; pin 1 the counter-clockwise end as before.

pcb.py --refit REF puts the footprint the schematic now names into a
placed part's holes on a routed board: every numbered pad must land
where the old one was and keeps its net, so the copper is untouched (only
the GND pour backs away from the two new leg pads); DRC 0, 0 unconnected,
fab outputs regenerated. The clock card was not in the pilot order.

ksch.write_fp_lib_table: the project's own library table, written by the
hub's and now the clock's builder. bom.py, order-1.md and audit.md name
the Bourns part; rebuild_check clock hub: the builders write what is
committed; bom --check and the pins selftest pass.

Co-Authored-By: Claude Fable 5.1 <noreply@anthropic.com>
Parts:
- RV1: footprint Potentiometer_Alpha_RD901F-40-00D_Single_Vertical -> Potentiometer_Bourns_PTV09A-4_Single_Vertical
